File: AWS PROJECT/AWS PROJECT.kicad_pcb (KiCad board)
At the start: 2 copper layers, 99 parts, among them J1 MEM2067-02-180-00-A_REVB, J11 Conn_01x01_Pin, J12 Conn_01x01_Pin, J14 Conn_01x01_Pin, J15 Conn_01x01_Pin, J16 Conn_01x01_Pin, J17 Conn_01x02_Pin, J2 SIM7100-8-1-15-00-A_REVC, J3 Conn_01x04_Pin, J4 10118194-0001LF, J5 Conn_01x02_Pin, J6 Conn_01x02_Pin, J7 Conn_01x02_Pin, J8 Conn_01x01_Pin, J9 Screw_Terminal_01x02, Q1 MMBT3904, Q2 MMBT3904, Q6 MMBT3904, SW1 SW_SPST, SW2 SW_SPST, SW3 SW_SPST, SW4 SW_SPST, U1 DS3231MZ_TRL, U2 ESP32-WROOM-32E__4MB_HIGH_TEM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, U3 Ai-Thinker RA-08H, U4 SIM7000E, U5 ST3485EBDR, U6 TXB0108RGYR

Commit message: finalised schematic
Parts:
- added C22: 0.1uF, Capacitor_SMD:C_0603_1608Metric, F.Cu at (144.9, 66.3)
- added C23: 0.1uF, Capacitor_SMD:C_0603_1608Metric, F.Cu at (144.9, 68.8)
- added C25: 10uF, Capacitor_SMD:C_1206_3216Metric_Pad1.33x1.80mm_HandSolder, F.Cu at (153.9, 80.5)
- added C26: 0.1uF, Capacitor_SMD:C_0603_1608Metric, F.Cu at (144.9, 71.3)
- added D4: NET_LED, Diode_SMD:D_0603_1608Metric, F.Cu at (157.3, 66.4)
- added D6: NET_LED, Diode_SMD:D_0603_1608Metric, F.Cu at (157.3, 69.0)
- added J10: Conn_01x03_Pin, Connector_Phoenix_MC:PhoenixContact_MC_1,5_3-GF-3.81_1x03_P3.81mm_Horizontal_ThreadedFlange_MountHole, F.Cu at (177.1, 40.6)
- added J13: Conn_01x04_Pin, Connector_Phoenix_MC:PhoenixContact_MC_1,5_4-GF-3.5_1x04_P3.50mm_Horizontal_ThreadedFlange_MountHole, F.Cu at (200.9, 40.6)
- added J18: Conn_01x02_Pin, Connector_Phoenix_MC:PhoenixContact_MC_1,5_2-GF-3.5_1x02_P3.50mm_Horizontal_ThreadedFlange_MountHole, F.Cu at (200.9, 65.0)
- added J19: Conn_01x02_Pin, Connector_Phoenix_MC:PhoenixContact_MC_1,5_2-GF-3.5_1x02_P3.50mm_Horizontal_ThreadedFlange_MountHole, F.Cu at (200.9, 77.2)
- added J20: Conn_01x03_Pin, Connector_Phoenix_MC:PhoenixContact_MC_1,5_3-GF-3.81_1x03_P3.81mm_Horizontal_ThreadedFlange_MountHole, F.Cu at (177.1, 52.8)
- added J21: Conn_01x03_Pin, Connector_Phoenix_MC:PhoenixContact_MC_1,5_3-GF-3.81_1x03_P3.81mm_Horizontal_ThreadedFlange_MountHole, F.Cu at (177.1, 65.0)
- added J22: Conn_01x04_Pin, Connector_Phoenix_MC:PhoenixContact_MC_1,5_4-GF-3.5_1x04_P3.50mm_Horizontal_ThreadedFlange_MountHole, F.Cu at (200.9, 52.8)
- added J23: Conn_01x03_Pin, Connector_Phoenix_MC:PhoenixContact_MC_1,5_3-GF-3.81_1x03_P3.81mm_Horizontal_ThreadedFlange_MountHole, F.Cu at (177.1, 77.2)
- added J24: Conn_01x03_Pin, Connector_Phoenix_MC:PhoenixContact_MC_1,5_3-GF-3.81_1x03_P3.81mm_Horizontal_ThreadedFlange_MountHole, F.Cu at (177.1, 89.3)
- added JP7: Jumper_2_Small_Open, Jumper:SolderJumper-2_P1.3mm_Open_RoundedPad1.0x1.5mm, F.Cu at (153.1, 66.8)
- added JP8: Jumper_2_Small_Open, Jumper:SolderJumper-2_P1.3mm_Open_RoundedPad1.0x1.5mm, F.Cu at (153.1, 70.4)
- added R15: 1k, Resistor_SMD:R_0603_1608Metric, F.Cu at (144.9, 73.9)
- added R16: 4.7k, Resistor_SMD:R_0603_1608Metric, F.Cu at (144.9, 76.4)
- added R17: 4.7k, Resistor_SMD:R_0603_1608Metric, F.Cu at (148.9, 66.3)
- added R18: 1k, Resistor_SMD:R_0603_1608Metric, F.Cu at (148.9, 68.8)
- added R19: 4.7k, Resistor_SMD:R_0603_1608Metric, F.Cu at (148.9, 71.3)
- added R20: 4.7k, Resistor_SMD:R_0603_1608Metric, F.Cu at (148.9, 73.9)
- added R21: 4.7k, Resistor_SMD:R_0603_1608Metric, F.Cu at (148.9, 76.4)
- added U7: ~, Package_DFN_QFN:DFN-6-1EP_3x3mm_P1mm_EP1.5x2.4mm, F.Cu at (145.4, 82.1)
- added U8: MPL3115A2, MPL3115A2:PSON125P300X500X120-8N, F.Cu at (153.9, 75.5)
- moved GSM2 0.44 mm to (113.0, 79.5)

Commit message: first pcb draft
Parts:
- removed the J24 at (177.1, 89.3)
- added J18: Conn_01x03_Pin, Connector_Phoenix_MC:PhoenixContact_MC_1,5_3-GF-3.81_1x03_P3.81mm_Horizontal_ThreadedFlange_MountHole, F.Cu at (127.1, 40.3)
- added REF**: MountingHole_3.2mm_M3_Pad_Via, MountingHole:MountingHole_3.2mm_M3_Pad_Via, F.Cu at (131.2, 128.0)
- added REF**: MountingHole_3.2mm_M3_Pad_Via, MountingHole:MountingHole_3.2mm_M3_Pad_Via, F.Cu at (131.2, 20.2)
- added REF**: MountingHole_3.2mm_M3_Pad_Via, MountingHole:MountingHole_3.2mm_M3_Pad_Via, F.Cu at (38.2, 128.0)
- added REF**: MountingHole_3.2mm_M3_Pad_Via, MountingHole:MountingHole_3.2mm_M3_Pad_Via, F.Cu at (38.2, 20.2)
- BT1: moved to B.Cu
- C25: renamed from C19; moved to B.Cu
- D13: renamed from D15; moved to B.Cu
- J1: renamed from J4; moved to B.Cu
- J19: renamed from J1; moved to B.Cu
- J24: renamed from J9; footprint Connector_Phoenix_MC:PhoenixContact_MCV_1,5_2-GF-3.5_1x02_P3.50mm_Vertical_ThreadedFlange_MountHole -> Connector_Phoenix_MC:PhoenixContact_MC_1,5_2-GF-3.5_1x02_P3.50mm_Horizontal_ThreadedFlange_MountHole
- JP8: renamed from JP4; moved to B.Cu
- R30: renamed from R33; moved to B.Cu
- R34: renamed from R32; moved to B.Cu
- moved J14 163.8 mm to (42.7, 107.3), turned to -90 degrees
- moved J16 160.0 mm to (42.2, 32.8), turned to -90 degrees
- moved J21 148.6 mm to (54.7, 124.8)
- moved J22 138.3 mm to (42.2, 83.2), turned to -90 degrees
- moved J23 134.6 mm to (42.6, 59.2), turned to -90 degrees
- moved J15 130.5 mm to (79.3, 124.6)
- moved J20 130.0 mm to (101.3, 124.1)
- moved J24 109.7 mm to (57.4, 24.1), turned to 180 degrees
- moved R35 102.7 mm to (47.2, 62.2), turned to 90 degrees
- moved J9 98.6 mm to (107.8, 23.5), turned to -90 degrees
- moved D8 93.5 mm to (69.2, 97.5), turned to 180 degrees
- moved U8 93.0 mm to (56.4, 34.3), turned to 90 degrees
- moved R21 92.7 mm to (62.5, 99.8)
- moved JP3 92.4 mm to (65.5, 96.3), turned to 90 degrees
- moved C16 85.8 mm to (68.2, 104.8), turned to -90 degrees
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- renumbered C11 to C1, C3 to C10, C5 to C11, C7 to C12, C6 to C13, C12 to C14, C26 to C15, C22 to C16, C23 to C19, C13 to C2, C25 to C20, C15 to C21, C20 to C22, C16 to C23, C21 to C24, C10 to C3, C2 to C4, C14 to C5, C1 to C6, C9 to C7, C4 to C9, D3 to D1, D11 to D10, D6 to D11, D16 to D12, D1 to D2, D14 to D3, D2 to D4, D10 to D6, D13 to D7, D4 to D8, D12 to D9, GSM2 to GSM1, GSM3 to GSM2, J2 to J10, J5 to J11, J6 to J12, J7 to J13, J18 to J14, J19 to J15, J22 to J16, J23 to J17, J17 to J2, J13 to J20, J10 to J21, J20 to J22, J21 to J23, J16 to J3, J8 to J4, J11 to J5, J12 to J6, J14 to J7, J15 to J8, J3 to J9, JP7 to JP3, JP3 to JP4, JP8 to JP5, JP5 to JP6, JP6 to JP7, Q2 to Q1, Q1 to Q2, Q6 to Q3, R13 to R1, R5 to R10, R3 to R11, R10 to R12, R11 to R13, R12 to R14, R28 to R15, R15 to R16, R20 to R17, R19 to R18, R35 to R19, R8 to R2, R34 to R20, R17 to R21, R27 to R22, R31 to R23, R36 to R24, R37 to R25, R16 to R26, R18 to R27, R38 to R28, R30 to R29, R6 to R3, R39 to R31, R40 to R32, R14 to R33, R21 to R35, R41 to R36, R9 to R4, R7 to R5, R1 to R6, R29 to R7, R4 to R8, R2 to R9, SW4 to SW3, SW3 to SW4, U6 to U1, U4 to U3, U8 to U4, U7 to U5, U1 to U6, U3 to U7, U5 to U8
Connections:
- R10 pad 1: /gate way/power in -> /gate way/ESP32 power in
- R17 pad 1: /gate way/I2C SDA -> /gate way/I2C SCL
- R2 pad 1: unconnected-(R8-Pad1) -> /gate way/gsm reset
- R3 pad 1: unconnected-(R6-Pad1) -> /gate way/gsm power key
- R8 pad 1: /gate way/power in -> /gate way/ESP32 power in
- U1 pad 1: /gate way/tx -> /gate way/gsm tx
- U1 pad 3: /gate way/rx -> /gate way/gsm rx
- U2 pad 26: unconnected-(U2-IO4-Pad26) -> /gate way/gsm power key
- U2 pad 5: unconnected-(U2-SENSOR_VN-Pad5) -> /gate way/gsm reset
- U3 pad 10: /gate way/rx -> /gate way/gsm rx
- U3 pad 9: /gate way/tx -> /gate way/gsm tx
Routing:
- net 3v3: track 0.00 -> 268.4 mm, vias 0 -> 7
- net /gate way/I2C SDA: track 0.00 -> 219.9 mm, vias 0 -> 8
- net /gate way/I2C SCL: track 0.00 -> 210.0 mm, vias 0 -> 5
- net /gate way/S1223: track 0.00 -> 127.4 mm, vias 0 -> 1
- net /gate way/INSPEEED VANE: track 0.00 -> 107.5 mm, vias 0 -> 1
- net /gate way/INSPEED VORTEX: track 0.00 -> 97.7 mm, vias 0 -> 1
- net Net-(U6-VBAT): track 0.00 -> 91.2 mm, vias 0 -> 1
- net /gate way/gsm reset: track 0.00 -> 79.6 mm, vias 0 -> 5
- net /gate way/lora power in: track 0.00 -> 76.9 mm, vias 0 -> 4
- net /gate way/VH400: track 0.00 -> 76.6 mm, vias 0 -> 1
- net /gate way/SD CS: track 0.00 -> 73.4 mm, vias 0 -> 1
- net /gate way/DAVIS 7852: track 0.00 -> 69.6 mm, vias 0 -> 1
- net /gate way/VSPI-MOSI: track 0.00 -> 68.7 mm, vias 0 -> 1
- net /gate way/GSM_pw in: track 0.00 -> 67.2 mm, vias 0 -> 4
- net /gate way/rx: track 0.00 -> 63.7 mm, vias 0 -> 2
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- added copper zone on B.Cu, net GND
- added copper zone on F.Cu, net GND
Other:
- board outline added: 103 x 117.8 mm
- board text added: "www.iot-ra.net"
