File: AWS PROJECT/power.kicad_sch (KiCad schematic)
At the start: 0 parts

Commit message: first pcb draft
Other:
- company: (none) -> AdeMNEA IoT-ra
- title: (none) -> POWER SCHEMATIC
Changed lines of the file:
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@@
 	(generator_version "9.0")
 	(paper "A4")
+	(title_block
+		(title "POWER SCHEMATIC")
+		(date "2025-11-03")
+		(rev "V-1.1")
+		(company "AdeMNEA IoT-ra")
+		(comment 1 "Designed By TN Muhanguzi")
+		(comment 2 "For MPSE Research at Makerere University")
+	)
 )

Commit message: finalised power schematic
Parts:
- added C26, C28: 10uF, Capacitor_SMD:CP_Elec_5x5.8, symbol Device:C_Polarized_Small_US
- added C27: 10uF, Capacitor_Tantalum_SMD:CP_EIA-3528-12_Kemet-T, symbol Device:C_Polarized
- added C29: 100nF, Capacitor_SMD:C_1206_3216Metric_Pad1.33x1.80mm_HandSolder, symbol Device:C
- added C30: 10nF, Capacitor_SMD:C_0603_1608Metric_Pad1.08x0.95mm_HandSolder, symbol Device:C
- added C31: OPEN, Capacitor_SMD:C_0201_0603Metric_Pad0.64x0.40mm_HandSolder, symbol Device:C
- added C32: 2.7nF, Capacitor_SMD:C_0603_1608Metric, symbol Device:C
- added C33, C35, C36: 22uF, Capacitor_SMD:C_0603_1608Metric_Pad1.08x0.95mm_HandSolder, symbol Device:C
- added C34: 33pF, Capacitor_SMD:C_0603_1608Metric, symbol Device:C
- added C37: 0.01uF, Capacitor_SMD:C_0603_1608Metric_Pad1.08x0.95mm_HandSolder, symbol Device:C
- added C52, C60: 2.2uF, Capacitor_SMD:C_0603_1608Metric_Pad1.08x0.95mm_HandSolder, symbol Device:C
- added C53, C64: 22pF, Capacitor_SMD:C_0603_1608Metric_Pad1.08x0.95mm_HandSolder, symbol Device:C
- added C54, C55, C57, C63: 1uF, Capacitor_SMD:C_0603_1608Metric_Pad1.08x0.95mm_HandSolder, symbol Device:C
- added C56: 0.1uf, Capacitor_SMD:C_0603_1608Metric_Pad1.08x0.95mm_HandSolder, symbol Device:C
- added C58, C59, C65: 10uF, Capacitor_SMD:C_1210_3225Metric_Pad1.33x2.70mm_HandSolder, symbol Device:C
- added C61: 0.1uF, Capacitor_SMD:C_0603_1608Metric_Pad1.08x0.95mm_HandSolder, symbol Device:C
- added C62: 10uF, Capacitor_SMD:C_0603_1608Metric_Pad1.08x0.95mm_HandSolder, symbol Device:C
- added D14, D15: NET_LED, Diode_SMD:D_0603_1608Metric, symbol Device:LED
- added D16, D23: D, Diode_SMD:D_1210_3225Metric, symbol Device:D
- added D22: PESDHC3D3V3U, Diode_SMD:D_SOD-323F, symbol PCM_JLCPCB-Diodes:TVS-Uni,SMAJ10A
- added J25, J26, J27, J28, J29: Screw_Terminal_01x02, TerminalBlock_MetzConnect:TerminalBlock_MetzConnect_Type011_RT05502HBWC_1x02_P5.00mm_Horizontal, symbol Connector:Screw_Terminal_01x02
- added JP10, JP11, JP12, JP13, JP18, JP9: Jumper_2_Small_Open, Jumper:SolderJumper-2_P1.3mm_Open_RoundedPad1.0x1.5mm, symbol Jumper:Jumper_2_Small_Open
- added JP19: Jumper_2_Small_Open, Jumper:SolderJumper-2_P1.3mm_Open_Pad1.0x1.5mm, symbol Jumper:Jumper_2_Small_Open
- added L1: SRN6045TA-3R3Y, Inductor_SMD:L_Bourns_SRN6045TA, symbol Device:L
- added L3: SRN6045TA-3R3Y, Inductor_SMD:L_APV_APH2213, symbol Device:L
- added Q12, Q4: 2N7002, PCM_JLCPCB:Q_SOT-23, symbol PCM_JLCPCB-Transistors:NMOS,2N7002
- added Q5, Q9: NMOS, NTMFS4H01NFT3G:TRANS_NVMFS5834NLWFT1G, symbol Simulation_SPICE:NMOS
- added R37, R38: R, Resistor_SMD:R_0603_1608Metric, symbol Device:R
- added R39, R40, R41: 5K1, Resistor_SMD:R_0603_1608Metric_Pad0.98x0.95mm_HandSolder, symbol Device:R
- added R42, R44: 23.7k, Resistor_SMD:R_0603_1608Metric_Pad0.98x0.95mm_HandSolder, symbol Device:R
- added R43, R45: 5k, Resistor_SMD:R_0603_1608Metric_Pad0.98x0.95mm_HandSolder, symbol Device:R
- added R46: 51.1K, Resistor_SMD:R_0603_1608Metric_Pad0.98x0.95mm_HandSolder, symbol Device:R
- added R47, R48: 3.9, Resistor_SMD:R_0603_1608Metric, symbol Device:R
- added R66: 499K, Resistor_SMD:R_0603_1608Metric, symbol Device:R
- added R67: 36K, Resistor_SMD:R_0603_1608Metric, symbol Device:R
- added R68: 25k, Resistor_SMD:R_0603_1608Metric, symbol Device:R
- added R69, R70: 10K, Resistor_SMD:R_0603_1608Metric, symbol Device:R
- added R71: 5.23k, Resistor_SMD:R_0603_1608Metric, symbol Device:R
- added R72: 7.5k, Resistor_SMD:R_0603_1608Metric, symbol Device:R
- added R73: 10, Resistor_SMD:R_0603_1608Metric, symbol Device:R
- added R74: 100, Resistor_SMD:R_0603_1608Metric, symbol Device:R
- added R75: 2.2, Resistor_SMD:R_0603_1608Metric, symbol Device:R
- added R76: 10, Resistor_SMD:R_1812_4532Metric, symbol Device:R
- added R77: 4.22M, Resistor_SMD:R_0603_1608Metric, symbol Device:R
- added R78: 154k, Resistor_SMD:R_0603_1608Metric, symbol Device:R
- added R79: 887k, Resistor_SMD:R_0603_1608Metric, symbol Device:R
- added R80: 162k, Resistor_SMD:R_0603_1608Metric, symbol Device:R
- added SW5, SW6: SW_SPST, Button_Switch_THT:SW_DIP_SPSTx01_Slide_9.78x4.72mm_W7.62mm_P2.54mm, symbol Switch:SW_SPST
- added TH2: 100k, Resistor_SMD:R_1812_4532Metric, symbol Device:Thermistor_NTC
- added TP1: TestPoint, TestPoint:TestPoint_Pad_1.0x1.0mm, symbol Connector:TestPoint
- added U10: BQ24650RVAR, BQ24650RVAR:QFN50P350X350X100-17N, symbol BQ24650RVAR:BQ24650RVAR
- added U11: LM1085IS-3.3, LM1085IS-3.3:TI_LM1085IS-3.3, symbol LM1085IS-3.3:LM1085IS-3.3
- added U12: TPS2121RUXR, TPS2121RUXR:IC_TPS2121RUXR, symbol TPS2121RUXR:TPS2121RUXR
- added U13: AP64501SP-13, AP64501SP-13:SOIC127P600X170-9N, symbol ap64501:AP64501SP-13
Connections:
- new net: C58.1, C59.1, C65.1, D16.1 (K), D23.1 (K), JP18.1 (A), Q9.5_6 (D), R73.2
- new net: C31.1, C33.1, C35.1, C36.1, JP12.1 (A), L1.2, R39.1
- new net: C29.2, U13.1 (BST)
- new net: C30.1, U13.4 (SS)
- new net: R78.1, R79.2, TH2.2
- new net: C32.1, R41.1
- new net: C34.1, R41.2, U13.6 (COMP)
- new net: R71.1, R72.2, R74.1
- new net: J26.2 (Pin_2), SW5.1 (A)
- new net: JP13.1 (A), U12.1 (OUT), U12.1_1 (OUT), U12.8 (OUT), U12.8_1 (OUT)
- new net: R46.1, U12.10 (ILIM)
- new net: C37.1, U12.11 (SS)
- new net: J25.2 (Pin_2), SW6.1 (A)
- new net: C28.1, JP11.1 (A), U13.2 (VIN), U13.3 (EN)
- new net: Q12.3 (D), R77.1
- new net: D14.2 (A), R69.1
- new net: C55.1, R73.1, U10.1 (VCC)
- new net: C26.1, JP9.1 (A), U11.3 (INPUT)
- new net: C56.1, D22.1, R75.1
- new net: R37.2, R38.1, U11.1 (ADJ/GND)
- new net: D15.2 (A), R68.2, R70.1
- new net: C52.1, R47.1, R48.1
- new net: C27.1, JP10.1 (A), R37.1, U11.2 (OUTPUT), U11.4 (OUTPUT), U11.5 (OUTPUT)
- new net: C53.2, Q4.3 (D), R66.1, R67.2, U10.2 (MPPSET)
- new net +3.3V: J29.1 (Pin_1), JP10.2 (B)
- new net +5V: J28.1 (Pin_1), JP12.2 (B), JP9.2 (B)
- new net BATTERY BMS: J27.1 (Pin_1), JP19.2 (B)
- new net CE: Q4.1 (G), TP1.1
- new net DC JACK INPUT: R42.1, SW5.2 (B), U12.2 (IN2), U12.2_1 (IN2)
- new net FB: C31.2, R39.2, R40.1, U13.5 (FB)
- new net GND: C26.2, C27.2, C28.2, C30.2, C32.2, C33.2, C34.2, C35.2, C36.2, C37.2, C52.2, C54.2, C55.2, C57.2, C58.2, C59.2, C61.2, C62.2, C63.2, C65.2, J25.1 (Pin_1), J26.1 (Pin_1), J27.2 (Pin_2), J28.2 (Pin_2), J29.2 (Pin_2), Q12.2 (S), Q4.2 (S), Q5.1 (S), Q5.2 (S), Q5.3 (S), R38.2, R40.2, R43.2, R45.2, R46.2, R67.1, R68.1, R72.1, R80.1, U10.11 (GND), U10.17 (EP), U12.12 (GND), U12.3 (CP2), U12.6 (PR1), U12.9 (ST), U13.7 (GND), U13.EPAD (GND)
- new net MUXOUT: C53.1, D16.2 (A), JP13.2 (B), R47.2, R48.2, R66.2, R69.2, R70.2
- new net OV1: R44.2, R45.1, U12.5 (OV1)
- new net OV2: R42.2, R43.1, U12.4 (OV2)
- new net SOLAR INPUT: R44.1, SW6.2 (B), U12.7 (IN1), U12.7_1 (IN1)
- new net SW_AP: C29.1, L1.1, U13.8 (SW)
- new net Vbuck: JP11.2 (B), JP18.2 (B)
- new net btst: R75.2, U10.16 (BTST)
- new net hidriv: Q9.4 (G), U10.15 (HIDRV)
- new net lodriv: Q5.4 (G), U10.13 (LODRV)
- new net ph: C56.2, L3.1, Q5.5_6 (D), Q9.1 (S), Q9.2 (S), Q9.3 (S), U10.14 (PH)
- new net regn: C57.1, D22.2, U10.12 (REGN)
- new net srn: C60.2, C62.1, C63.1, C64.1, D23.2 (A), JP19.1 (A), R76.2, R78.2, TH2.1, U10.9 (SRN)
- new net srp: C60.1, C61.1, L3.2, R76.1, U10.10 (SRP)
- new net stat1: D14.1 (K), U10.5 (STAT2)
- new net stat2: D15.1 (K), Q12.1 (G), U10.3 (STAT1)
- new net ts: R74.2, U10.4 (TS)
- new net vfb: C64.2, R77.2, R79.1, R80.2, U10.8 (VFB)
- new net vref: C54.1, R71.2, U10.6 (VREF), U10.7 (TERM_EN)
Other:
- note added: "12V - 5V BUCK CONVERTER"
- note added: "12V - 5V converter"
- note added: "12V / 16v output"
- note added: "3A 3.3V LDO"
- note added: "DC in 17.5 - 19V"
- note added: "MPPT SOLAR CHARGE CONTROLLER"
- note added: "POWER MULTIPLEXER"
- note added: "R1"
- note added: "R2"
- note added: "TO BMS"
- note added: "Vout = 1.25(1 + R2/R1)"
- note added: "bms can be 3S /4S"
- note added: "for setting battery output voltage"
- note added: "for setting input voltage"
- note added: "input power must be >15v"
- note added: "solar no load voltage 22V MP 17.5V"
