File: AWS PROJECT/power.kicad_sch (KiCad schematic)
At the start: 84 parts, among them J25 Screw_Terminal_01x02, J26 Screw_Terminal_01x02, J27 Screw_Terminal_01x02, J28 Screw_Terminal_01x02, J29 Screw_Terminal_01x02, Q12 2N7002, Q4 2N7002, Q5 NMOS, Q9 NMOS, SW5 SW_SPST, SW6 SW_SPST, U10 BQ24650RVAR, U11 LM1085IS-3.3, U12 TPS2121RUXR, U13 AP64501SP-13

Commit message: algorirthim design start
Parts:
- removed J28, J29: Screw_Terminal_01x02, TerminalBlock_MetzConnect:TerminalBlock_MetzConnect_Type011_RT05502HBWC_1x02_P5.00mm_Horizontal, symbol Connector:Screw_Terminal_01x02
- added BOOT1, RST1: Jumper_2_Small_Open, Connector_PinHeader_2.54mm:PinHeader_1x02_P2.54mm_Vertical, symbol Jumper:Jumper_2_Small_Open
- added C43: 1uF, Capacitor_SMD:C_0603_1608Metric, symbol Device:C_Small
- added C44, C47, C50: 10nF, Capacitor_SMD:C_0603_1608Metric, symbol Device:C_Small
- added C48, C51: 4.7uF, Capacitor_SMD:C_0603_1608Metric, symbol Device:C_Small
- added C49: 0.1uF, Capacitor_SMD:C_0603_1608Metric, symbol Device:C_Small
- added C66, C67: 27pF, Capacitor_SMD:C_0603_1608Metric, symbol Device:C_Small
- added D19: D, Diode_SMD:D_1210_3225Metric, symbol Device:D
- added D24: green, LED_SMD:LED_1206_3216Metric, symbol Device:LED
- added D25: red, LED_SMD:LED_1206_3216Metric, symbol Device:LED
- added DBG_RX1, DBG_TX1: TestPoint, Connector_PinHeader_2.54mm:PinHeader_1x01_P2.54mm_Vertical, symbol Connector:TestPoint
- added J22, J36: B4B-XH-A_LF__SN_, B4B-XH-A_LF__SN_:JST_B4B-XH-A_LF__SN_, symbol B4B-XH-A_LF__SN_:B4B-XH-A_LF__SN_
- added J30, J33: B2B-XH-A_LF__SN_, B2B-XH-A_LF__SN_:JST_B2B-XH-A_LF__SN_, symbol B2B-XH-A_LF__SN_:B2B-XH-A_LF__SN_
- added JP15: Jumper_2_Small_Open, Jumper:SolderJumper-2_P1.3mm_Open_RoundedPad1.0x1.5mm, symbol Jumper:Jumper_2_Small_Open
- added OSC_IN1, OSC_OUT1, PB8, PB9, RS_RX1, RS_TX1, SNS_RX1, SNS_TX1: TestPoint, TestPoint:TestPoint_Pad_D1.5mm, symbol Connector:TestPoint
- added R54, R55, R63: 10K, Resistor_SMD:R_0603_1608Metric, symbol Device:R
- added R61: 330, Resistor_SMD:R_0603_1608Metric, symbol Device:R
- added R62: 1M, Resistor_SMD:R_0603_1608Metric, symbol Device:R
- added U16: STM32F103C8T6, STM32F103C8T6:QFP50P900X900X160-48N, symbol STM32F103C8T6:STM32F103C8T6
- added X1: X50328MSB2GI, PCM_JLCPCB:CRYSTAL-SMD_L5.0-W3.2, symbol PCM_JLCPCB-Crystals:Crystal, 8MHz, 20pF, ±10ppm
Connections:
- net +3.3V: now also J36.3, JP15.2 (B)
- net +5V: now also J36.1
- net CE: now also U16.42 (PB6)
- net FB: now also U16.39 (PB3)
- net GND: now also C43.2, C44.2, C47.2, C48.2, C49.2, C50.2, C51.2, C66.2, C67.2, J36.2, J36.4, R54.1, R55.1, R61.1, R63.1, U16.23 (VSS), U16.35 (VSS), U16.47 (VSS), U16.8 (VSSA)
- net OV1: now also U16.41 (PB5)
- net OV2: now also U16.28 (PB15)
- net vfb: now also U16.40 (PB4)
- net 3v3 comout: now reaches R37.2, R38.1, U11.1 (ADJ/GND)
- net 3v3 comout: now also U16.20 (PB2)
- net at C27.1, R37.1, U11.2 (OUTPUT)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: now also D19.2 (A); no longer JP10.1 (A)
- net mpptset: now reaches C53.2, Q4.3 (D), R66.1, R67.2, U10.2 (MPPSET)
- net mpptset: now also U16.25 (PB12)
- new net: OSC_IN1.1, U16.5 (PD0_OSC_IN)
- new net: RS_RX1.1, U16.12 (PA2)
- new net: PB8.1, U16.45 (PB8)
- new net: DBG_TX1.1, U16.21 (PB10)
- new net: RS_TX1.1, U16.13 (PA3)
- new net: DBG_RX1.1, U16.22 (PB11)
- new net: SNS_RX1.1, U16.30 (PA9)
- new net: SNS_TX1.1, U16.31 (PA10)
- new net: PB9.1, U16.46 (PB9)
- new net: OSC_OUT1.1, U16.6 (PD1_OSC_OUT)
- new net: R54.2, RST1.1 (A)
- new net: D24.1 (K), R61.2
- new net: BOOT1.1 (A), R55.2
- new net: D19.1 (K), JP10.1 (A)
- new net: D25.1 (K), R63.2
- new net CS: J22.1, U16.14 (PA4)
- new net MCU MISO: J22.3, U16.16 (PA6)
- new net MCU MOSI: J22.4, U16.17 (PA7)
- new net MCU SCK: J22.2, U16.15 (PA5)
- new net MCU power: BOOT1.2 (B), C43.1, C44.1, C47.1, C48.1, C49.1, C50.1, C51.1, D25.2 (A), JP15.1 (A), RST1.2 (B), U16.1 (VBAT), U16.24 (VDD), U16.36 (VDD), U16.44 (BOOT0), U16.48 (VDD), U16.7 (NRST), U16.9 (VDDA)
- new net MCU_SCL: J30.1, U16.34 (PA13)
- new net MCU_SDA: J30.2, U16.37 (PA14)
- new net SWDCLK: J33.2, U16.27 (PB14)
- new net SWDIO: J33.1, U16.26 (PB13)
- new net c-i: C67.1, R62.1, U16.18 (PB0), X1.2
- new net c-o: C66.1, R62.2, U16.19 (PB1), X1.1
- new net debug_led (PWM): D24.2 (A), U16.43 (PB7)
- no-connect marks 0 -> 9
Other:
- note added: "BOOT AND RESET OPTION"
- note added: "CRYSTAL OSCILLATOR"
- note added: "MICROCONTROLLER SECTION"
- note added: "PROGRAMING INTERFACE"
- note added: "boot and reset is active low,"
- note added: "power indication led"
- moved on the sheet: C26, C27, C28, C29, C30, C31, C32, C33, C34, C35, C36, C37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

Commit message: updates to the power board
Parts:
- removed BOOT1, RST1: Jumper_2_Small_Open, Connector_PinHeader_2.54mm:PinHeader_1x02_P2.54mm_Vertical, symbol Jumper:Jumper_2_Small_Open
- removed C26: 10uF, Capacitor_SMD:CP_Elec_5x5.8, symbol Device:C_Polarized_Small_US
- removed C27: 10uF, Capacitor_Tantalum_SMD:CP_EIA-3528-12_Kemet-T, symbol Device:C_Polarized
- removed C47, C50: 10nF, Capacitor_SMD:C_0603_1608Metric, symbol Device:C_Small
- removed C48, C51: 4.7uF, Capacitor_SMD:C_0603_1608Metric, symbol Device:C_Small
- removed C49: 0.1uF, Capacitor_SMD:C_0603_1608Metric, symbol Device:C_Small
- removed C66, C67: 27pF, Capacitor_SMD:C_0603_1608Metric, symbol Device:C_Small
- removed D19: D, Diode_SMD:D_1210_3225Metric, symbol Device:D
- removed D24: green, LED_SMD:LED_1206_3216Metric, symbol Device:LED
- removed D25: red, LED_SMD:LED_1206_3216Metric, symbol Device:LED
- removed DBG_RX1, DBG_TX1: TestPoint, Connector_PinHeader_2.54mm:PinHeader_1x01_P2.54mm_Vertical, symbol Connector:TestPoint
- removed J22: B4B-XH-A_LF__SN_, B4B-XH-A_LF__SN_:JST_B4B-XH-A_LF__SN_, symbol B4B-XH-A_LF__SN_:B4B-XH-A_LF__SN_
- removed J30, J33: B2B-XH-A_LF__SN_, B2B-XH-A_LF__SN_:JST_B2B-XH-A_LF__SN_, symbol B2B-XH-A_LF__SN_:B2B-XH-A_LF__SN_
- removed JP10, JP15: Jumper_2_Small_Open, Jumper:SolderJumper-2_P1.3mm_Open_RoundedPad1.0x1.5mm, symbol Jumper:Jumper_2_Small_Open
- removed L3: SRN6045TA-3R3Y, Inductor_SMD:L_APV_APH2213, symbol Device:L
- removed OSC_IN1, OSC_OUT1, RS_RX1, RS_TX1, SNS_RX1, SNS_TX1: TestPoint, TestPoint:TestPoint_Pad_D1.5mm, symbol Connector:TestPoint
- removed R38: R, Resistor_SMD:R_0603_1608Metric, symbol Device:R
- removed R54, R55, R63: 10K, Resistor_SMD:R_0603_1608Metric, symbol Device:R
- removed R61: 330, Resistor_SMD:R_0603_1608Metric, symbol Device:R
- removed R62: 1M, Resistor_SMD:R_0603_1608Metric, symbol Device:R
- removed U11: LM1085IS-3.3, LM1085IS-3.3:TI_LM1085IS-3.3, symbol LM1085IS-3.3:LM1085IS-3.3
- removed U16: STM32F103C8T6, STM32F103C8T6:QFP50P900X900X160-48N, symbol STM32F103C8T6:STM32F103C8T6
- removed X1: X50328MSB2GI, PCM_JLCPCB:CRYSTAL-SMD_L5.0-W3.2, symbol PCM_JLCPCB-Crystals:Crystal, 8MHz, 20pF, ±10ppm
- added C26, C27, C68, C69: 0.1uF, Capacitor_SMD:C_0603_1608Metric, symbol Device:C_Small
- added C45, C46: 22pF, Capacitor_SMD:C_0603_1608Metric, symbol Device:C_Small
- added C70, C72: 4.7uF, Capacitor_SMD:C_0603_1608Metric, symbol Device:C_Small
- added C71: 10nF, Capacitor_SMD:C_0603_1608Metric, symbol Device:C_Small
- added C73: 10uF, Capacitor_SMD:C_0603_1608Metric, symbol Device:C_Small
- added C74: 1uF, Capacitor_SMD:C_0603_1608Metric, symbol Device:C_Small
- added D10: red, LED_SMD:LED_1206_3216Metric, symbol Device:LED
- added D19: green, LED_SMD:LED_1206_3216Metric, symbol Device:LED
- added J4: B2B-XH-A_LF__SN_, B2B-XH-A_LF__SN_:JST_B2B-XH-A_LF__SN_, symbol B2B-XH-A_LF__SN_:B2B-XH-A_LF__SN_
- added J5, J6, J7, J8: Conn_01x02_Pin, Connector_PinHeader_2.54mm:PinHeader_1x02_P2.54mm_Vertical, symbol Connector:Conn_01x02_Pin
- added JP20, JP21: Jumper_2_Small_Open, Jumper:SolderJumper-2_P1.3mm_Open_RoundedPad1.0x1.5mm, symbol Jumper:Jumper_2_Small_Open
- added L2: 6.1uH, MPPT INDUCTORS:CDEP147NP-6R1MC-95, symbol Device:L
- added PB1, PB11, PB12, PB13, PB14, PB15, PB16, PB17, PB18, PB19, PB2, PB20, PB21, PB22, PB3, PB4, PB5, PB6, PB7: TestPoint, TestPoint:TestPoint_Pad_D1.0mm, symbol Connector:TestPoint
- added R31, R32, R33, R49, R57, R59, R64, R81: 10K, Resistor_SMD:R_0603_1608Metric, symbol Device:R
- added R56: 20k, Resistor_SMD:R_0603_1608Metric, symbol Device:R
- added R58: 13k, Resistor_SMD:R_0603_1608Metric, symbol Device:R
- added R60: 1.5K, Resistor_SMD:R_0603_1608Metric, symbol Device:R
- added R65: 2k, Resistor_SMD:R_0603_1608Metric, symbol Device:R
- added R82: 1.2K, Resistor_SMD:R_0603_1608Metric, symbol Device:R
- added U15: STM32F401CCU6, STM32F401CCU6 (1):QFN50P700X700X60-49N, symbol STM32F401CCU6:STM32F401CCU6
- added U17: AMS1117-3.3, Package_TO_SOT_SMD:SOT-223-3_TabPin2, symbol Regulator_Linear:AMS1117-3.3
- added Y1: C3E-25.000-12-3030-X-R, C3E-25.000-12-3030-X-R:XTAL_C3E-25.000-12-3030-X-R, symbol C3E-25.000-12-3030-X-R:C3E-25.000-12-3030-X-R
- C43: value 1uF -> 10uF; LCSC C1592 -> (none)
- C44: value 10nF -> 1uF; LCSC C1589 -> (none)
- PB8, PB9: footprint TestPoint:TestPoint_Pad_D1.5mm -> TestPoint:TestPoint_Pad_D1.0mm
- R37: value R -> 330; LCSC (none) -> C23138
Connections:
- net +3.3V: now also JP20.2 (B), JP21.2 (B), R49.1
- net +5V: now also R57.1
- net CE: now also U15.16 (PA6)
- net DC JACK INPUT: now also R59.1
- net GND: now also R37.1, C26.2, C27.2, C45.1, C46.1, C68.2, C69.2, C70.2, C71.2, C72.2, C73.2, C74.2, J8.2 (Pin_2), R31.1, R33.1, R56.2, R58.2, R60.2, R65.2, R82.2, U15.23 (VSS), U15.35 (VSS), U15.47 (VSS), U15.49 (EXP), U15.8 (VSSA/VREF-), U17.1 (GND), Y1.2 (GND), Y1.4 (GND)
- net MCU_SCL: now also J4.1, U15.42 (PB6)
- net MCU_SDA: now also J4.2, U15.43 (PB7)
- net SOLAR INPUT: now also R81.1
- net ph: now also L2.1
- net srp: now also L2.2
- net at PB8.1: now also U15.38 (PA15/JTDI)
- net at JP9.1 (A): now also C43.1, C73.1, U17.3 (VI)
- net BOOT1_MCU: now reaches PB9.1
- net BOOT1_MCU: now also U15.20 (PB2)
- net 3v3 comout: no longer names the net of R37.2
- net 3v3 comout: now also D19.1 (K)
- net MCU power: no longer names the net of C44.1
- net MCU power: now also C74.1, JP21.1 (A), U17.2 (VO); no longer C43.1
- net srn renamed BATT_VAL
- net BATT_VAL: now also R64.1
- new net: PB5.1, U15.33 (PA12)
- new net: PB17.1, U15.28 (PB15)
- new net: PB21.1, U15.18 (PB0)
- new net: D19.2 (A), U15.2 (PC13)
- new net: PB16.1, U15.27 (PB14)
- new net: PB15.1, U15.26 (PB13)
- new net: PB18.1, U15.41 (PB5)
- new net: PB4.1, U15.32 (PA11)
- new net: J6.1 (Pin_1), U15.34 (PA13/JTMS-SWDIO)
- new net: J6.2 (Pin_2), U15.37 (PA14/JTCK-SWCLK)
- new net: PB2.1, U15.29 (PA8)
- new net: PB13.1, U15.21 (PB10)
- new net: PB3.1, U15.15 (PA5)
- new net: PB1.1, U15.17 (PA7)
- new net: D10.1 (K), R31.2
- new net: PB12.1, U15.46 (PB9)
- new net: PB19.1, U15.40 (PB4/~{JTRST})
- new net: J5.1 (Pin_1), U15.30 (PA9)
- new net: J5.2 (Pin_2), U15.31 (PA10)
- new net: PB14.1, U15.25 (PB12)
- new net: PB20.1, U15.39 (PB3/JTDO-SWO)
- new net: PB11.1, U15.45 (PB8)
- new net: PB6.1, U15.4 (PC15-OSC32_OUT)
- new net: PB22.1, U15.19 (PB1)
- new net: PB7.1, U15.3 (PC14-OSC32_IN)
- new net 3V3_INPUT: R49.2, R56.1, U15.10 (PA0)
- new net 5V_INPUT: R57.2, R58.1, U15.11 (PA1)
- new net BATT_INPUT: R64.2, R65.1, U15.13 (PA3)
- new net BOOT0_MCU: J7.2 (Pin_2), R33.2, U15.44 (BOOT0)
- new net DC_INPUT: R59.2, R60.1, U15.12 (PA2)
- new net RST_MCU: J8.1 (Pin_1), R32.1, U15.7 (~{RST})
- new net SOLAR_INPUT: R81.2, R82.1, U15.14 (PA4)
- new net VDD: C26.1, C27.1, C68.1, C69.1, C70.1, C71.1, C72.1, D10.2 (A), J7.1 (Pin_1), JP20.1 (A), R32.2, U15.1 (VBAT), U15.22 (VCAP_1), U15.24 (VDD), U15.36 (VDD), U15.48 (VDD), U15.9 (VDDA/VREF+)
- new net cin: C45.2, U15.5 (PH0-OSC_IN), Y1.1
- new net cout: C46.2, U15.6 (PH1-OSC_OUT), Y1.3
- no-connect marks 9 -> 0
Other:
- note added: "JTAG PROGRAMING"
- note added: "UART PROGRAMING"
- note removed: "CRYSTAL OSCILLATOR"
- note removed: "PROGRAMING INTERFACE"
- note removed: "R1"
- note removed: "R2"
- note removed: "Vout = 1.25(1 + R2/R1)"
- moved on the sheet: C28, C29, C30, C31, C32, C33, C34, C35, C36, C37, C52, C53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
