File: AWS PROJECT/AWS PROJECT.kicad_sch (KiCad schematic)
At the start: 0 parts

Commit message: first pcb draft
Other:
- company: (none) -> AdeMNEA IoT-ra
- title: (none) -> GENERAL  DESIGN SHEET
Changed lines of the file:
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@@
 	(generator_version "9.0")
 	(paper "A4")
+	(title_block
+		(title "GENERAL  DESIGN SHEET")
+		(company "AdeMNEA IoT-ra")
+		(comment 1 "Designed By TN Muhanguzi")
+		(comment 2 "For MPSE Research at Makerere University")
+	)
 	(sheet
 		(at 152.4 27.94)
