File: AWS PROJECT/gateway.kicad_sch (KiCad schematic)
At the start: 99 parts, among them J1 MEM2067-02-180-00-A_REVB, J11 Conn_01x01_Pin, J12 Conn_01x01_Pin, J14 Conn_01x01_Pin, J15 Conn_01x01_Pin, J16 Conn_01x01_Pin, J17 Conn_01x02_Pin, J2 SIM7100-8-1-15-00-A_REVC, J3 Conn_01x04_Pin, J4 10118194-0001LF, J5 Conn_01x02_Pin, J6 Conn_01x02_Pin, J7 Conn_01x02_Pin, J8 Conn_01x01_Pin, J9 Screw_Terminal_01x02, Q1 MMBT3904, Q2 MMBT3904, Q6 MMBT3904, SW1 SW_SPST, SW2 SW_SPST, SW3 SW_SPST, SW4 SW_SPST, U1 DS3231MZ_TRL, U2 ESP32-WROOM-32E__4MB_HIGH_TEM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, U3 Ai-Thinker RA-08H, U4 SIM7000E, U5 ST3485EBDR, U6 TXB0108RGYR

Commit message: finalised schematic
Parts:
- added C22, C23, C26: 0.1uF, Capacitor_SMD:C_0603_1608Metric, symbol Device:C_Small
- added C25: 10uF, Capacitor_SMD:C_1206_3216Metric_Pad1.33x1.80mm_HandSolder, symbol Device:C
- added D4, D6: NET_LED, Diode_SMD:D_0603_1608Metric, symbol Device:LED
- added J10, J20, J21, J23, J24: Conn_01x03_Pin, Connector_Phoenix_MC:PhoenixContact_MC_1,5_3-GF-3.81_1x03_P3.81mm_Horizontal_ThreadedFlange_MountHole, symbol Connector:Conn_01x03_Pin
- added J13, J22: Conn_01x04_Pin, Connector_Phoenix_MC:PhoenixContact_MC_1,5_4-GF-3.5_1x04_P3.50mm_Horizontal_ThreadedFlange_MountHole, symbol Connector:Conn_01x04_Pin
- added J18, J19: Conn_01x02_Pin, Connector_Phoenix_MC:PhoenixContact_MC_1,5_2-GF-3.5_1x02_P3.50mm_Horizontal_ThreadedFlange_MountHole, symbol Connector:Conn_01x02_Pin
- added JP7, JP8: Jumper_2_Small_Open, Jumper:SolderJumper-2_P1.3mm_Open_RoundedPad1.0x1.5mm, symbol Jumper:Jumper_2_Small_Open
- added R15, R18: 1k, Resistor_SMD:R_0603_1608Metric, symbol Device:R
- added R16, R17, R19, R20, R21: 4.7k, Resistor_SMD:R_0603_1608Metric, symbol Device:R
- added U7: ~, Package_DFN_QFN:DFN-6-1EP_3x3mm_P1mm_EP1.5x2.4mm, symbol SHT25:SHT25
- added U8: MPL3115A2, MPL3115A2:PSON125P300X500X120-8N, symbol MPL3115A2:MPL3115A2
Connections:
- net 3v3: now also JP7.2 (B), JP8.2 (B), R21.2
- net DAVIS 7852: now also J22.4 (Pin_4)
- net DS18B20: now also J21.2 (Pin_2), R21.1
- net GND: now also C22.2, C23.2, C25.2, C26.2, D4.1 (K), D6.1 (K), U7.2 (VSS/GND), U8.3 (GND)
- net I2C SCL: now also J13.3 (Pin_3), J23.2 (Pin_2), R16.1, U7.6 (SCL), U8.8 (SCL)
- net I2C SDA: now also J13.2 (Pin_2), J23.3 (Pin_3), R17.1, R19.1, R20.1, U7.1 (SDA), U8.7 (SDL)
- net INSPEED VORTEX: now also J18.2 (Pin_2)
- net INSPEEED VANE: now also J10.2 (Pin_2)
- net S1223: now also J19.2 (Pin_2)
- net VH400: now also J20.2 (Pin_2)
- new net: C26.1, U8.2 (CAP)
- new net: D6.2 (A), R18.1
- new net: D4.2 (A), R15.1
- new net MPL power input: C23.1, C25.1, JP8.1 (A), R18.2, R19.2, R20.2, U8.1 (VDD), U8.4 (VDDIO)
- new net SHT25 power in: C22.1, JP7.1 (A), R15.2, R16.2, R17.2, U7.5 (VDD)
- no-connect marks 19 -> 21
Other:
- note added: "DAVIS 7852"
- note added: "DS18B20"
- note added: "INSPEED EVANE"
- note added: "INSPEED VORTEX"
- note added: "MPL3115ARI"
- note added: "S1223"
- note added: "SHT25"
- note added: "VH400"
- moved on the sheet: C10, C11, C12, C13, C14, C21, C5, C6, C7, C8, C9, D1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

Commit message: first pcb draft
Parts:
- J24: renamed from J9; footprint Connector_Phoenix_MC:PhoenixContact_MCV_1,5_2-GF-3.5_1x02_P3.50mm_Vertical_ThreadedFlange_MountHole -> Connector_Phoenix_MC:PhoenixContact_MC_1,5_2-GF-3.5_1x02_P3.50mm_Horizontal_ThreadedFlange_MountHole
- renumbered C11 to C1, C3 to C10, C5 to C11, C7 to C12, C6 to C13, C12 to C14, C26 to C15, C22 to C16, C23 to C19, C13 to C2, C25 to C20, C15 to C21, C20 to C22, C16 to C23, C21 to C24, C19 to C25, C10 to C3, C2 to C4, C14 to C5, C1 to C6, C9 to C7, C4 to C9, D3 to D1, D11 to D10, D6 to D11, D16 to D12, D15 to D13, D1 to D2, D14 to D3, D2 to D4, D10 to D6, D13 to D7, D4 to D8, D12 to D9, GSM2 to GSM1, GSM3 to GSM2, J4 to J1, J2 to J10, J5 to J11, J6 to J12, J7 to J13, J18 to J14, J19 to J15, J22 to J16, J23 to J17, J24 to J18, J1 to J19, J17 to J2, J13 to J20, J10 to J21, J20 to J22, J21 to J23, J16 to J3, J8 to J4, J11 to J5, J12 to J6, J14 to J7, J15 to J8, J3 to J9, JP7 to JP3, JP3 to JP4, JP8 to JP5, JP5 to JP6, JP6 to JP7, JP4 to JP8, Q2 to Q1, Q1 to Q2, Q6 to Q3, R13 to R1, R5 to R10, R3 to R11, R10 to R12, R11 to R13, R12 to R14, R28 to R15, R15 to R16, R20 to R17, R19 to R18, R35 to R19, R8 to R2, R34 to R20, R17 to R21, R27 to R22, R31 to R23, R36 to R24, R37 to R25, R16 to R26, R18 to R27, R38 to R28, R30 to R29, R6 to R3, R33 to R30, R39 to R31, R40 to R32, R14 to R33, R32 to R34, R21 to R35, R41 to R36, R9 to R4, R7 to R5, R1 to R6, R29 to R7, R4 to R8, R2 to R9, SW4 to SW3, SW3 to SW4, U6 to U1, U4 to U3, U8 to U4, U7 to U5, U1 to U6, U3 to U7, U5 to U8
Connections:
- net power in is gone; now on net ESP32 power in: R10.1, R8.1
- net I2C SCL: now also R17.1
- net I2C SDA: no longer R17.1
- net rx: no longer U1.3 (A2), U3.10 (RXD)
- net tx: no longer U1.1 (A1), U3.9 (TXD)
- net gsm power key: now reaches R3.1
- net gsm power key: now also U2.26 (IO4)
- net gsm reset: now reaches U2.5 (SENSOR_VN)
- net gsm reset: now also R2.1
- new net gsm rx: U1.3 (A2), U3.10 (RXD)
- new net gsm tx: U1.1 (A1), U3.9 (TXD)
Other:
- note added: "ESP 32 MICROCONTROLLER"
- note added: "GSM COMMUNICATION"
- note added: "LORA COMMUNICATION"
- note added: "MEMORY CARD"
- note added: "MEMS PRESSURE SENSOR"
- note added: "REAL TIME CLOCK"
- note added: "RS485 COMMUNICATION"
- note added: "SENSOR CONNECTORS"
- note added: "TEMPERATURE AND HUMIDITY SENSOR"
- note added: "boot option straping pin refenced from datasheet"
- note added: "level shifter"
- note added: "power indication led, optional, placed for block debugging"
- note added: "programming connector, input power scheme covered in power board"
- note added: "reset shcematic refernced from resources"
- company: (none) -> AdeMNEA IoT-ra
- title: (none) -> GATEWAY BOARD
- moved on the sheet: BT1, C1, C10, C11, C12, C13, C14, C15, C16, C17, C18, C19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

Commit message: finalised power schematic
Parts:
- removed J17: Conn_01x03_Pin, Connector_Phoenix_MC:PhoenixContact_MC_1,5_3-GF-3.81_1x03_P3.81mm_Horizontal_ThreadedFlange_MountHole, symbol Connector:Conn_01x03_Pin
- added J17: Conn_01x04_Pin, Connector_Phoenix_MC:PhoenixContact_MC_1,5_4-GF-3.5_1x04_P3.50mm_Horizontal_ThreadedFlange_MountHole, symbol Connector:Conn_01x04_Pin
- C15, C16, C19, C20, JP3, JP5, R17, R18, R21, R26, U4, U5: now not fitted
Connections:
- net I2C SCL: now also J17.2 (Pin_2)
- net I2C SDA: now also J17.3 (Pin_3)
Changed lines of the file:
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@@
 	(text "MPL3115ARI"
 		(exclude_from_sim no)
-		(at 474.472 236.982 0)
+		(at 477.012 234.95 0)
 		(effects
 			(font
@@
 		)
 	)
-	(text_box "ESD protection to be added in future design, communication default set to \nI2C, module set specifically for storing data, and hence transfer speeds are slow"
+	(text_box "ESD protection to be added in future design, communication default set to \nSPI, module set specifically for storing data, and hence transfer speeds are slow"
 		(exclude_from_sim no)
 		(at 436.88 193.04 0)
@@
 	(wire
 		(pts
-			(xy 454.66 241.3) (xy 466.09 241.3)
-		)
-		(stroke
-			(width 0)
-			(type default)
-		)
-	)
-	(wire
-		(pts
 			(xy 125.73 290.83) (xy 147.32 290.83)
 		)
@@
 	(wire
 		(pts
-			(xy 454.66 243.84) (xy 466.09 243.84)
-		)
-		(stroke
-			(width 0)
-			(type default)
-		)
-	)
-	(wire
-		(pts
 			(xy 297.18 298.45) (xy 307.34 298.45)
 		)
@@
 	(wire
 		(pts
+			(xy 454.66 237.49) (xy 464.82 237.49)
+		)
+		(stroke
+			(width 0)
+			(type default)
+		)
+	)
+	(wire
+		(pts
 			(xy 494.03 177.8) (xy 494.03 181.61)
 		)
@@
 	(wire
 		(pts
+			(xy 454.66 240.03) (xy 464.82 240.03)
+		)
+		(stroke
+			(width 0)
+			(type default)
+		)
+	)
+	(wire
+		(pts
 			(xy 288.29 248.92) (xy 288.29 251.46)
 		)
@@
 		)
 	)
-	(label "I2C SCL"
-		(at 454.66 241.3 0)
-		(effects
-			(font
-				(size 1.27 1.27)
-			)
-			(justify left bottom)
-		)
-	)
 	(label "strap12"
 		(at 135.89 280.67 0)
@@
 		)
 	)
+	(label "I2C SCL"
+		(at 454.66 240.03 0)
+		(effects
+			(font
+				(size 1.27 1.27)
+			)
+			(justify left bottom)
+		)
+	)
 	(label "SIM RST"
 		(at 220.98 171.45 0)
@@
 		)
 	)
-	(label "I2C SDA"
-		(at 454.66 243.84 0)
-		(effects
-			(font
-				(size 1.27 1.27)
-			)
-			(justify left bottom)
-		)
-	)
 	(label "lora power in"
 		(at 359.41 88.9 0)
@@
 		)
 	)
+	(label "I2C SDA"
+		(at 454.66 237.49 0)
+		(effects
+			(font
+				(size 1.27 1.27)
+			)
+			(justify left bottom)
+		)
+	)
 	(label "RI"
 		(at 91.44 72.39 0)
@@
 		(in_bom yes)
 		(on_board yes)
-		(dnp no)
+		(dnp yes)
 		(property "Reference" "R21"
 			(at 322.58 227.838 0)
@@
 		(in_bom yes)
 		(on_board yes)
-		(dnp no)
+		(dnp yes)
 		(fields_autoplaced yes)
 		(property "Reference" "#PWR037"
@@
 		(in_bom yes)
 		(on_board yes)
-		(dnp no)
+		(dnp yes)
 		(property "Reference" "C15"
 			(at 292.354 176.022 0)
@@
 		(in_bom yes)
 		(on_board yes)
-		(dnp no)
+		(dnp yes)
 		(property "Reference" "JP5"
 			(at 360.172 156.21 0)
@@
 		(in_bom yes)
 		(on_board yes)
-		(dnp no)
+		(dnp yes)
 		(fields_autoplaced yes)
 		(property "Reference" "U4"
@@
 		(in_bom yes)
 		(on_board yes)
-		(dnp no)
+		(dnp yes)
 		(property "Reference" "JP3"
 			(at 306.832 233.68 0)
@@
 		(in_bom yes)
 		(on_board yes)
-		(dnp no)
+		(dnp yes)
 		(fields_autoplaced yes)
 		(property "Reference" "R18"
@@
 		(in_bom yes)
 		(on_board yes)
-		(dnp no)
+		(dnp yes)
 		(fields_autoplaced yes)
 		(property "Reference" "#PWR027"
@@
 	)
 	(symbol
+		(lib_id "Connector:Conn_01x04_Pin")
+		(at 469.9 240.03 180)
+		(unit 1)
+		(exclude_from_sim no)
+		(in_bom yes)
+		(on_board yes)
+		(dnp no)
+		(fields_autoplaced yes)
+		(property "Reference" "J17"
+			(at 471.17 237.4899 0)
+			(effects
+				(font
+					(size 1.27 1.27)
+				)
+				(justify right)
+			)
+		)
+		(property "Value" "Conn_01x04_Pin"
+			(at 471.17 240.0299 0)
+			(effects
+				(font
+					(size 1.27 1.27)
+				)
+				(justify right)
+				(hide yes)
+			)
+		)
+		(property "Footprint" "Connector_Phoenix_MC:PhoenixContact_MC_1,5_4-GF-3.5_1x04_P3.50mm_Horizontal_ThreadedFlange_MountHole"
+			(at 469.9 240.03 0)
+			(effects
+				(font
+					(size 1.27 1.27)
+				)
+				(hide yes)
+			)
+		)
+		(property "Datasheet" "~"
+			(at 469.9 240.03 0)
+			(effects
+				(font
+					(size 1.27 1.27)
+				)
+				(hide yes)
+			)
+		)
+		(property "Description" "Generic connector, single row, 01x04, script generated"
+			(at 469.9 240.03 0)
+			(effects
+				(font
+					(size 1.27 1.27)
+				)
+				(hide yes)
+			)
+		)
+		(pin "1"
+		)
+		(pin "4"
+		)
+		(pin "2"
+		)
+		(pin "3"
+		)
+		(instances
+			(project "AWS PROJECT"
+				(path "/28dd5718-f0db-4cd1-9b2d-c2f5533a75a3/918a84d0-2382-4e9e-a083-abfab5a808df"
+					(reference "J17")
+					(unit 1)
+				)
+			)
+		)
+	)
+	(symbol
 		(lib_id "Jumper:Jumper_2_Small_Open")
 		(at 163.83 260.35 90)
@@
 	)
 	(symbol
-		(lib_id "Connector:Conn_01x03_Pin")
-		(at 471.17 241.3 0)
-		(mirror y)
-		(unit 1)
-		(exclude_from_sim no)
-		(in_bom yes)
-		(on_board yes)
-		(dnp no)
-		(fields_autoplaced yes)
-		(property "Reference" "J17"
-			(at 470.535 233.68 0)
-			(effects
-				(font
-					(size 1.27 1.27)
-				)
-			)
-		)
-		(property "Value" "Conn_01x03_Pin"
-			(at 470.535 236.22 0)
-			(effects
-				(font
-					(size 1.27 1.27)
-				)
-				(hide yes)
-			)
-		)
-		(property "Footprint" "Connector_Phoenix_MC:PhoenixContact_MC_1,5_3-GF-3.81_1x03_P3.81mm_Horizontal_ThreadedFlange_MountHole"
-			(at 471.17 241.3 0)
-			(effects
-				(font
-					(size 1.27 1.27)
-				)
-				(hide yes)
-			)
-		)
-		(property "Datasheet" "~"
-			(at 471.17 241.3 0)
-			(effects
-				(font
-					(size 1.27 1.27)
-				)
-				(hide yes)
-			)
-		)
-		(property "Description" "Generic connector, single row, 01x03, script generated"
-			(at 471.17 241.3 0)
-			(effects
-				(font
-					(size 1.27 1.27)
-				)
-				(hide yes)
-			)
-		)
-		(pin "2"
-		)
-		(pin "1"
-		)
-		(pin "3"
-		)
-		(instances
-			(project "AWS PROJECT"
-				(path "/28dd5718-f0db-4cd1-9b2d-c2f5533a75a3/918a84d0-2382-4e9e-a083-abfab5a808df"
-					(reference "J17")
-					(unit 1)
-				)
-			)
-		)
-	)
-	(symbol
 		(lib_id "Device:C_Small")
 		(at 40.64 104.14 0)
@@
 		(in_bom yes)
 		(on_board yes)
-		(dnp no)
+		(dnp yes)
 		(property "Reference" "C16"
 			(at 305.054 238.252 0)
@@
 		(in_bom yes)
 		(on_board yes)
-		(dnp no)
+		(dnp yes)
 		(property "Reference" "R17"
 			(at 284.988 153.924 0)
@@
 					(size 1.27 1.27)
 				)
+				(hide yes)
 			)
 		)
@@
 		(in_bom yes)
 		(on_board yes)
-		(dnp no)
+		(dnp yes)
 		(fields_autoplaced yes)
 		(property "Reference" "U5"
@@
 		(in_bom yes)
 		(on_board yes)
-		(dnp no)
+		(dnp yes)
 		(fields_autoplaced yes)
 		(property "Reference" "C20"
@@
 		(in_bom yes)
 		(on_board yes)
-		(dnp no)
+		(dnp yes)
 		(fields_autoplaced yes)
 		(property "Reference" "R26"
@@
 		(in_bom yes)
 		(on_board yes)
-		(dnp no)
+		(dnp yes)
 		(fields_autoplaced yes)
 		(property "Reference" "#PWR033"
@@
 		(in_bom yes)
 		(on_board yes)
-		(dnp no)
+		(dnp yes)
 		(property "Reference" "C19"
 			(at 348.234 164.592 0)

Commit message: algorirthim design start
Parts:
- removed J14, J15: Conn_01x02_Pin, Connector_Phoenix_MC:PhoenixContact_MC_1,5_2-GF-3.5_1x02_P3.50mm_Horizontal_ThreadedFlange_MountHole, symbol Connector:Conn_01x02_Pin
- removed J16, J17, J20: Conn_01x04_Pin, Connector_Phoenix_MC:PhoenixContact_MC_1,5_4-GF-3.5_1x04_P3.50mm_Horizontal_ThreadedFlange_MountHole, symbol Connector:Conn_01x04_Pin
- removed J18, J21, J22, J23: Conn_01x03_Pin, Connector_Phoenix_MC:PhoenixContact_MC_1,5_3-GF-3.81_1x03_P3.81mm_Horizontal_ThreadedFlange_MountHole, symbol Connector:Conn_01x03_Pin
- removed J24: Screw_Terminal_01x02, Connector_Phoenix_MC:PhoenixContact_MC_1,5_2-GF-3.5_1x02_P3.50mm_Horizontal_ThreadedFlange_MountHole, symbol Connector:Screw_Terminal_01x02
- removed R8: 10k, Resistor_SMD:R_0603_1608Metric, symbol Device:R
- added C38, C40: 0.1uF, Capacitor_SMD:C_0603_1608Metric, symbol Device:C_Small
- added C39: 4.7uF, Capacitor_SMD:C_0603_1608Metric, symbol Device:C_Small
- added C41: 10uF, Capacitor_SMD:C_0603_1608Metric, symbol Device:C_Small
- added C42: 1uF, Capacitor_SMD:C_0603_1608Metric, symbol Device:C_Small
- added D17, D18: NET_LED, Diode_SMD:D_0603_1608Metric, symbol Device:LED
- added FB2: FerriteBead_Small, BLM03HG601SZ1D:BEADC0603X33N, symbol Device:FerriteBead_Small
- added J14, J15, J24, J29: B2B-XH-A_LF__SN_, B2B-XH-A_LF__SN_:JST_B2B-XH-A_LF__SN_, symbol B2B-XH-A_LF__SN_:B2B-XH-A_LF__SN_
- added J16, J17, J18, J23, J28: B4B-XH-A_LF__SN_, B4B-XH-A_LF__SN_:JST_B4B-XH-A_LF__SN_, symbol B4B-XH-A_LF__SN_:B4B-XH-A_LF__SN_
- added J20, J21, J32, J37: B3B-XH-A_LF__SN_, B3B-XH-A_LF__SN_:JST_B3B-XH-A_LF__SN_, symbol B3B-XH-A_LF__SN_:B3B-XH-A_LF__SN_
- added J31: TYPE-C-31-M-12, TYPE-C-31-M-12:HRO_TYPE-C-31-M-12, symbol TYPE-C-31-M-12:TYPE-C-31-M-12
- added JP14, JP16, JP17: Jumper_2_Small_Open, Jumper:SolderJumper-2_P1.3mm_Open_RoundedPad1.0x1.5mm, symbol Jumper:Jumper_2_Small_Open
- added R50, R51: 270R, Resistor_SMD:R_0603_1608Metric, symbol Device:R
- added R52, R53: 5.1k, Resistor_SMD:R_0603_1608Metric, symbol Device:R
- added SNS_TX2, SNS_TX3, SNS_TX4, SNS_TX5, SNS_TX6: TestPoint, TestPoint:TestPoint_Pad_D1.5mm, symbol Connector:TestPoint
- added U14: AMS1117-3.3, Package_TO_SOT_SMD:SOT-223-3_TabPin2, symbol Regulator_Linear:AMS1117-3.3
- added U9: FT232RL-REEL, FT232RL-REEL:SOP65P780X200-28N, symbol FT232RL-REEL:FT232RL-REEL
- U2: footprint ESP32-WROOM-32E__4MB_HIGH_TEMP_:XCVR_ESP32-WROOM-32E__4MB_HIGH_TEMP_ -> ESP32-WROOM-32UE_M113EH6400UH3Q0_:MODULE_ESP32-WROOM-32UE_M113EH6400UH3Q0_
Connections:
- net 3v3: now also J17.1, J18.3, J28.1, JP17.2 (B); no longer J9.4 (Pin_4), R35.2
- net DAVIS 7852: now also J16.1
- net DS18B20: now also J21.2
- net GND: now also C38.2, C39.2, C40.2, C41.2, C42.2, J14.2, J15.2, J16.2, J16.3, J16.4, J17.4, J18.2, J18.4, J20.3, J21.3, J28.4, J31.A1_B12 (GND), J31.B1_A12 (GND), J31.S1 (SHIELD), J31.S2 (SHIELD), J31.S3 (SHIELD), J31.S4 (SHIELD), J32.3, J37.3, JP14.2 (B), R52.1, R53.1, U14.1 (GND), U9.18 (GND), U9.21 (GND), U9.25 (AGND), U9.26 (TEST), U9.7 (GND)
- net I2C SCL: now also J2.2 (Pin_2), U2.36 (IO22), J17.2, J28.3, J29.1; no longer J2.1 (Pin_1), U2.33 (IO21)
- net I2C SDA: now also J2.1 (Pin_1), U2.33 (IO21), J17.3, J28.2, J29.2; no longer J2.2 (Pin_2), U2.36 (IO22)
- net INSPEED VORTEX: now also J14.1
- net INSPEEED VANE: now also J37.2
- net S1223: now also J15.1
- net VBUS: now also FB2.1, J31.A4_B9 (VBUS), J31.B4_A9 (VBUS)
- net VH400: now also J20.2
- net VSPI-CLK: now also J23.2
- net VSPI-MISO: now also J23.3
- net VSPI-MOSI: now also J23.4
- net rx: now also U9.1 (TXD)
- net strap 5: now also J23.1; no longer U2.29 (IO5)
- net tx: now also U9.5 (RXD)
- net at R36.1, U8.7 (B): now also J24.2
- net at R36.2, U8.6 (A): now also J24.1
- net at U7.2 (IO8): now also SNS_TX6.1
- net at U7.3 (IO11): now also SNS_TX5.1
- net at U7.4 (IO9): now also SNS_TX4.1
- net at U7.5 (IO4): now also SNS_TX3.1
- net at U7.6 (IO5): now also SNS_TX2.1
- new net: C42.1, JP17.1 (A), U14.2 (VO)
- new net: C38.1, C39.1, FB2.2, JP16.1 (A), U9.20 (VCC), U9.4 (VCCIO)
- new net: D17.1 (K), U9.23 (CBUS0)
- new net: D17.2 (A), R50.1
- new net: J31.B5 (CC2), R53.2
- new net: D18.1 (K), U9.22 (CBUS1)
- new net: D18.2 (A), R51.1
- new net: J31.A5 (CC1), R52.2
- new net: C40.1, U9.17 (3V3OUT)
- new net: JP14.1 (A), U9.19 (~{RESET})
- new net 5v: J18.1, J20.1, J21.1, J32.1, J37.1, R35.2
- new net DHT22: J32.2, U2.29 (IO5)
- new net USBD+: J31.A6 (DP1), J31.B6 (DP2), U9.15 (USBDP)
- new net USBD-: J31.A7 (DN1), J31.B7 (DN2), U9.16 (USBDM)
- new net VCC: C41.1, J9.4 (Pin_4), JP16.2 (B), R50.2, R51.2, U14.3 (VI)
- no-connect marks 21 -> 50
Other:
- moved on the sheet: BT1, C1, C10, C11, C12, C13, C14, C15, C16, C17, C18, C19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
