File: KiCAD FILES/gateway.kicad_sch (KiCad schematic)
At the start: 176 parts, among them J1 Conn_01x02_Pin, J10 SIM7100-8-1-15-00-A_REVC, J12 Conn_01x02_Pin, J13 Conn_01x02_Pin, J14 B2B-XH-A_LF__SN_, J15 B2B-XH-A_LF__SN_, J17 B4B-XH-A_LF__SN_, J18 B4B-XH-A_LF__SN_, J19 MEM2067-02-180-00-A_REVB, J2 Conn_01x02_Pin, J20 B3B-XH-A_LF__SN_, J21 B3B-XH-A_LF__SN_, J24 B2B-XH-A_LF__SN_, J28 B4B-XH-A_LF__SN_, J29 B2B-XH-A_LF__SN_, J3 B3B-XH-A_LF__SN_, J31 TYPE-C-31-M-12, J32 B3B-XH-A_LF__SN_, J35 Conn_01x02_Pin, J37 B3B-XH-A_LF__SN_, J38 Conn_01x02_Pin, J39 Conn_01x02_Pin, J40 Conn_01x06_Pin, J9 Conn_01x04_Pin, Q1 MMBT3904, Q2 MMBT3904, Q3 MMBT3904, U1 TXB0108RGYR, U11 AMS1117-3.3, U14 AMS1117-3.3, U16 AMS1117-3.3, U18 AMS1117-3.3, U2 ESP32-WROOM-32E__4MB_HIGH_TEM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, U3 SIM7000E, U4 MPL3115A2, U6 DS3231MZ_TRL, U7 Ai-Thinker RA-08H, U8 ST3485EBDR, U9 FT232RL-REEL

Commit message: edits to the boards, got lcsc part numbers for bom, swapped unavailable components, fixed net label confilcts
Parts:
- removed J10: SIM7100-8-1-15-00-A_REVC, SIM7100-8-1-15-00-A_REVC:GCT_SIM7100-8-1-15-00-A_REVC, symbol SIM7100-8-1-15-00-A_REVC:SIM7100-8-1-15-00-A_REVC
- removed J19: MEM2067-02-180-00-A_REVB, MEM2067-02-180-00-A_REVB:GCT_MEM2067-02-180-00-A_REVB, symbol MEM2067-02-180-00-A_REVB:MEM2067-02-180-00-A_REVB
- added J16: 503398-1892, 503398-1892:MOLEX_503398-1892, symbol 503398-1892:503398-1892
- added J7: 104224-0820, 104224-0820:MOLEX_104224-0820, symbol 104224-0820:104224-0820
- added SNS_TX20, SNS_TX8: TestPoint, TestPoint:TestPoint_Pad_D1.5mm, symbol Connector:TestPoint
- BT1: LCSC (none) -> C6868959
- C1: renamed from C76; LCSC (none) -> C19702
- C11: renamed from C7; LCSC (none) -> C14663
- C12: renamed from C8; LCSC (none) -> C14663
- C13: renamed from C9; LCSC (none) -> C14663
- C14: renamed from C10; LCSC (none) -> C12891
- C15: renamed from C11; LCSC (none) -> C14663
- C16: renamed from C12; LCSC (none) -> C15849
- C17: renamed from C13; LCSC (none) -> C15008
- C18: renamed from C14; LCSC (none) -> C14663
- C19: renamed from C15; LCSC (none) -> C14663
- C2: renamed from C1; LCSC (none) -> C14663
- C20: renamed from C16; LCSC (none) -> C14663
- C23: renamed from C19; LCSC (none) -> C14663
- C24: renamed from C20; LCSC (none) -> C89632
- C25: renamed from C21; LCSC (none) -> C89632
- C26: renamed from C22; LCSC (none) -> C14663
- C27: renamed from C23; LCSC (none) -> C14663
- C28: renamed from C24; LCSC (none) -> C14663
- C29: renamed from C25; LCSC (none) -> C15849
- C3: renamed from C47; LCSC (none) -> C19702
- C30: renamed from C51; LCSC (none) -> C19702
- C31: renamed from C67; LCSC (none) -> C15849
- C32: renamed from C39; LCSC (none) -> C1705
- C33: renamed from C38; LCSC (none) -> C14663
- C34: renamed from C40; LCSC (none) -> C14663
- C35: renamed from C41; LCSC (none) -> C19702
- C36: renamed from C42; LCSC (none) -> C15849
- C4: LCSC (none) -> C14663
- C6: renamed from C3; LCSC (none) -> C14663
- C7: renamed from C78; LCSC (none) -> C15849
- C8: renamed from C6; LCSC (none) -> C15849
- C9: renamed from C49; LCSC (none) -> C15849
- D1: renamed from D21; LCSC (none) -> C191023
- D11: renamed from D9; LCSC (none) -> C22371297
- D13: renamed from D12; LCSC (none) -> C22371297
- D14: renamed from D13; LCSC (none) -> C22371297
- D15: renamed from D25; LCSC (none) -> C191023
- D16: renamed from D20; LCSC (none) -> C191023
- D17, D18: LCSC (none) -> C22371297
- D2: renamed from D24; LCSC (none) -> C191023
- D5: renamed from D3; LCSC (none) -> C22371297
- D6: renamed from D5; LCSC (none) -> C48677
- D8: renamed from D6; LCSC (none) -> C22371297
- D9: renamed from D7; LCSC (none) -> C22371297
- FB1: LCSC (none) -> C3764553
- GSM1, GSM2: LCSC (none) -> C434808
- J1: renamed from J35; now left out of the parts list
- J10: renamed from J12; now left out of the parts list
- J11: renamed from J28; now left out of the parts list
- J12: renamed from J3; now left out of the parts list
- J13: renamed from J14; now left out of the parts list
- J14: renamed from J15; now left out of the parts list
- J15: renamed from J18; now left out of the parts list
- J17: now left out of the parts list
- J18: renamed from J37; now left out of the parts list
- J19: renamed from J20; now left out of the parts list
- J2: renamed from J38; now left out of the parts list
- J20: renamed from J21; now left out of the parts list
- J21: renamed from J24; now left out of the parts list
- J22: renamed from J32; now left out of the parts list
- J23: renamed from J29; now left out of the parts list
- J24: renamed from J31; LCSC (none) -> C165948
- J3: renamed from J1; now left out of the parts list
- J4: renamed from J2; now left out of the parts list
- J5: renamed from J9; now left out of the parts list
- J6: renamed from J40; now left out of the parts list
- J8: renamed from J39; now left out of the parts list
- J9: renamed from J13; now left out of the parts list
- JP1: renamed from JP24; now left out of the parts list
- JP10: renamed from JP6; now left out of the parts list
- JP11: renamed from JP7; now left out of the parts list
- JP12: renamed from JP8; now left out of the parts list
- JP13: renamed from JP22; now left out of the parts list
- JP14: renamed from JP23; now left out of the parts list
- JP15: renamed from JP16; now left out of the parts list
- JP16: renamed from JP17; now left out of the parts list
- JP17: renamed from JP14; now left out of the parts list
- JP2: renamed from JP10; now left out of the parts list
- JP3: renamed from JP25; now left out of the parts list
- JP4: renamed from JP15; now left out of the parts list
- JP5: renamed from JP1; now left out of the parts list
- JP6: renamed from JP2; now left out of the parts list
- JP7: renamed from JP3; now left out of the parts list
- JP8: renamed from JP4; now left out of the parts list
- JP9: renamed from JP5; now left out of the parts list
- Q1, Q2, Q3: LCSC (none) -> C242260
- R1: LCSC (none) -> C95177
- R10: renamed from R9; LCSC (none) -> C98220
- R12: renamed from R11; LCSC (none) -> C98220
- R13: renamed from R12; LCSC (none) -> C99782
- R14: renamed from R13; LCSC (none) -> C99782
- R15: renamed from R14; LCSC (none) -> C22548
- R16: renamed from R15; LCSC (none) -> C22548
- R2, R3: LCSC (none) -> C99782
- R20: renamed from R19; LCSC (none) -> C99782
- R21: renamed from R20; LCSC (none) -> C99782
- R23: renamed from R22; LCSC (none) -> C22548
- R24: renamed from R23; LCSC (none) -> C95177
- R25: renamed from R24; LCSC (none) -> C99782
- R26: renamed from R25; LCSC (none) -> C99782
- R29: renamed from R28; LCSC (none) -> C22548
- R30: renamed from R29; LCSC (none) -> C98220
- R31: renamed from R30; LCSC (none) -> C22548
- R32: renamed from R61; LCSC (none) -> C99782
- R33: renamed from R55; LCSC (none) -> C99782
- R34: renamed from R8; LCSC (none) -> C98220
- R35: renamed from R34; LCSC (none) -> C22548
- R36: renamed from R63; LCSC (none) -> C105575
- R37: renamed from R62; LCSC (none) -> C98220
- R38: renamed from R35; LCSC (none) -> C99782
- R39: renamed from R36; LCSC (none) -> C22787
- R4: renamed from R6; LCSC (none) -> C98220
- R40: renamed from R52; LCSC (none) -> C2907044
- R41: renamed from R53; LCSC (none) -> C2907044
- R42: renamed from R50; LCSC (none) -> C2907020
- R43: renamed from R51; LCSC (none) -> C2907020
- R5: renamed from R4; LCSC (none) -> C99782
- R6: renamed from R5; LCSC (none) -> C99782
- R7: renamed from R54; LCSC (none) -> C99782
- R8: renamed from R38; LCSC (none) -> C99782
- R9: renamed from R7; LCSC (none) -> C22548
- U1: renamed from U18; LCSC (none) -> C6186
- U10: renamed from U16; LCSC (none) -> C6186
- U11: renamed from U8; LCSC (none) -> C75809
- U12: renamed from U14; LCSC (none) -> C6186
- U13: renamed from U9; LCSC (none) -> C8690
- U2: renamed from U11; LCSC (none) -> C6186
- U3: renamed from U1; LCSC (none) -> C194701
- U4: renamed from U2; LCSC (none) -> C701344
- U5: renamed from U3; LCSC (none) -> C126272
- U8: renamed from U6; LCSC (none) -> C107410
- U9: renamed from U7; LCSC (none) -> C2991932
- renumbered C5 to C10, C17 to C21, C18 to C22, C2 to C5, D8 to D10, D11 to D12, D1 to D3, D2 to D4, D4 to D7, R10 to R11, R16 to R17, R17 to R18, R18 to R19, R21 to R22, R26 to R27, R27 to R28, SNS_TX9 to SNS_TX10, SNS_TX8 to SNS_TX11, SNS_TX11 to SNS_TX12, SNS_TX12 to SNS_TX13, SNS_TX6 to SNS_TX14, SNS_TX5 to SNS_TX15, SNS_TX4 to SNS_TX16, SNS_TX3 to SNS_TX17, SNS_TX2 to SNS_TX18, SNS_TX7 to SNS_TX19, SNS_TX13 to SNS_TX2, SNS_TX16 to SNS_TX3, SNS_TX17 to SNS_TX4, SNS_TX18 to SNS_TX5, SNS_TX14 to SNS_TX6, SNS_TX15 to SNS_TX7, SNS_TX10 to SNS_TX9, U4 to U6, U5 to U7
Connections:
- net GND: now also J16.6 (VSS), J16.9 (VSS), J16.P1 (SHIELD), J16.P2 (SHIELD), J16.P3 (SHIELD), J16.P4 (SHIELD), J7.G1 (GND), J7.G2 (GND), J7.G3 (GND), J7.G4 (GND), J7.S4 (GND)
- net SD CS: now also J16.2 (CD/DAT3^2)
- net SD power in: now also J16.4 (VDD)
- net SIM CLK: now also D6.1, J7.S3 (CLK); no longer D6.3
- net SIM DATA: now also D6.3, J7.S6 (I/O); no longer D6.1
- net SIM DET: now also SNS_TX8.1
- net SIM RST: now also D6.4, J7.S2 (RST); no longer D6.5
- net SIM VDD: now also D6.5, J7.S1 (VCC); no longer D6.4
- net VSPI-CLK: now also J16.5 (CLK)
- net VSPI-MISO: now also J16.7 (DAT0)
- net VSPI-MOSI: now also J16.3 (CMD)
- new net: J16.10 (DETECT_SWITCH), SNS_TX20.1
- no-connect marks 51 -> 50
Other:
- moved on the sheet: C18, D6
