File: KiCAD FILES/gateway.kicad_sch (KiCad schematic)
At the start: 173 parts, among them J1 Conn_01x02_Pin, J10 SIM7100-8-1-15-00-A_REVC, J12 Conn_01x02_Pin, J13 Conn_01x02_Pin, J14 B2B-XH-A_LF__SN_, J15 B2B-XH-A_LF__SN_, J17 B4B-XH-A_LF__SN_, J18 B4B-XH-A_LF__SN_, J19 MEM2067-02-180-00-A_REVB, J2 Conn_01x02_Pin, J20 B3B-XH-A_LF__SN_, J21 B3B-XH-A_LF__SN_, J24 B2B-XH-A_LF__SN_, J28 B4B-XH-A_LF__SN_, J29 B2B-XH-A_LF__SN_, J3 B3B-XH-A_LF__SN_, J31 TYPE-C-31-M-12, J32 B3B-XH-A_LF__SN_, J35 Conn_01x02_Pin, J37 B3B-XH-A_LF__SN_, J38 Conn_01x02_Pin, J39 Conn_01x02_Pin, J40 Conn_01x06_Pin, J9 Conn_01x04_Pin, Q1 MMBT3904, Q2 MMBT3904, Q3 MMBT3904, U1 TXB0108RGYR, U11 AMS1117-3.3, U14 AMS1117-3.3, U16 AMS1117-3.3, U18 AMS1117-3.3, U2 ESP32-WROOM-32E__4MB_HIGH_TEM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, U3 SIM7000E, U4 MPL3115A2, U6 DS3231MZ_TRL, U7 Ai-Thinker RA-08H, U8 ST3485EBDR, U9 FT232RL-REEL

Commit message: Merge branch 'main' of https://github.com/marydovika/AWS
Parts:
- renumbered BT1 to BT?, C2 to C?, C51 to C?, C47 to C?, C14 to C?, C15 to C?, C38 to C?, C76 to C?, C5 to C?, C9 to C?, C67 to C?, C8 to C?, C13 to C?, C22 to C?, C1 to C?, C39 to C?, C17 to C?, C21 to C?, C12 to C?, C3 to C?, C16 to C?, C49 to C?, C7 to C?, C41 to C?, C23 to C?, C42 to C?, C18 to C?, C24 to C?, C40 to C?, C20 to C?, C6 to C?, C78 to C?, C19 to C?, C10 to C?, C25 to C?, C4 to C?, C11 to C?, D11 to D?, D1 to D?, D17 to D?, D9 to D?, D8 to D?, D6 to D?, D3 to D?, D5 to D?, D21 to D?, D7 to D?, D2 to D?, D25 to D?, D18 to D?, D4 to D?, D13 to D?, D24 to D?, D12 to D?, D20 to D?, FB1 to FB?, GSM2 to GSM?, GSM1 to GSM?, J29 to J?, J1 to J?, J9 to J?, J28 to J?, J12 to J?, J20 to J?, J17 to J?, J32 to J?, J18 to J?, J35 to J?, J40 to J?, J38 to J?, J3 to J?, J14 to J?, J15 to J?, J21 to J?, J10 to J?, J19 to J?, J37 to J?, J13 to J?, J31 to J?, J39 to J?, J2 to J?, J24 to J?, JP16 to JP?, JP25 to JP?, JP17 to JP?, JP5 to JP?, JP23 to JP?, JP24 to JP?, JP3 to JP?, JP22 to JP?, JP10 to JP?, JP1 to JP?, JP15 to JP?, JP7 to JP?, JP2 to JP?, JP4 to JP?, JP8 to JP?, JP6 to JP?, JP14 to JP?, Q2 to Q?, Q3 to Q?, Q1 to Q?, R34 to R?, R8 to R?, R36 to R?, R21 to R?, R11 to R?, R28 to R?, R13 to R?, R7 to R?, R62 to R?, R18 to R?, R16 to R?, R1 to R?, R20 to R?, R5 to R?, R12 to R?, R3 to R?, R14 to R?, R53 to R?, R50 to R?, R22 to R?, R24 to R?, R27 to R?, R63 to R?, R15 to R?, R25 to R?, R55 to R?, R9 to R?, R30 to R?, R2 to R?, R17 to R?, R4 to R?, R52 to R?, R54 to R?, R51 to R?, R19 to R?, R38 to R?, R26 to R?, R6 to R?, R35 to R?, R23 to R?, R10 to R?, R61 to R?, R29 to R?, SNS_TX7 to SNS_TX?, SNS_TX5 to SNS_TX?, SNS_TX4 to SNS_TX?, SNS_TX13 to SNS_TX?, SNS_TX11 to SNS_TX?, SNS_TX14 to SNS_TX?, SNS_TX12 to SNS_TX?, SNS_TX8 to SNS_TX?, SNS_TX10 to SNS_TX?, SNS_TX1 to SNS_TX?, SNS_TX6 to SNS_TX?, SNS_TX3 to SNS_TX?, SNS_TX2 to SNS_TX?, SNS_TX15 to SNS_TX?, SNS_TX9 to SNS_TX?, U14 to U?, U1 to U?, U7 to U?, U4 to U?, U3 to U?, U8 to U?, U6 to U?, U2 to U?, U11 to U?, U16 to U?, U18 to U?, U5 to U?, U9 to U?
Other:
- note added: "FTDI USB-Serial Interface IC"

Commit message: All previous PCBA edits
Parts:
- GSM1, GSM2: renamed from GSM?; DESCRIPTION U.FL Series 50 Ohm Receptacle Male Pins Ultra Small SMT Coa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 -> (none)
- U5: renamed from U?; value ~ -> (none)
- gave numbers to parts that had none: 170
