File: KiCAD FILES/power.kicad_sch (KiCad schematic)
At the start: 137 parts, among them J25 Screw_Terminal_01x02, J26 Screw_Terminal_01x02, J27 Screw_Terminal_01x02, J36 B4B-XH-A_LF__SN_, J4 B2B-XH-A_LF__SN_, J5 Conn_01x02_Pin, J6 Conn_01x02_Pin, J7 Conn_01x02_Pin, J8 Conn_01x02_Pin, Q12 2N7002, Q4 2N7002, Q5 NMOS, Q9 NMOS, SW5 SW_SPST, SW6 SW_SPST, U10 BQ24650RVAR, U12 TPS2121RUXR, U13 AP64501SP-13, U15 STM32F401CCU6, U17 AMS1117-3.3, Y1 C3E-25.000-12-3030-X-R

Commit message: edits to the boards, got lcsc part numbers for bom, swapped unavailable components, fixed net label confilcts
Parts:
- C37: renamed from C52; LCSC (none) -> C23630
- C38: renamed from C53; LCSC (none) -> C92670
- C39: renamed from C37; LCSC (none) -> C100042
- C40: renamed from C54; LCSC (none) -> C15849
- C41: renamed from C55; LCSC (none) -> C15849
- C42: renamed from C56; LCSC (none) -> C14663
- C43: renamed from C57; LCSC (none) -> C15849
- C44: renamed from C28; LCSC (none) -> C30110
- C45: renamed from C29; LCSC (none) -> C24497
- C46: renamed from C30; LCSC (none) -> C100042
- C47: renamed from C58; footprint Capacitor_SMD:C_1210_3225Metric_Pad1.33x2.70mm_HandSolder -> Capacitor_SMD:C_1206_3216Metric_Pad1.33x1.80mm_HandSolder; LCSC (none) -> C89632
- C48: renamed from C59; footprint Capacitor_SMD:C_1210_3225Metric_Pad1.33x2.70mm_HandSolder -> Capacitor_SMD:C_1206_3216Metric_Pad1.33x1.80mm_HandSolder; LCSC (none) -> C89632
- C49: renamed from C60; LCSC (none) -> C23630
- C50: renamed from C61; LCSC (none) -> C14663
- C51: renamed from C62; LCSC (none) -> C19702; now left out of the parts list
- C52: renamed from C31; footprint Capacitor_SMD:C_0201_0603Metric_Pad0.64x0.40mm_HandSolder -> Capacitor_SMD:C_0603_1608Metric_Pad1.08x0.95mm_HandSolder; now not fitted
- C53: renamed from C63; LCSC (none) -> C15849
- C54: renamed from C64; LCSC (none) -> C92670
- C55: renamed from C32; LCSC (none) -> C107085
- C56: renamed from C33; LCSC (none) -> C86295
- C57: renamed from C65; LCSC (none) -> C89632
- C58: renamed from C34; LCSC (none) -> C107047
- C59: renamed from C35; LCSC (none) -> C86295
- C60: renamed from C36; LCSC (none) -> C86295
- C61: renamed from C43; LCSC (none) -> C19702
- C62: renamed from C73; LCSC (none) -> C19702
- C63: renamed from C74; LCSC (none) -> C15849
- C64: renamed from C44; LCSC (none) -> C15849
- C73: renamed from C46; LCSC (none) -> C92670
- D19: renamed from D14; LCSC (none) -> C22371297
- D20: renamed from D15; LCSC (none) -> C22371297
- D21: renamed from D16; value D -> B540C-13-F; footprint Diode_SMD:D_1210_3225Metric -> Diode_SMD:D_SMB-SMC_Universal_Handsoldering; LCSC (none) -> C72264
- D23: value D -> B540C-13-F; footprint Diode_SMD:D_1210_3225Metric -> Diode_SMD:D_SMB-SMC_Universal_Handsoldering; LCSC (none) -> C72264
- J25, J26, J27, TP1: now left out of the parts list
- J28: renamed from J36; now left out of the parts list
- J29: renamed from J8; now left out of the parts list
- J30: renamed from J7; now left out of the parts list
- J31: renamed from J5; now left out of the parts list
- J32: renamed from J6; now left out of the parts list
- J33: renamed from J4; now left out of the parts list
- JP18: renamed from JP13; now left out of the parts list
- JP19: renamed from JP11; now left out of the parts list
- JP20: renamed from JP18; now left out of the parts list
- JP21: renamed from JP19; now left out of the parts list
- JP22: renamed from JP12; now left out of the parts list
- JP23: renamed from JP9; now left out of the parts list
- JP24: renamed from JP21; now left out of the parts list
- JP25: renamed from JP20; now left out of the parts list
- L1: renamed from L2; LCSC (none) -> C2454102
- L2: renamed from L1; LCSC (none) -> C3221229
- Q5: renamed from Q9; LCSC (none) -> C604579
- Q6: renamed from Q5; LCSC (none) -> C604579
- R44: renamed from R47; LCSC (none) -> C2930150
- R45: renamed from R48; LCSC (none) -> C2930150
- R46: renamed from R44; LCSC (none) -> C22912
- R47: renamed from R45; LCSC (none) -> C2828621
- R48: renamed from R42; LCSC (none) -> C22912
- R49: renamed from R43; LCSC (none) -> C2828621
- R50: renamed from R66; LCSC (none) -> C26751
- R51: renamed from R67; LCSC (none) -> C2930097
- R52: renamed from R68; LCSC (none) -> C2828637
- R53: renamed from R46; LCSC (none) -> C2933234
- R54: renamed from R69; LCSC (none) -> C98220
- R55: renamed from R70; LCSC (none) -> C98220
- R56: renamed from R71; LCSC (none) -> C2930111
- R57: renamed from R72; LCSC (none) -> C2930127
- R58: renamed from R73; LCSC (none) -> C109318
- R59: renamed from R74; LCSC (none) -> C105588
- R60: renamed from R75; LCSC (none) -> C22939
- R61: renamed from R76; LCSC (none) -> C2933875
- R62: renamed from R39; LCSC (none) -> C2907044
- R63: renamed from R40; LCSC (none) -> C2907044
- R64: renamed from R77; LCSC (none) -> C3009313
- R65: renamed from R41; LCSC (none) -> C2907044
- R66: renamed from R78; LCSC (none) -> C861677
- R67: renamed from R79; LCSC (none) -> C5126163
- R68: renamed from R80; LCSC (none) -> C2998114
- R69: renamed from R49; LCSC (none) -> C98220
- R70: renamed from R56; LCSC (none) -> C105575
- R71: renamed from R57; LCSC (none) -> C98220
- R72: renamed from R58; LCSC (none) -> C2906992
- R73: renamed from R59; LCSC (none) -> C98220
- R74: renamed from R60; LCSC (none) -> C22843
- R75: renamed from R64; LCSC (none) -> C98220
- R76: renamed from R65; LCSC (none) -> C22975
- R77: renamed from R81; LCSC (none) -> C98220
- R78: renamed from R82; LCSC (none) -> C2906976
- TH1: renamed from TH2; LCSC (none) -> C5146262
- U14: renamed from U10; LCSC (none) -> C53712
- U15: renamed from U12; LCSC (none) -> C485916
- U16: renamed from U13; LCSC (none) -> C2071517
- U17: LCSC (none) -> C6186
- U18: renamed from U15; LCSC (none) -> C79861
- Y1: LCSC (none) -> C5567192
- renumbered C68 to C65, C71 to C66, C26 to C67, C72 to C68, C27 to C69, C69 to C70, C70 to C71, C45 to C72, D19 to D24, D10 to D25, PB3 to PB1, PB19 to PB10, PB18 to PB11, PB11 to PB12, PB12 to PB13, PB13 to PB14, PB14 to PB15, PB15 to PB16, PB16 to PB17, PB17 to PB18, PB7 to PB19, PB1 to PB2, PB6 to PB20, PB9 to PB21, PB2 to PB3, PB5 to PB4, PB4 to PB5, PB8 to PB6, PB21 to PB7, PB22 to PB8, PB20 to PB9, Q12 to Q7, R32 to R79, R33 to R80, R37 to R81, R31 to R82, SW6 to SW1, SW5 to SW2

Commit message: updates to pcb board and creation of BOM
Parts:
- SW1, SW2: now left out of the parts list
Changed lines of the file:
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@@
 		(unit 1)
 		(exclude_from_sim no)
-		(in_bom yes)
+		(in_bom no)
 		(on_board yes)
 		(dnp no)
@@
 		(unit 1)
 		(exclude_from_sim no)
-		(in_bom yes)
+		(in_bom no)
 		(on_board yes)
 		(dnp no)
