File: KiCAD FILES__PCB/gateway.kicad_sch (KiCad schematic)
At the start: 157 parts, among them J1 Conn_01x02_Pin, J10 SIM7100-8-1-15-00-A_REVC, J12 Conn_01x02_Pin, J13 Conn_01x02_Pin, J14 B2B-XH-A_LF__SN_, J15 B2B-XH-A_LF__SN_, J17 B4B-XH-A_LF__SN_, J18 B4B-XH-A_LF__SN_, J19 MEM2067-02-180-00-A_REVB, J2 Conn_01x02_Pin, J20 B3B-XH-A_LF__SN_, J21 B3B-XH-A_LF__SN_, J24 B2B-XH-A_LF__SN_, J28 B4B-XH-A_LF__SN_, J29 B2B-XH-A_LF__SN_, J3 B3B-XH-A_LF__SN_, J31 TYPE-C-31-M-12, J32 B3B-XH-A_LF__SN_, J35 Conn_01x02_Pin, J37 B3B-XH-A_LF__SN_, J38 Conn_01x02_Pin, J39 Conn_01x02_Pin, J40 Conn_01x06_Pin, J9 Conn_01x04_Pin, Q1 MMBT3904, Q2 MMBT3904, Q3 MMBT3904, U1 TXB0108RGYR, U11 AMS1117-3.3, U14 AMS1117-3.3, U16 AMS1117-3.3, U18 AMS1117-3.3, U2 ESP32-WROOM-32E__4MB_HIGH_TEM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, U3 SIM7000E, U6 DS3231MZ_TRL, U7 Ai-Thinker RA-08H, U8 ST3485EBDR, U9 FT232RL-REEL

Commit message: [3rd] Updated layout and routed the Power Board.
Parts:
- removed BT1: BHX1-1225-PC, BHX1-1225-PC:BAT_BHX1-1225-PC, symbol BHX1-1225-PC:BHX1-1225-PC
- removed C1, C11, C14, C22, C23, C24, C3, C38, C4, C40, C7, C8, C9: 0.1uF, Capacitor_SMD:C_0603_1608Metric, symbol Device:C_Small
- removed C10: 22uF, Capacitor_SMD:C_1206_3216Metric_Pad1.33x1.80mm_HandSolder, symbol Device:C
- removed C12, C25, C42, C49, C6, C67, C78: 1uF, Capacitor_SMD:C_0603_1608Metric, symbol Device:C_Small
- removed C13: 100uF, Capacitor_SMD:C_1206_3216Metric_Pad1.33x1.80mm_HandSolder, symbol Device:C
- removed C17, C18, C2, C5: Cm, Capacitor_SMD:C_0603_1608Metric, symbol Device:C_Small
- removed C21: 10uF, Capacitor_SMD:C_1206_3216Metric_Pad1.33x1.80mm_HandSolder, symbol Device:C
- removed C39: 4.7uF, Capacitor_SMD:C_0603_1608Metric, symbol Device:C_Small
- removed C41, C47, C51, C76: 10uF, Capacitor_SMD:C_0603_1608Metric, symbol Device:C_Small
- removed D1, D2, D4: PESDHC3D3V3U, Diode_SMD:D_SOD-323F, symbol PCM_JLCPCB-Diodes:TVS-Uni,SMAJ10A
- removed D12, D13, D17, D18, D6, D9: NET_LED, Diode_SMD:D_0603_1608Metric, symbol Device:LED
- removed D20, D21, D24, D25: 1N5819WS, Diode_SMD:D_SOD-323, symbol Diode:1N5819WS
- removed D5: ESDA6V1W5, ESDA6V1W5:SOT65P210X110-5N, symbol ESDA6V1W5:ESDA6V1W5
- removed FB1: FerriteBead_Small, BLM03HG601SZ1D:BEADC0603X33N, symbol Device:FerriteBead_Small
- removed GSM1, GSM2: U.FL-R-SMT(10), Connector_Coaxial:U.FL_Molex_MCRF_73412-0110_Vertical, symbol U.FL-R-SMT_10_:U.FL-R-SMT(10)
- removed J1, J12, J13, J2, J35, J38, J39: Conn_01x02_Pin, Connector_PinHeader_2.54mm:PinHeader_1x02_P2.54mm_Vertical, symbol Connector:Conn_01x02_Pin
- removed J10: SIM7100-8-1-15-00-A_REVC, SIM7100-8-1-15-00-A_REVC:GCT_SIM7100-8-1-15-00-A_REVC, symbol SIM7100-8-1-15-00-A_REVC:SIM7100-8-1-15-00-A_REVC
- removed J14, J15, J24, J29: B2B-XH-A_LF__SN_, B2B-XH-A_LF__SN_:JST_B2B-XH-A_LF__SN_, symbol B2B-XH-A_LF__SN_:B2B-XH-A_LF__SN_
- removed J17, J18, J28: B4B-XH-A_LF__SN_, B4B-XH-A_LF__SN_:JST_B4B-XH-A_LF__SN_, symbol B4B-XH-A_LF__SN_:B4B-XH-A_LF__SN_
- removed J19: MEM2067-02-180-00-A_REVB, MEM2067-02-180-00-A_REVB:GCT_MEM2067-02-180-00-A_REVB, symbol MEM2067-02-180-00-A_REVB:MEM2067-02-180-00-A_REVB
- removed J20, J21, J3, J32, J37: B3B-XH-A_LF__SN_, B3B-XH-A_LF__SN_:JST_B3B-XH-A_LF__SN_, symbol B3B-XH-A_LF__SN_:B3B-XH-A_LF__SN_
- removed J31: TYPE-C-31-M-12, TYPE-C-31-M-12:HRO_TYPE-C-31-M-12, symbol TYPE-C-31-M-12:TYPE-C-31-M-12
- removed J40: Conn_01x06_Pin, Connector_PinHeader_2.54mm:PinHeader_1x06_P2.54mm_Vertical, symbol Connector:Conn_01x06_Pin
- removed J9: Conn_01x04_Pin, Connector_PinHeader_2.54mm:PinHeader_1x04_P2.54mm_Vertical, symbol Connector:Conn_01x04_Pin
- removed JP1, JP10, JP14, JP15, JP16, JP17, JP2, JP22, JP23, JP24, JP25, JP4, JP6, JP7, JP8: Jumper_2_Small_Open, Jumper:SolderJumper-2_P1.3mm_Open_RoundedPad1.0x1.5mm, symbol Jumper:Jumper_2_Small_Open
- removed Q1, Q2, Q3: MMBT3904, Package_TO_SOT_SMD:SOT-23, symbol Transistor_BJT:MMBT3904
- removed R1, R23: 0R, Resistor_SMD:R_0603_1608Metric, symbol Device:R
- removed R12, R19, R2, R20, R24, R25, R3, R35, R38, R4, R5, R54, R55, R61: 4.7k, Resistor_SMD:R_0603_1608Metric, symbol Device:R
- removed R22, R28, R30, R34: 1k, Resistor_SMD:R_0603_1608Metric, symbol Device:R
- removed R29: 10k, Resistor_SMD:R_0603_1608Metric, symbol Device:R
- removed R36: 120, Resistor_SMD:R_0603_1608Metric, symbol Device:R
- removed R50, R51: 270R, Resistor_SMD:R_0603_1608Metric, symbol Device:R
- removed R52, R53: 5.1k, Resistor_SMD:R_0603_1608Metric, symbol Device:R
- removed R62: 10K, Resistor_SMD:R_0603_1608Metric, symbol Device:R
- removed R63: 20K, Resistor_SMD:R_0603_1608Metric, symbol Device:R
- removed SNS_TX1, SNS_TX10, SNS_TX11, SNS_TX12, SNS_TX13, SNS_TX14, SNS_TX15, SNS_TX2, SNS_TX3, SNS_TX4, SNS_TX5, SNS_TX6, SNS_TX7, SNS_TX8, SNS_TX9: TestPoint, TestPoint:TestPoint_Pad_D1.5mm, symbol Connector:TestPoint
- removed U1: TXB0108RGYR, TXB0108RGYR:IC_TXB0108RGYR, symbol TXB0108RGYR:TXB0108RGYR
- removed U11, U14, U16, U18: AMS1117-3.3, Package_TO_SOT_SMD:SOT-223-3_TabPin2, symbol Regulator_Linear:AMS1117-3.3
- removed U2: ESP32-WROOM-32E__4MB_HIGH_TEMP_, ESP32-WROOM-32UE_M113EH6400UH3Q0_:MODULE_ESP32-WROOM-32UE_M113EH6400UH3Q0_, symbol ESP32-WROOM-32E__4MB_HIGH_TEMP_:ESP32-WROOM-32E__4MB_HIGH_TEMP_
- removed U3: SIM7000E, SIM7000E:SIMCON_SIM7000E, symbol SIM7000E:SIM7000E
- removed U6: DS3231MZ_TRL, DS3231MZ_TRL:SOIC127P600X175-8N, symbol DS3231MZ_TRL:DS3231MZ_TRL
- removed U7: Ai-Thinker RA-08H, RA-08H-Ai-Thinker-Symbol-Kicad-88998:RA-08H, symbol RA-08H:Ai-Thinker RA-08H
- removed U8: ST3485EBDR, ST3485EBDR:SOIC127P600X175-8N, symbol ST3485EBDR:ST3485EBDR
- removed U9: FT232RL-REEL, FT232RL-REEL:SOP65P780X200-28N, symbol FT232RL-REEL:FT232RL-REEL
- added C1: 10uF, Capacitor_THT:CP_Radial_D4.0mm_P2.00mm, symbol Device:C
- added C2: 0.1uF, Capacitor_THT:CP_Radial_D4.0mm_P2.00mm, symbol Device:C
- added J31: +3.3V, TerminalBlock_Phoenix:TerminalBlock_Phoenix_MKDS-1-2-3.81_1x02_P3.81mm_Horizontal, symbol Connector:Screw_Terminal_01x02
- added J32: Conn_01x09_Socket, Connector_PinSocket_2.54mm:PinSocket_1x09_P2.54mm_Vertical, symbol Connector:Conn_01x09_Socket
- added J33: Conn_01x08_Socket, Connector_PinSocket_2.54mm:PinSocket_1x08_P2.54mm_Vertical, symbol Connector:Conn_01x08_Socket
- added J34: GSM, Connector_Molex:Molex_SL_171971-0007_1x07_P2.54mm_Vertical, symbol Connector:Conn_01x07_Socket
- added J35: +5V, TerminalBlock_Phoenix:TerminalBlock_Phoenix_MKDS-1-2-3.81_1x02_P3.81mm_Horizontal, symbol Connector:Screw_Terminal_01x02
- added J36: WIND SPEED, TerminalBlock_Phoenix:TerminalBlock_Phoenix_MKDS-1-2-3.81_1x02_P3.81mm_Horizontal, symbol Connector:Screw_Terminal_01x02
- added J37: LIGHT INTENSITY, TerminalBlock_Phoenix:TerminalBlock_Phoenix_MKDS-1-2-3.81_1x02_P3.81mm_Horizontal, symbol Connector:Screw_Terminal_01x02
- added J38, J48: I2C, TerminalBlock_Phoenix:TerminalBlock_Phoenix_MKDS-1-2-3.81_1x02_P3.81mm_Horizontal, symbol Connector:Screw_Terminal_01x02
- added J39: RAINFALL SENSOR, TerminalBlock_Phoenix:TerminalBlock_Phoenix_MKDS-1-2-3.81_1x02_P3.81mm_Horizontal, symbol Connector:Screw_Terminal_01x02
- added J40: SH25, TerminalBlock_Phoenix:TerminalBlock_Phoenix_MKDS-1-4-3.81_1x04_P3.81mm_Horizontal, symbol Connector:Screw_Terminal_01x04
- added J41: ATM PRESSURE, TerminalBlock_Phoenix:TerminalBlock_Phoenix_MKDS-1-4-3.81_1x04_P3.81mm_Horizontal, symbol Connector:Screw_Terminal_01x04
- added J42: SD CARD, Connector_Molex:Molex_SL_171971-0006_1x06_P2.54mm_Vertical, symbol Connector:Conn_01x06_Socket
- added J43: SOIL MOISTURE, TerminalBlock_Phoenix:TerminalBlock_Phoenix_MKDS-1-3-3.81_1x03_P3.81mm_Horizontal, symbol Connector:Screw_Terminal_01x03
- added J44: SOIL TEMP, TerminalBlock_Phoenix:TerminalBlock_Phoenix_MKDS-1-3-3.81_1x03_P3.81mm_Horizontal, symbol Connector:Screw_Terminal_01x03
- added J45: DHT 22, TerminalBlock_Phoenix:TerminalBlock_Phoenix_MKDS-1-3-3.81_1x03_P3.81mm_Horizontal, symbol Connector:Screw_Terminal_01x03
- added J46: WIND VANE, TerminalBlock_Phoenix:TerminalBlock_Phoenix_MKDS-1-3-3.81_1x03_P3.81mm_Horizontal, symbol Connector:Screw_Terminal_01x03
- added J47: Real Time Clock, Connector_Molex:Molex_SL_171971-0006_1x06_P2.54mm_Vertical, symbol Connector:Conn_01x06_Socket
- added U1: ESP32-DEVKITC-32U, MODULE_ESP32-DEVKITC-32U:MODULE_ESP32-DEVKITC-32U, symbol ESP32-DEVKITC-32U:ESP32-DEVKITC-32U
- D3: value NET_LED -> RED; footprint Diode_SMD:D_0603_1608Metric -> LED_SMD:LED_0402_1005Metric
- D7: value NET_LED -> YELLOW; footprint Diode_SMD:D_0603_1608Metric -> LED_SMD:LED_0402_1005Metric
- R10: value 10k -> 4.7k; footprint Resistor_SMD:R_0603_1608Metric -> Resistor_THT:R_Axial_DIN0204_L3.6mm_D1.6mm_P7.62mm_Horizontal; now fitted
- R11, R6: value 10k -> 4.7k; footprint Resistor_SMD:R_0603_1608Metric -> Resistor_THT:R_Axial_DIN0204_L3.6mm_D1.6mm_P7.62mm_Horizontal
- R13: value 4.7k -> 2k; footprint Resistor_SMD:R_0603_1608Metric -> Resistor_THT:R_Axial_DIN0204_L3.6mm_D1.6mm_P7.62mm_Horizontal
- R14: footprint Resistor_SMD:R_0603_1608Metric -> Resistor_THT:R_Axial_DIN0204_L3.6mm_D1.6mm_P7.62mm_Horizontal
- R15: value 1k -> 2k; footprint Resistor_SMD:R_0603_1608Metric -> Resistor_THT:R_Axial_DIN0204_L3.6mm_D1.6mm_P7.62mm_Horizontal
- R7: value 1k -> 4.7k; footprint Resistor_SMD:R_0603_1608Metric -> Resistor_THT:R_Axial_DIN0204_L3.6mm_D1.6mm_P7.62mm_Horizontal
- R8: value 10k -> 0.47k; footprint Resistor_SMD:R_0603_1608Metric -> Resistor_THT:R_Axial_DIN0204_L3.6mm_D1.6mm_P7.62mm_Horizontal
- R9: value 10k -> 1k; footprint Resistor_SMD:R_0603_1608Metric -> Resistor_THT:R_Axial_DIN0204_L3.6mm_D1.6mm_P7.62mm_Horizontal
Connections:
- net LORA_TX is gone; now on net +3.3V: R10.2
- net S1223 is gone; now on an unnamed net: R8.2
- net GND: now also R13.2, C1.2, C2.2, J31.2 (Pin_2), J32.1 (Pin_1), J33.8 (Pin_8), J34.6 (Pin_6), J35.2 (Pin_2), J36.2 (Pin_2), J37.2 (Pin_2), J39.2 (Pin_2), J40.4 (Pin_4), J41.4 (Pin_4), J42.1 (Pin_1), J43.3 (Pin_3), J44.3 (Pin_3), J45.3 (Pin_3), J46.3 (Pin_3), J47.6 (Pin_6), U1.38 (GND3); no longer R11.2, R13.1, R8.1, R9.2
- net at D3.2 (A): no longer R7.1
- net at R14.1: now also J46.2 (Pin_2)
- net +3.3V: now reaches R6.2
- net +3.3V: now also R11.2, R7.2, R8.1, C1.1, C2.1, J31.1 (Pin_1), J32.9 (Pin_9), J40.1 (Pin_1), J41.1 (Pin_1), J42.6 (Pin_6)
- net at D7.2 (A): now also R9.2; no longer R15.1
- removed net ESP32 power in: R10.1, R6.1, R7.2
- net GSM_pw in renamed G27
- net G27: now also R13.1, U1.11 (IO27); no longer R15.2
- net strap12 renamed G35
- net G35: now also J37.1 (Pin_1), J39.1 (Pin_1), U1.6 (IO35)
- net strap2 renamed G15
- net G15: now also J33.2 (Pin_2), U1.23 (IO15)
- new net +5V: J34.7 (Pin_7), J35.1 (Pin_1), J43.1 (Pin_1), J44.1 (Pin_1), J45.1 (Pin_1), J46.1 (Pin_1), J47.5 (Pin_5), R15.1, U1.19 (EXT_5V)
- new net G12: J36.1 (Pin_1), R10.1, U1.13 (IO12)
- new net G14: J33.1 (Pin_1), U1.12 (IO14)
- new net G18: J42.3 (Pin_3), U1.30 (IO18)
- new net G19: J42.4 (Pin_4), U1.31 (IO19)
- new net G21: J38.2 (Pin_2), J40.2 (Pin_2), J41.2 (Pin_2), J47.3 (Pin_3), J48.1 (Pin_1), R7.1, U1.33 (IO21)
- new net G22: J38.1 (Pin_1), J40.3 (Pin_3), J41.3 (Pin_3), J47.4 (Pin_4), J48.2 (Pin_2), R6.1, U1.36 (IO22)
- new net G23: J42.5 (Pin_5), U1.37 (IO23)
- new net G33: J44.2 (Pin_2), R15.2, U1.8 (IO33)
- new net G34: J43.2 (Pin_2), U1.5 (IO34)
- new net G4: J42.2 (Pin_2), U1.26 (IO4)
- new net G5: J45.2 (Pin_2), U1.29 (IO5)
- new net GSM_RST: J34.1 (Pin_1), U1.15 (IO13)
- new net RXD: J34.3 (Pin_3), U1.28 (IO17)
- new net TXD: J34.4 (Pin_4), U1.27 (IO16)
- no-connect marks 46 -> 35
Other:
- note added: "3.3V SUPPLY"
- note added: "32K"
- note added: "5V SUPPLY"
- note added: "CLK"
- note added: "CS"
- note added: "ESP32 DEV-KIT"
- note added: "GND"
- note added: "I2C"
- note added: "MISO"
- note added: "MOSI"
- note added: "SCL"
- note added: "SDA"
- note added: "SD_CARD"
- note added: "SIM800L GSM"
- note added: "SQW"
- note added: "VCC"
- note removed: "DAVIS 7852"
- note removed: "DS18B20"
- note removed: "ESP 32 MICROCONTROLLER"
- note removed: "FTDI USB-Serial Interface IC"
- note removed: "GL5506 used instead of S1223, both are LDR hence interchangable"
- note removed: "GSM COMMUNICATION"
- note removed: "INSPEED EVANE"
- note removed: "INSPEED VORTEX"
- note removed: "MEMORY CARD"
- note removed: "MPL3115ARI"
- note removed: "PROPER UART CONNECTION"
- note removed: "RESET CONTROLLED BY ESP32"
- note removed: "RS485 COMMUNICATION"
- note removed: "S1223"
- note removed: "SHT25"
- note removed: "VH400"
- note removed: "boot option straping pin refenced from datasheet"
- note removed: "level shifter"
- note removed: "power indication led, optional, placed for block debugging"
- note removed: "programming connector, input power scheme covered in power board"
