File: KiCAD FILES__PCB/gateway.kicad_sch (KiCad schematic)
At the start: 157 parts, among them J1 Conn_01x02_Pin, J10 SIM7100-8-1-15-00-A_REVC, J12 Conn_01x02_Pin, J13 Conn_01x02_Pin, J14 B2B-XH-A_LF__SN_, J15 B2B-XH-A_LF__SN_, J17 B4B-XH-A_LF__SN_, J18 B4B-XH-A_LF__SN_, J19 MEM2067-02-180-00-A_REVB, J2 Conn_01x02_Pin, J20 B3B-XH-A_LF__SN_, J21 B3B-XH-A_LF__SN_, J24 B2B-XH-A_LF__SN_, J28 B4B-XH-A_LF__SN_, J29 B2B-XH-A_LF__SN_, J3 B3B-XH-A_LF__SN_, J31 TYPE-C-31-M-12, J32 B3B-XH-A_LF__SN_, J35 Conn_01x02_Pin, J37 B3B-XH-A_LF__SN_, J38 Conn_01x02_Pin, J39 Conn_01x02_Pin, J40 Conn_01x06_Pin, J9 Conn_01x04_Pin, Q1 MMBT3904, Q2 MMBT3904, Q3 MMBT3904, U1 TXB0108RGYR, U11 AMS1117-3.3, U14 AMS1117-3.3, U16 AMS1117-3.3, U18 AMS1117-3.3, U2 ESP32-WROOM-32E__4MB_HIGH_TEM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, U3 SIM7000E, U6 DS3231MZ_TRL, U7 Ai-Thinker RA-08H, U8 ST3485EBDR, U9 FT232RL-REEL

Commit message: Finished the gateway schematic and pcb successfully
Parts:
- removed BT1: BHX1-1225-PC, BHX1-1225-PC:BAT_BHX1-1225-PC, symbol BHX1-1225-PC:BHX1-1225-PC
- removed C1, C11, C14, C22, C23, C24, C3, C38, C4, C40, C7, C8, C9: 0.1uF, Capacitor_SMD:C_0603_1608Metric, symbol Device:C_Small
- removed C10: 22uF, Capacitor_SMD:C_1206_3216Metric_Pad1.33x1.80mm_HandSolder, symbol Device:C
- removed C12, C25, C42, C49, C6, C67, C78: 1uF, Capacitor_SMD:C_0603_1608Metric, symbol Device:C_Small
- removed C13: 100uF, Capacitor_SMD:C_1206_3216Metric_Pad1.33x1.80mm_HandSolder, symbol Device:C
- removed C17, C18, C2, C5: Cm, Capacitor_SMD:C_0603_1608Metric, symbol Device:C_Small
- removed C21: 10uF, Capacitor_SMD:C_1206_3216Metric_Pad1.33x1.80mm_HandSolder, symbol Device:C
- removed C39: 4.7uF, Capacitor_SMD:C_0603_1608Metric, symbol Device:C_Small
- removed C41, C47, C51, C76: 10uF, Capacitor_SMD:C_0603_1608Metric, symbol Device:C_Small
- removed D1, D2, D4: PESDHC3D3V3U, Diode_SMD:D_SOD-323F, symbol PCM_JLCPCB-Diodes:TVS-Uni,SMAJ10A
- removed D12, D13, D17, D18, D3, D6, D7, D9: NET_LED, Diode_SMD:D_0603_1608Metric, symbol Device:LED
- removed D20, D21, D24, D25: 1N5819WS, Diode_SMD:D_SOD-323, symbol Diode:1N5819WS
- removed D5: ESDA6V1W5, ESDA6V1W5:SOT65P210X110-5N, symbol ESDA6V1W5:ESDA6V1W5
- removed FB1: FerriteBead_Small, BLM03HG601SZ1D:BEADC0603X33N, symbol Device:FerriteBead_Small
- removed GSM1, GSM2: U.FL-R-SMT(10), Connector_Coaxial:U.FL_Molex_MCRF_73412-0110_Vertical, symbol U.FL-R-SMT_10_:U.FL-R-SMT(10)
- removed J1, J12, J13, J2, J35, J38, J39: Conn_01x02_Pin, Connector_PinHeader_2.54mm:PinHeader_1x02_P2.54mm_Vertical, symbol Connector:Conn_01x02_Pin
- removed J10: SIM7100-8-1-15-00-A_REVC, SIM7100-8-1-15-00-A_REVC:GCT_SIM7100-8-1-15-00-A_REVC, symbol SIM7100-8-1-15-00-A_REVC:SIM7100-8-1-15-00-A_REVC
- removed J14, J15, J24, J29: B2B-XH-A_LF__SN_, B2B-XH-A_LF__SN_:JST_B2B-XH-A_LF__SN_, symbol B2B-XH-A_LF__SN_:B2B-XH-A_LF__SN_
- removed J17, J18, J28: B4B-XH-A_LF__SN_, B4B-XH-A_LF__SN_:JST_B4B-XH-A_LF__SN_, symbol B4B-XH-A_LF__SN_:B4B-XH-A_LF__SN_
- removed J19: MEM2067-02-180-00-A_REVB, MEM2067-02-180-00-A_REVB:GCT_MEM2067-02-180-00-A_REVB, symbol MEM2067-02-180-00-A_REVB:MEM2067-02-180-00-A_REVB
- removed J20, J21, J3, J32, J37: B3B-XH-A_LF__SN_, B3B-XH-A_LF__SN_:JST_B3B-XH-A_LF__SN_, symbol B3B-XH-A_LF__SN_:B3B-XH-A_LF__SN_
- removed J31: TYPE-C-31-M-12, TYPE-C-31-M-12:HRO_TYPE-C-31-M-12, symbol TYPE-C-31-M-12:TYPE-C-31-M-12
- removed J40: Conn_01x06_Pin, Connector_PinHeader_2.54mm:PinHeader_1x06_P2.54mm_Vertical, symbol Connector:Conn_01x06_Pin
- removed J9: Conn_01x04_Pin, Connector_PinHeader_2.54mm:PinHeader_1x04_P2.54mm_Vertical, symbol Connector:Conn_01x04_Pin
- removed JP1, JP10, JP14, JP15, JP16, JP17, JP2, JP22, JP23, JP24, JP25, JP4, JP6, JP7, JP8: Jumper_2_Small_Open, Jumper:SolderJumper-2_P1.3mm_Open_RoundedPad1.0x1.5mm, symbol Jumper:Jumper_2_Small_Open
- removed Q1, Q2, Q3: MMBT3904, Package_TO_SOT_SMD:SOT-23, symbol Transistor_BJT:MMBT3904
- removed R1, R23: 0R, Resistor_SMD:R_0603_1608Metric, symbol Device:R
- removed R11, R29: 10k, Resistor_SMD:R_0603_1608Metric, symbol Device:R
- removed R12, R13, R19, R2, R20, R24, R25, R3, R35, R38, R4, R54, R55, R61: 4.7k, Resistor_SMD:R_0603_1608Metric, symbol Device:R
- removed R14, R15, R22, R28, R30, R34: 1k, Resistor_SMD:R_0603_1608Metric, symbol Device:R
- removed R36: 120, Resistor_SMD:R_0603_1608Metric, symbol Device:R
- removed R50, R51: 270R, Resistor_SMD:R_0603_1608Metric, symbol Device:R
- removed R52, R53: 5.1k, Resistor_SMD:R_0603_1608Metric, symbol Device:R
- removed R62: 10K, Resistor_SMD:R_0603_1608Metric, symbol Device:R
- removed R63: 20K, Resistor_SMD:R_0603_1608Metric, symbol Device:R
- removed SNS_TX1, SNS_TX10, SNS_TX11, SNS_TX12, SNS_TX13, SNS_TX14, SNS_TX15, SNS_TX2, SNS_TX3, SNS_TX4, SNS_TX5, SNS_TX6, SNS_TX7, SNS_TX8, SNS_TX9: TestPoint, TestPoint:TestPoint_Pad_D1.5mm, symbol Connector:TestPoint
- removed U1: TXB0108RGYR, TXB0108RGYR:IC_TXB0108RGYR, symbol TXB0108RGYR:TXB0108RGYR
- removed U11, U14, U16, U18: AMS1117-3.3, Package_TO_SOT_SMD:SOT-223-3_TabPin2, symbol Regulator_Linear:AMS1117-3.3
- removed U2: ESP32-WROOM-32E__4MB_HIGH_TEMP_, ESP32-WROOM-32UE_M113EH6400UH3Q0_:MODULE_ESP32-WROOM-32UE_M113EH6400UH3Q0_, symbol ESP32-WROOM-32E__4MB_HIGH_TEMP_:ESP32-WROOM-32E__4MB_HIGH_TEMP_
- removed U3: SIM7000E, SIM7000E:SIMCON_SIM7000E, symbol SIM7000E:SIM7000E
- removed U6: DS3231MZ_TRL, DS3231MZ_TRL:SOIC127P600X175-8N, symbol DS3231MZ_TRL:DS3231MZ_TRL
- removed U7: Ai-Thinker RA-08H, RA-08H-Ai-Thinker-Symbol-Kicad-88998:RA-08H, symbol RA-08H:Ai-Thinker RA-08H
- removed U8: ST3485EBDR, ST3485EBDR:SOIC127P600X175-8N, symbol ST3485EBDR:ST3485EBDR
- removed U9: FT232RL-REEL, FT232RL-REEL:SOP65P780X200-28N, symbol FT232RL-REEL:FT232RL-REEL
- added C1: 10uF, Capacitor_SMD:C_0402_1005Metric_Pad0.74x0.62mm_HandSolder, symbol Device:C
- added C2: 0.1uF, Capacitor_SMD:C_0402_1005Metric_Pad0.74x0.62mm_HandSolder, symbol Device:C
- added J1: GSM, Connector_PinSocket_2.54mm:PinSocket_1x07_P2.54mm_Vertical, symbol Connector:Conn_01x07_Socket
- added J10: I2C, TerminalBlock_Phoenix:TerminalBlock_Phoenix_MKDS-3-2-5.08_1x02_P5.08mm_Horizontal, symbol Connector:Screw_Terminal_01x02
- added J11: WIND SPEED, TerminalBlock_Phoenix:TerminalBlock_Phoenix_MKDS-3-2-5.08_1x02_P5.08mm_Horizontal, symbol Connector:Screw_Terminal_01x02
- added J12: LIGHT INTENSITY, TerminalBlock_Phoenix:TerminalBlock_Phoenix_MKDS-3-2-5.08_1x02_P5.08mm_Horizontal, symbol Connector:Screw_Terminal_01x02
- added J13: RAINFALL SENSOR, TerminalBlock_Phoenix:TerminalBlock_Phoenix_MKDS-3-2-5.08_1x02_P5.08mm_Horizontal, symbol Connector:Screw_Terminal_01x02
- added J14: SH25, TerminalBlock_Phoenix:TerminalBlock_Phoenix_MKDS-3-4-5.08_1x04_P5.08mm_Horizontal, symbol Connector:Screw_Terminal_01x04
- added J15: ATM PRESSURE, TerminalBlock_Phoenix:TerminalBlock_Phoenix_MKDS-3-4-5.08_1x04_P5.08mm_Horizontal, symbol Connector:Screw_Terminal_01x04
- added J16, J17: Conn_01x09_Socket, Connector_PinSocket_2.54mm:PinSocket_1x09_P2.54mm_Vertical, symbol Connector:Conn_01x09_Socket
- added J18: SOIL TEMP, TerminalBlock_Phoenix:TerminalBlock_Phoenix_MKDS-3-3-5.08_1x03_P5.08mm_Horizontal, symbol Connector:Screw_Terminal_01x03
- added J19: DHT 22, TerminalBlock_Phoenix:TerminalBlock_Phoenix_MKDS-3-3-5.08_1x03_P5.08mm_Horizontal, symbol Connector:Screw_Terminal_01x03
- added J2: Conn_01x02_Socket, symbol Connector:Conn_01x02_Socket
- added J20: SOIL MOISTURE, TerminalBlock_Phoenix:TerminalBlock_Phoenix_MKDS-3-3-5.08_1x03_P5.08mm_Horizontal, symbol Connector:Screw_Terminal_01x03
- added J21: WIND VANE, TerminalBlock_Phoenix:TerminalBlock_Phoenix_MKDS-3-3-5.08_1x03_P5.08mm_Horizontal, symbol Connector:Screw_Terminal_01x03
- added J3: RTC_MODULE, Connector_PinSocket_2.54mm:PinSocket_1x06_P2.54mm_Vertical, symbol Connector:Conn_01x06_Socket
- added J9: SD_CARD, Connector_PinSocket_2.54mm:PinSocket_1x06_P2.54mm_Vertical, symbol Connector:Conn_01x06_Socket
- added U1: ESP32-DEVKITC-32U, ESP32devkit:MODULE_ESP32-DEVKITC-32U, symbol ESP32-DEVKITC-32U:ESP32-DEVKITC-32U
- R10: value 10k -> 4.7k; footprint Resistor_SMD:R_0603_1608Metric -> Resistor_THT:R_Axial_DIN0207_L6.3mm_D2.5mm_P7.62mm_Horizontal; now fitted
- R5, R7: footprint Resistor_SMD:R_0603_1608Metric -> Resistor_THT:R_Axial_DIN0207_L6.3mm_D2.5mm_P7.62mm_Horizontal
- R6, R9: value 10k -> 4.7k; footprint Resistor_SMD:R_0603_1608Metric -> Resistor_THT:R_Axial_DIN0207_L6.3mm_D2.5mm_P7.62mm_Horizontal
- R8: value 10k -> 2k; footprint Resistor_SMD:R_0603_1608Metric -> Resistor_THT:R_Axial_DIN0207_L6.3mm_D2.5mm_P7.62mm_Horizontal
Connections:
- net LORA_TX is gone; now on net +3V3: R10.2
- net S1223 is gone; now on net GND: R8.2
- net GND: now also C1.2, C2.2, J1.2 (Pin_2), J11.2 (Pin_2), J12.2 (Pin_2), J13.2 (Pin_2), J14.4 (Pin_4), J15.4 (Pin_4), J16.1 (Pin_1), J17.2 (Pin_2), J18.3 (Pin_3), J19.3 (Pin_3), J20.3 (Pin_3), J21.3 (Pin_3), J3.6 (Pin_6), J9.6 (Pin_6), U1.38 (GND3); no longer R5.1, R8.1, R9.2
- net at R7.1: now also J21.2 (Pin_2)
- net +3V3: now reaches R5.2
- net +3V3: now also R6.2, R9.2, J14.1 (Pin_1), J15.1 (Pin_1), J9.5 (Pin_5)
- removed net ESP32 power in: R10.1, R6.1, R7.2
- net strap2 renamed G21
- net G21: now also J10.2 (Pin_2), J14.2 (Pin_2), J15.2 (Pin_2), J3.3 (Pin_3), U1.33 (IO21)
- new net +5V: J1.1 (Pin_1), J3.5 (Pin_5), U1.19 (EXT_5V)
- new net 3V3: C1.1, C2.1, J16.9 (Pin_9)
- new net 5V: J18.1 (Pin_1), J19.1 (Pin_1), J20.1 (Pin_1), J21.1 (Pin_1)
- new net ANT: J17.1 (Pin_1)
- new net G12: J11.1 (Pin_1), R5.1
- new net G14: J17.9 (Pin_9), U1.12 (IO14)
- new net G15: J17.8 (Pin_8), U1.23 (IO15)
- new net G16: J1.4 (Pin_4), U1.27 (IO16)
- new net G17: J1.5 (Pin_5), U1.28 (IO17)
- new net G18: J9.2 (Pin_2), U1.30 (IO18)
- new net G19: J9.4 (Pin_4), U1.31 (IO19)
- new net G22: J10.1 (Pin_1), J14.3 (Pin_3), J15.3 (Pin_3), J3.4 (Pin_4), R10.1, U1.36 (IO22)
- new net G23: J9.3 (Pin_3), U1.37 (IO23)
- new net G27: R7.2, R8.1
- new net G33: J18.2 (Pin_2)
- new net G34: J20.2 (Pin_2)
- new net G35: J12.1 (Pin_1), J13.1 (Pin_1), R6.1
- new net G4: J9.1 (Pin_1), U1.26 (IO4)
- new net G5: J19.2 (Pin_2)
- new net GSM_RST: J1.7 (Pin_7), U1.15 (IO13)
- new net I02: J17.4 (Pin_4)
- new net RST: J17.3 (Pin_3)
- no-connect marks 46 -> 7
Other:
- note added: "LDO"
- note added: "RXD"
- note added: "TXD"
- note removed: "DAVIS 7852"
- note removed: "DS18B20"
- note removed: "FTDI USB-Serial Interface IC"
- note removed: "GL5506 used instead of S1223, both are LDR hence interchangable"
- note removed: "INSPEED EVANE"
- note removed: "INSPEED VORTEX"
- note removed: "MPL3115ARI"
- note removed: "PROPER UART CONNECTION"
- note removed: "RESET CONTROLLED BY ESP32"
- note removed: "RS485 COMMUNICATION"
- note removed: "S1223"
- note removed: "SHT25"
- note removed: "VH400"
- note removed: "boot option straping pin refenced from datasheet"
- note removed: "level shifter"
- note removed: "power indication led, optional, placed for block debugging"
- note removed: "programming connector, input power scheme covered in power board"
