File: KiCAD FILES__PCB/power.kicad_sch (KiCad schematic)
At the start: 137 parts, among them J25 Screw_Terminal_01x02, J26 Screw_Terminal_01x02, J27 Screw_Terminal_01x02, J36 B4B-XH-A_LF__SN_, J4 B2B-XH-A_LF__SN_, J5 Conn_01x02_Pin, J6 Conn_01x02_Pin, J7 Conn_01x02_Pin, J8 Conn_01x02_Pin, Q12 2N7002, Q4 2N7002, Q5 NMOS, Q9 NMOS, SW5 SW_SPST, SW6 SW_SPST, U10 BQ24650RVAR, U12 TPS2121RUXR, U13 AP64501SP-13, U15 STM32F401CCU6, U17 AMS1117-3.3, Y1 C3E-25.000-12-3030-X-R

Commit message: Finished the gateway schematic and pcb successfully
Parts:
- removed C26, C27, C68, C69: 0.1uF, Capacitor_SMD:C_0603_1608Metric, symbol Device:C_Small
- removed C28: 10uF, Capacitor_SMD:CP_Elec_5x5.8, symbol Device:C_Polarized_Small_US
- removed C29: 100nF, Capacitor_SMD:C_1206_3216Metric_Pad1.33x1.80mm_HandSolder, symbol Device:C
- removed C30: 10nF, Capacitor_SMD:C_0603_1608Metric_Pad1.08x0.95mm_HandSolder, symbol Device:C
- removed C31: OPEN, Capacitor_SMD:C_0201_0603Metric_Pad0.64x0.40mm_HandSolder, symbol Device:C
- removed C32: 2.7nF, Capacitor_SMD:C_0603_1608Metric, symbol Device:C
- removed C33, C35, C36: 22uF, Capacitor_SMD:C_0603_1608Metric_Pad1.08x0.95mm_HandSolder, symbol Device:C
- removed C34: 33pF, Capacitor_SMD:C_0603_1608Metric, symbol Device:C
- removed C37: 0.01uF, Capacitor_SMD:C_0603_1608Metric_Pad1.08x0.95mm_HandSolder, symbol Device:C
- removed C43, C73: 10uF, Capacitor_SMD:C_0603_1608Metric, symbol Device:C_Small
- removed C44, C74: 1uF, Capacitor_SMD:C_0603_1608Metric, symbol Device:C_Small
- removed C45, C46: 22pF, Capacitor_SMD:C_0603_1608Metric, symbol Device:C_Small
- removed C52, C60: 2.2uF, Capacitor_SMD:C_0603_1608Metric_Pad1.08x0.95mm_HandSolder, symbol Device:C
- removed C53, C64: 22pF, Capacitor_SMD:C_0603_1608Metric_Pad1.08x0.95mm_HandSolder, symbol Device:C
- removed C54, C55, C57, C63: 1uF, Capacitor_SMD:C_0603_1608Metric_Pad1.08x0.95mm_HandSolder, symbol Device:C
- removed C56: 0.1uf, Capacitor_SMD:C_0603_1608Metric_Pad1.08x0.95mm_HandSolder, symbol Device:C
- removed C58, C59, C65: 10uF, Capacitor_SMD:C_1210_3225Metric_Pad1.33x2.70mm_HandSolder, symbol Device:C
- removed C61: 0.1uF, Capacitor_SMD:C_0603_1608Metric_Pad1.08x0.95mm_HandSolder, symbol Device:C
- removed C62: 10uF, Capacitor_SMD:C_0603_1608Metric_Pad1.08x0.95mm_HandSolder, symbol Device:C
- removed C70, C72: 4.7uF, Capacitor_SMD:C_0603_1608Metric, symbol Device:C_Small
- removed C71: 10nF, Capacitor_SMD:C_0603_1608Metric, symbol Device:C_Small
- removed D10: red, LED_SMD:LED_1206_3216Metric, symbol Device:LED
- removed D14, D15: NET_LED, Diode_SMD:D_0603_1608Metric, symbol Device:LED
- removed D16, D23: D, Diode_SMD:D_1210_3225Metric, symbol Device:D
- removed D19: green, LED_SMD:LED_1206_3216Metric, symbol Device:LED
- removed D22: PESDHC3D3V3U, Diode_SMD:D_SOD-323F, symbol PCM_JLCPCB-Diodes:TVS-Uni,SMAJ10A
- removed J25, J26, J27: Screw_Terminal_01x02, TerminalBlock_MetzConnect:TerminalBlock_MetzConnect_Type011_RT05502HBWC_1x02_P5.00mm_Horizontal, symbol Connector:Screw_Terminal_01x02
- removed J36: B4B-XH-A_LF__SN_, B4B-XH-A_LF__SN_:JST_B4B-XH-A_LF__SN_, symbol B4B-XH-A_LF__SN_:B4B-XH-A_LF__SN_
- removed J4: B2B-XH-A_LF__SN_, B2B-XH-A_LF__SN_:JST_B2B-XH-A_LF__SN_, symbol B2B-XH-A_LF__SN_:B2B-XH-A_LF__SN_
- removed J5, J6, J7, J8: Conn_01x02_Pin, Connector_PinHeader_2.54mm:PinHeader_1x02_P2.54mm_Vertical, symbol Connector:Conn_01x02_Pin
- removed JP11, JP12, JP13, JP18, JP20, JP21, JP9: Jumper_2_Small_Open, Jumper:SolderJumper-2_P1.3mm_Open_RoundedPad1.0x1.5mm, symbol Jumper:Jumper_2_Small_Open
- removed JP19: Jumper_2_Small_Open, Jumper:SolderJumper-2_P1.3mm_Open_Pad1.0x1.5mm, symbol Jumper:Jumper_2_Small_Open
- removed L1: SRN6045TA-3R3Y, Inductor_SMD:L_Bourns_SRN6045TA, symbol Device:L
- removed L2: 6.1uH, MPPT INDUCTORS:CDEP147NP-6R1MC-95, symbol Device:L
- removed PB1, PB11, PB12, PB13, PB14, PB15, PB16, PB17, PB18, PB19, PB2, PB20, PB21, PB22, PB3, PB4, PB5, PB6, PB7, PB8, PB9: TestPoint, TestPoint:TestPoint_Pad_D1.0mm, symbol Connector:TestPoint
- removed Q12, Q4: 2N7002, PCM_JLCPCB:Q_SOT-23, symbol PCM_JLCPCB-Transistors:NMOS,2N7002
- removed Q5, Q9: NMOS, NTMFS4H01NFT3G:TRANS_NVMFS5834NLWFT1G, symbol Simulation_SPICE:NMOS
- removed R31, R32, R33, R49, R57, R59, R64, R69, R70, R81: 10K, Resistor_SMD:R_0603_1608Metric, symbol Device:R
- removed R37: 330, Resistor_SMD:R_0603_1608Metric, symbol Device:R
- removed R39, R40, R41: 5K1, Resistor_SMD:R_0603_1608Metric_Pad0.98x0.95mm_HandSolder, symbol Device:R
- removed R42, R44: 23.7k, Resistor_SMD:R_0603_1608Metric_Pad0.98x0.95mm_HandSolder, symbol Device:R
- removed R43, R45: 5k, Resistor_SMD:R_0603_1608Metric_Pad0.98x0.95mm_HandSolder, symbol Device:R
- removed R46: 51.1K, Resistor_SMD:R_0603_1608Metric_Pad0.98x0.95mm_HandSolder, symbol Device:R
- removed R47, R48: 3.9, Resistor_SMD:R_0603_1608Metric, symbol Device:R
- removed R56: 20k, Resistor_SMD:R_0603_1608Metric, symbol Device:R
- removed R58: 13k, Resistor_SMD:R_0603_1608Metric, symbol Device:R
- removed R60: 1.5K, Resistor_SMD:R_0603_1608Metric, symbol Device:R
- removed R65: 2k, Resistor_SMD:R_0603_1608Metric, symbol Device:R
- removed R66: 499K, Resistor_SMD:R_0603_1608Metric, symbol Device:R
- removed R67: 36K, Resistor_SMD:R_0603_1608Metric, symbol Device:R
- removed R68: 25k, Resistor_SMD:R_0603_1608Metric, symbol Device:R
- removed R71: 5.23k, Resistor_SMD:R_0603_1608Metric, symbol Device:R
- removed R72: 7.5k, Resistor_SMD:R_0603_1608Metric, symbol Device:R
- removed R73: 10, Resistor_SMD:R_0603_1608Metric, symbol Device:R
- removed R74: 100, Resistor_SMD:R_0603_1608Metric, symbol Device:R
- removed R75: 2.2, Resistor_SMD:R_0603_1608Metric, symbol Device:R
- removed R76: 10, Resistor_SMD:R_1812_4532Metric, symbol Device:R
- removed R77: 4.22M, Resistor_SMD:R_0603_1608Metric, symbol Device:R
- removed R78: 154k, Resistor_SMD:R_0603_1608Metric, symbol Device:R
- removed R79: 887k, Resistor_SMD:R_0603_1608Metric, symbol Device:R
- removed R80: 162k, Resistor_SMD:R_0603_1608Metric, symbol Device:R
- removed R82: 1.2K, Resistor_SMD:R_0603_1608Metric, symbol Device:R
- removed SW5, SW6: SW_SPST, Button_Switch_THT:SW_DIP_SPSTx01_Slide_9.78x4.72mm_W7.62mm_P2.54mm, symbol Switch:SW_SPST
- removed TH2: 100k, Resistor_SMD:R_1812_4532Metric, symbol Device:Thermistor_NTC
- removed TP1: TestPoint, TestPoint:TestPoint_Pad_1.0x1.0mm, symbol Connector:TestPoint
- removed U10: BQ24650RVAR, BQ24650RVAR:QFN50P350X350X100-17N, symbol BQ24650RVAR:BQ24650RVAR
- removed U12: TPS2121RUXR, TPS2121RUXR:IC_TPS2121RUXR, symbol TPS2121RUXR:TPS2121RUXR
- removed U13: AP64501SP-13, AP64501SP-13:SOIC127P600X170-9N, symbol ap64501:AP64501SP-13
- removed U15: STM32F401CCU6, STM32F401CCU6 (1):QFN50P700X700X60-49N, symbol STM32F401CCU6:STM32F401CCU6
- removed U17: AMS1117-3.3, Package_TO_SOT_SMD:SOT-223-3_TabPin2, symbol Regulator_Linear:AMS1117-3.3
- removed Y1: C3E-25.000-12-3030-X-R, C3E-25.000-12-3030-X-R:XTAL_C3E-25.000-12-3030-X-R, symbol C3E-25.000-12-3030-X-R:C3E-25.000-12-3030-X-R
- added D1, D4: LED, LED_THT:LED_D5.0mm, symbol Device:LED
- added D2, D5, D6: 1N5822, Diode_THT:D_DO-201AD_P12.70mm_Horizontal, symbol Diode:1N5822
- added J22: SOLAR_INPUT, TerminalBlock_MetzConnect:TerminalBlock_MetzConnect_Type055_RT01502HDWU_1x02_P5.00mm_Horizontal, symbol Connector:Screw_Terminal_01x02
- added J23: DCJACK_INPUT, TerminalBlock_MetzConnect:TerminalBlock_MetzConnect_Type011_RT05502HBWC_1x02_P5.00mm_Horizontal, symbol Connector:Screw_Terminal_01x02
- added J24, J30: IN+, Connector_PinSocket_2.54mm:PinSocket_1x01_P2.54mm_Vertical, symbol Connector:Conn_01x01_Socket
- added J25, J31: IN-, Connector_PinSocket_2.54mm:PinSocket_1x01_P2.54mm_Vertical, symbol Connector:Conn_01x01_Socket
- added J26: P-, Connector_PinSocket_2.54mm:PinSocket_1x01_P2.54mm_Vertical, symbol Connector:Conn_01x01_Socket
- added J27: 4.2V, Connector_PinSocket_2.54mm:PinSocket_1x01_P2.54mm_Vertical, symbol Connector:Conn_01x01_Socket
- added J28, J33: OUT+, Connector_PinSocket_2.54mm:PinSocket_1x01_P2.54mm_Vertical, symbol Connector:Conn_01x01_Socket
- added J29, J34: OUT-, Connector_PinSocket_2.54mm:PinSocket_1x01_P2.54mm_Vertical, symbol Connector:Conn_01x01_Socket
- added J32: 5V_OUTPUT, TerminalBlock_MetzConnect:TerminalBlock_MetzConnect_Type055_RT01502HDWU_1x02_P5.00mm_Horizontal, symbol Connector:Screw_Terminal_01x02
- added J35: IN, Connector_PinSocket_2.54mm:PinSocket_1x02_P2.54mm_Vertical, symbol Connector:Conn_01x02_Socket
- added J36, J37: Conn_01x03_Socket, Connector_PinSocket_2.54mm:PinSocket_1x03_P2.54mm_Vertical, symbol Connector:Conn_01x03_Socket
- added J38: 3.3V_OUTPUT, TerminalBlock_MetzConnect:TerminalBlock_MetzConnect_Type055_RT01502HDWU_1x02_P5.00mm_Horizontal, symbol Connector:Screw_Terminal_01x02
- added J39: OUT, Connector_PinSocket_2.54mm:PinSocket_1x02_P2.54mm_Vertical, symbol Connector:Conn_01x02_Socket
- added J4: BATTERY_INPUT, TerminalBlock_MetzConnect:TerminalBlock_MetzConnect_Type055_RT01504HDWU_1x04_P5.00mm_Horizontal, symbol Connector:Screw_Terminal_01x04
- added J40, J45: Conn_01x20_Socket, Connector_PinSocket_2.54mm:PinSocket_1x20_P2.54mm_Vertical, symbol Connector:Conn_01x20_Socket
- added J41, J42, J43, J44, J7: 12.6V, Connector_PinSocket_2.54mm:PinSocket_1x01_P2.54mm_Vertical, symbol Connector:Conn_01x01_Socket
- added J46: I2C, TerminalBlock_MetzConnect:TerminalBlock_MetzConnect_Type055_RT01502HDWU_1x02_P5.00mm_Horizontal, symbol Connector:Screw_Terminal_01x02
- added J5: 8.4V, Connector_PinSocket_2.54mm:PinSocket_1x01_P2.54mm_Vertical, symbol Connector:Conn_01x01_Socket
- added J6: 0V, Connector_PinSocket_2.54mm:PinSocket_1x01_P2.54mm_Vertical, symbol Connector:Conn_01x01_Socket
- added J8: P+, Connector_PinSocket_2.54mm:PinSocket_1x01_P2.54mm_Vertical, symbol Connector:Conn_01x01_Socket
- added R1, R2: 4.7k, Resistor_THT:R_Axial_DIN0207_L6.3mm_D2.5mm_P7.62mm_Horizontal, symbol Device:R
- added R11, R13, R15, R17, R19, R21, R3: 10K, Resistor_SMD:R_0603_1608Metric, symbol Device:R
- added R12, R20, R22: 13k, Resistor_SMD:R_0603_1608Metric, symbol Device:R
- added R14: 1.5K, Resistor_SMD:R_0603_1608Metric, symbol Device:R
- added R16: 2k, Resistor_SMD:R_0603_1608Metric, symbol Device:R
- added R18: 1.2K, Resistor_SMD:R_0603_1608Metric, symbol Device:R
- added R4: 20k, Resistor_SMD:R_0603_1608Metric, symbol Device:R
- added SW2, SW3: SW_SPST, Button_Switch_THT:SW_DIP_SPSTx01_Slide_9.78x4.72mm_W7.62mm_P2.54mm, symbol Switch:SW_SPST
Connections:
- net +3.3V: now also J38.1 (Pin_1), J39.2 (Pin_2), R3.1
- net +5V: now also J32.1 (Pin_1), J33.1 (Pin_1), J35.1 (Pin_1), J45.18 (Pin_18), R11.1
- net 3V3_INPUT: now also J40.6 (Pin_6), R3.2, R4.1
- net 5V_INPUT: now also J40.7 (Pin_7), R11.2, R12.1
- net BATT_INPUT: now also J40.9 (Pin_9), R15.2, R16.1
- net DC_INPUT: now also J40.8 (Pin_8), R13.2, R14.1
- net GND: now also D1.1 (K), D4.1 (K), J26.1 (Pin_1), J29.1 (Pin_1), J31.1 (Pin_1), J32.2 (Pin_2), J34.1 (Pin_1), J35.2 (Pin_2), J38.2 (Pin_2), J39.1 (Pin_1), J45.19 (Pin_19), R12.2, R14.2, R16.2, R18.2, R20.2, R22.2, R4.2
- net SOLAR_INPUT: now also J40.10 (Pin_10), R17.2, R18.1
- new net: D1.2 (A), R1.2
- new net: D2.2 (A), J28.1 (Pin_1)
- new net: D4.2 (A), R2.2
- new net: D5.1 (K), D6.1 (K), J24.1 (Pin_1)
- new net 3V3: J40.18 (Pin_18), J45.20 (Pin_20)
- new net 5V1: J36.3 (Pin_3), J37.3 (Pin_3), J40.20 (Pin_20)
- new net A10: J45.7 (Pin_7)
- new net A11: J45.8 (Pin_8)
- new net A12: J45.9 (Pin_9)
- new net A15: J45.10 (Pin_10)
- new net A7: J40.13 (Pin_13)
- new net A8: J45.5 (Pin_5)
- new net A9: J45.6 (Pin_6)
- new net B+: J4.4 (Pin_4), J7.1 (Pin_1)
- new net B-: J4.1 (Pin_1), J6.1 (Pin_1)
- new net B0: J40.14 (Pin_14)
- new net B1: J27.1 (Pin_1), J4.2 (Pin_2), J40.15 (Pin_15)
- new net B10: J40.17 (Pin_17)
- new net B12: J45.1 (Pin_1)
- new net B13: J45.2 (Pin_2)
- new net B14: J45.3 (Pin_3)
- new net B15: J45.4 (Pin_4)
- new net B2: J4.3 (Pin_3), J40.16 (Pin_16), J5.1 (Pin_1)
- new net B3: J45.11 (Pin_11)
- new net B4: J45.12 (Pin_12)
- new net B5: J45.13 (Pin_13)
- new net B8: J45.16 (Pin_16)
- new net B9: J45.17 (Pin_17)
- new net BATT2_INPUT: J40.11 (Pin_11), R19.2, R20.1
- new net BATT2_TEST: J37.2 (Pin_2), R19.1
- new net BATT_TEST: J43.1 (Pin_1), R1.1, R15.1
- new net BMS_P+: D2.1 (K), J30.1 (Pin_1), J44.1 (Pin_1), J8.1 (Pin_1), R2.1
- new net C13: J40.2 (Pin_2)
- new net C14: J40.3 (Pin_3)
- new net C15: J40.4 (Pin_4)
- new net DC+: J23.2 (Pin_2), SW2.1 (A)
- new net DC-: J22.1 (Pin_1), J23.1 (Pin_1), J25.1 (Pin_1)
- new net DCJACK_TEST: D6.2 (A), R13.1, SW2.2 (B)
- new net GND1: J36.1 (Pin_1), J37.1 (Pin_1), J40.19 (Pin_19)
- new net IP+1: J42.1 (Pin_1), R17.1, SW3.2 (B)
- new net IP-1: D5.2 (A), J41.1 (Pin_1)
- new net R: J40.5 (Pin_5)
- new net S+: J22.2 (Pin_2), SW3.1 (A)
- new net SCL: J45.14 (Pin_14), J46.2 (Pin_2)
- new net SDA: J45.15 (Pin_15), J46.1 (Pin_1)
- new net SOLAR2_INPUT: J40.12 (Pin_12), R21.2, R22.1
- new net SOLAR2_TEST: J36.2 (Pin_2), R21.1
- new net VB: J40.1 (Pin_1)
- no-connect marks 0 -> 29
Other:
- note added: "5V - 3.3V LDO"
- note added: "A0"
- note added: "A1"
- note added: "A2"
- note added: "A3"
- note added: "A4"
- note added: "A5"
- note added: "A6"
- note added: "ACS712_MODULE"
- note added: "BATTERY INPUT AND BMS_MODULE"
- note added: "BMS_3S30A_MODULE"
- note added: "CN4015-2_MODULE"
- note added: "CURRENT SENSORS"
- note added: "GND"
- note added: "HW122_MODULE"
- note added: "Inputs connected through an OR-ing circuit in case the user accidentally turns both switches on at the same time"
- note added: "OUT"
- note added: "SOLAR INPUT AND BUCK_CONVERTER"
- note added: "STM32F401_MODULE"
- note added: "VCC"
- note added: "VOLTAGE DIVIDERS"
- note removed: "12V - 5V converter"
- note removed: "12V / 16v output"
- note removed: "3A 3.3V LDO"
- note removed: "BOOT AND RESET OPTION"
- note removed: "DC in 17.5 - 19V"
- note removed: "JTAG PROGRAMING"
- note removed: "MPPT SOLAR CHARGE CONTROLLER"
- note removed: "POWER MULTIPLEXER"
- note removed: "TO BMS"
- note removed: "UART PROGRAMING"
- note removed: "bms can be 3S /4S"
- note removed: "boot and reset is active low,"
- note removed: "for setting battery output voltage"
- note removed: "for setting input voltage"
- note removed: "input power must be >15v"
- note removed: "power indication led"
- note removed: "solar no load voltage 22V MP 17.5V"
