File: KiCAD FILES__PCB/aws.kicad_pcb (KiCad board)
At the start: 2 copper layers, 214.9 x 91.5 mm, 33 parts, among them J17 B4B-XH-A_LF__SN_, J20 B3B-XH-A_LF__SN_, J21 B3B-XH-A_LF__SN_, J25 Screw_Terminal_01x02, J26 Screw_Terminal_01x02, J27 Screw_Terminal_01x02, J28 B4B-XH-A_LF__SN_, J3 B3B-XH-A_LF__SN_, J32 B3B-XH-A_LF__SN_, J37 B3B-XH-A_LF__SN_, J39 Conn_01x02_Pin, SW6 SW_SPST

Commit message: Finished the gateway schematic and pcb successfully
Parts:
- removed the ? at (152.6, 123.1)
- removed the ? at (109.0, 41.0)
- removed the ? at (106.5, 41.0)
- removed the ? at (111.5, 41.0)
- removed the ? at (104.0, 41.0)
- removed J17, J28: B4B-XH-A_LF__SN_, B4B-XH-A_LF__SN_:JST_B4B-XH-A_LF__SN_
- removed J20, J21, J32, J37: B3B-XH-A_LF__SN_, B3B-XH-A_LF__SN_:JST_B3B-XH-A_LF__SN_
- removed J25 (x3), J26 (x6), J27: Screw_Terminal_01x02, TerminalBlock_MetzConnect:TerminalBlock_MetzConnect_Type011_RT05502HBWC_1x02_P5.00mm_Horizontal
- removed J39: Conn_01x02_Pin, Connector_PinHeader_2.54mm:PinHeader_1x02_P2.54mm_Vertical
- removed the REF** at (133.7, 123.3)
- removed the REF** at (133.7, 42.1)
- removed the REF** at (245.6, 123.1)
- removed the REF** at (40.7, 123.3)
- removed the REF** at (152.6, 123.1)
- removed the REF** at (245.6, 41.9)
- removed the REF** at (152.6, 41.9)
- removed the REF** at (40.7, 42.1)
- removed SW6 (x2): SW_SPST, Button_Switch_THT:SW_DIP_SPSTx01_Slide_9.78x4.72mm_W7.62mm_P2.54mm
- added ?: , , F.Cu at (26.1, 39.7)
- added C1: 10uF, Capacitor_SMD:C_0402_1005Metric_Pad0.74x0.62mm_HandSolder, F.Cu at (74.3, 64.9)
- added C2: 0.1uF, Capacitor_SMD:C_0402_1005Metric_Pad0.74x0.62mm_HandSolder, F.Cu at (92.3, 64.9)
- added J1: GSM, Connector_PinSocket_2.54mm:PinSocket_1x07_P2.54mm_Vertical, F.Cu at (33.8, 56.6)
- added J10: RAINFALL SENSOR, TerminalBlock_Phoenix:TerminalBlock_Phoenix_MKDS-3-2-5.08_1x02_P5.08mm_Horizontal, F.Cu at (141.6, 139.4)
- added J11: SOIL MOISTURE, TerminalBlock_Phoenix:TerminalBlock_Phoenix_MKDS-3-3-5.08_1x03_P5.08mm_Horizontal, F.Cu at (42.7, 139.9)
- added J12: SOIL TEMP, TerminalBlock_Phoenix:TerminalBlock_Phoenix_MKDS-3-3-5.08_1x03_P5.08mm_Horizontal, F.Cu at (51.1, 139.9)
- added J13: DHT 22, TerminalBlock_Phoenix:TerminalBlock_Phoenix_MKDS-3-3-5.08_1x03_P5.08mm_Horizontal, F.Cu at (69.8, 139.9)
- added J14: SH25, TerminalBlock_Phoenix:TerminalBlock_Phoenix_MKDS-3-4-5.08_1x04_P5.08mm_Horizontal, F.Cu at (28.6, 129.9)
- added J15: ATM PRESSURE, TerminalBlock_Phoenix:TerminalBlock_Phoenix_MKDS-3-4-5.08_1x04_P5.08mm_Horizontal, F.Cu at (28.5, 106.9)
- added J16: WIND VANE, TerminalBlock_Phoenix:TerminalBlock_Phoenix_MKDS-3-3-5.08_1x03_P5.08mm_Horizontal, F.Cu at (87.7, 139.9)
- added J4: SD_CARD, Connector_PinSocket_2.54mm:PinSocket_1x06_P2.54mm_Vertical, F.Cu at (128.6, 105.5)
- added J5: Conn_01x09_Socket, Connector_PinSocket_2.54mm:PinSocket_1x09_P2.54mm_Vertical, F.Cu at (103.9, 39.0)
- added J6: Conn_01x09_Socket, Connector_PinSocket_2.54mm:PinSocket_1x09_P2.54mm_Vertical, F.Cu at (131.8, 39.0)
- added J7: I2C, TerminalBlock_Phoenix:TerminalBlock_Phoenix_MKDS-3-2-5.08_1x02_P5.08mm_Horizontal, F.Cu at (121.3, 139.9)
- added J8: WIND SPEED, TerminalBlock_Phoenix:TerminalBlock_Phoenix_MKDS-3-2-5.08_1x02_P5.08mm_Horizontal, F.Cu at (154.9, 138.9)
- added J9: LIGHT INTENSITY, TerminalBlock_Phoenix:TerminalBlock_Phoenix_MKDS-3-2-5.08_1x02_P5.08mm_Horizontal, F.Cu at (106.7, 139.4)
- added R10: 4.7k, Resistor_THT:R_Axial_DIN0207_L6.3mm_D2.5mm_P7.62mm_Horizontal, F.Cu at (55.4, 116.2)
- added R5: 4.7k, Resistor_THT:R_Axial_DIN0207_L6.3mm_D2.5mm_P7.62mm_Horizontal, F.Cu at (116.4, 85.9)
- added R6: 4.7k, Resistor_THT:R_Axial_DIN0207_L6.3mm_D2.5mm_P7.62mm_Horizontal, F.Cu at (116.4, 100.9)
- added R7: 1k, Resistor_THT:R_Axial_DIN0207_L6.3mm_D2.5mm_P7.62mm_Horizontal, F.Cu at (116.9, 115.2)
- added R8: 2k, Resistor_THT:R_Axial_DIN0207_L6.3mm_D2.5mm_P7.62mm_Horizontal, F.Cu at (55.4, 87.8)
- added R9: 4.7k, Resistor_THT:R_Axial_DIN0207_L6.3mm_D2.5mm_P7.62mm_Horizontal, F.Cu at (55.4, 103.2)
- added REF**: MountingHole_3.2mm_M3_Pad_Via, MountingHole:MountingHole_3.2mm_M3_Pad_Via, F.Cu at (24.5, 140.2)
- added REF**: MountingHole_3.2mm_M3_Pad_Via, MountingHole:MountingHole_3.2mm_M3_Pad_Via, F.Cu at (165.7, 39.2)
- added REF**: MountingHole_3.2mm_M3_Pad_Via, MountingHole:MountingHole_3.2mm_M3_Pad_Via, F.Cu at (167.2, 141.7)
- added U1: ESP32-DEVKITC-32U, ESP32devkit:MODULE_ESP32-DEVKITC-32U, F.Cu at (86.2, 98.6)
- J3: value B3B-XH-A_LF__SN_ -> RTC_MODULE; footprint B3B-XH-A_LF__SN_:JST_B3B-XH-A_LF__SN_ -> Connector_PinSocket_2.54mm:PinSocket_1x06_P2.54mm_Vertical
- moved J3 89.6 mm to (129.3, 90.5), turned to 180 degrees
Connections:
- J3 pad 1: /gate way/DAVIS 7852 -> unconnected-(J3-Pin_1-Pad1)
- J3 pad 2: GND -> unconnected-(J3-Pin_2-Pad2)
- J3 pad 3: GND -> G21
Routing:
- net GND: track 6.56 -> 579.4 mm, vias 72 -> 2
- net +3V3: track 0.00 -> 236.7 mm
- net +5V: track 0.00 -> 210.1 mm
- net G22: track 0.00 -> 207.8 mm, vias 0 -> 2
- net G21: track 0.00 -> 201.2 mm, vias 0 -> 6
- net G16: track 0.00 -> 137.1 mm, vias 0 -> 2
- net G35: track 0.00 -> 115.5 mm, vias 0 -> 2
- net G17: track 0.00 -> 101.4 mm, vias 0 -> 4
- net G14: track 0.00 -> 92.8 mm, vias 0 -> 3
- net GSM_RST: track 0.00 -> 92.7 mm
- net G12: track 0.00 -> 80.0 mm, vias 0 -> 2
- net G27: track 0.00 -> 78.7 mm, vias 0 -> 2
- net G15: track 0.00 -> 74.3 mm, vias 0 -> 3
- net 5V: track 0.00 -> 68.0 mm
- net Net-(J26-Pin_2): track 66.7 -> 0.00 mm
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Other:
- board size 214.9 x 91.5 mm -> 153.6 x 115.1 mm
- board text added: "ATM_PRESSURE"
- board text added: "CS"
- board text added: "ESP_32_MODULE"
- board text added: "GSM_MODULE"
- board text added: "LIGHT_SENSOR"
- board text added: "LoRa_MODULE"
- board text added: "MOSI"
- board text added: "RAIN_SENSOR"
- board text added: "RTC_MODULE"
- board text added: "SCL"
- board text added: "SD_CARD_MODULE"
- board text added: "SOIL_MOISTURE"
- board text added: "SQW"
- board text added: "VCC"
- board text added: "WIND_SPEED"
- board text added: "WIND_VANE"
- board text removed: "+"
- board text removed: "3.3V"
- board text removed: "3V"
- board text removed: "5V"
- board text removed: "ATM PRESSSURE"
- board text removed: "AWS Gen4 V1, 2025"
- board text removed: "BATTERY PACK 3S@12V /4S@16V"
- board text removed: "DC INPUT 19V"
- board text removed: "DHT22"
- board text removed: "G"
- board text removed: "GATE WAY BOARD"
- board text removed: "I2C"
- board text removed: "LIGHT INTENSITY"
- board text removed: "POWER"
- board text removed: "POWER BOARD"
- board text removed: "RAINFALL"
- board text removed: "SHT25"
- board text removed: "SOIL MOISTURE"
- board text removed: "SOIL TEMP"
- board text removed: "SOLAR INPUT 17.5V"
- board text removed: "WIND VANE"
- board text removed: "www.ademnea.net"
- board text removed: "www.iot-ra.net"
