File: KiCAD FILES_PCB/.history/AWS PROJECT.kicad_sch (KiCad schematic)
At the start: 0 parts

Commit message: Updated gateway board PCB
Other:
- title: GENERAL  DESIGN SHEET -> POWER SCHEMATIC
Changed lines of the file:
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@@
 	(paper "A4")
 	(title_block
-		(title "GENERAL  DESIGN SHEET")
+		(title "POWER SCHEMATIC")
+		(date "2026-07-05")
 		(company "AdeMNEA IoT-ra")
-		(comment 1 "Designed By TN Muhanguzi")
+		(comment 1 "Designed By Edrine Ssennungi")
 		(comment 2 "For MPSE Research at Makerere University")
 	)
