File: KiCAD FILES_PCB/.history/AWS PROJECT.kicad_pcb (KiCad board)
At the start: 2 copper layers, 103 x 91.2 mm, 39 parts, among them J1 Real Time Clock, J10 WIND VANE, J11 SD CARD, J12 SOIL TEMP, J13 DHT 22, J14 SH25, J15 ATM PRESSURE, J16 SOIL MOISTURE, J2 GSM, J3 Conn_Coaxial, J6 I2C, J7 WIND SPEED, J8 LIGHT INTENSITY, J9 RAINFALL SENSOR, SW1 SW_Push, SW2 SW_Push, U1 ESP32-DEVKITC-32U, U10 AMS1117-3.3

Commit message: Updated gateway board PCB
Parts:
- removed C3: 10uF, Capacitor_THT:CP_Radial_D10.0mm_P7.50mm
- removed C4: 22uF, Capacitor_THT:CP_Radial_D10.0mm_P7.50mm
- removed C5, C6: 100n, Capacitor_THT:CP_Radial_D10.0mm_P7.50mm
- removed C7, C8: 10pF, Capacitor_SMD:C_0402_1005Metric_Pad0.74x0.62mm_HandSolder
- removed J3: Conn_Coaxial, Connector_Coaxial:U.FL_Molex_MCRF_73412-0110_Vertical
- removed R10: 4.7k, Resistor_SMD:R_0805_2012Metric
- removed R11: 2k, Resistor_SMD:R_0805_2012Metric
- removed SW1, SW2: SW_Push, Button_Switch_THT:SW_PUSH_6mm_H4.3mm
- removed U10: AMS1117-3.3, Package_TO_SOT_SMD:SOT-223-3_TabPin2
- added D1: RED, LED_SMD:LED_0402_1005Metric, F.Cu at (56.3, 51.1)
- added D2: YELLOW, LED_SMD:LED_0402_1005Metric, F.Cu at (56.3, 56.3)
- added J17: +3.3V, TerminalBlock_Phoenix:TerminalBlock_Phoenix_MKDS-1-2-3.81_1x02_P3.81mm_Horizontal, F.Cu at (86.0, 140.0)
- added J18: +5V, TerminalBlock_Phoenix:TerminalBlock_Phoenix_MKDS-1-2-3.81_1x02_P3.81mm_Horizontal, F.Cu at (70.0, 140.2)
- added REF**: MountingHole_3.2mm_M3_Pad_Via, MountingHole:MountingHole_3.2mm_M3_Pad_Via, F.Cu at (275.3, 140.9)
- added REF**: MountingHole_3.2mm_M3_Pad_Via, MountingHole:MountingHole_3.2mm_M3_Pad_Via, F.Cu at (16.4, 37.1)
- added REF**: MountingHole_3.2mm_M3_Pad_Via, MountingHole:MountingHole_3.2mm_M3_Pad_Via, F.Cu at (156.5, 140.9)
- added REF**: MountingHole_3.2mm_M3_Pad_Via, MountingHole:MountingHole_3.2mm_M3_Pad_Via, F.Cu at (156.5, 37.1)
- added REF**: MountingHole_3.2mm_M3_Pad_Via, MountingHole:MountingHole_3.2mm_M3_Pad_Via, F.Cu at (135.2, 140.9)
- added REF**: MountingHole_3.2mm_M3_Pad_Via, MountingHole:MountingHole_3.2mm_M3_Pad_Via, F.Cu at (275.3, 37.1)
- added REF**: MountingHole_3.2mm_M3_Pad_Via, MountingHole:MountingHole_3.2mm_M3_Pad_Via, F.Cu at (135.2, 37.1)
- added REF**: MountingHole_3.2mm_M3_Pad_Via, MountingHole:MountingHole_3.2mm_M3_Pad_Via, F.Cu at (16.4, 140.9)
- C1, C2: footprint Capacitor_THT:CP_Radial_D10.0mm_P7.50mm -> Capacitor_THT:CP_Radial_D4.0mm_P2.00mm
- J1, J11: footprint Connector_Molex:Molex_SPOX_5267-06A_1x06_P2.50mm_Vertical -> Connector_Molex:Molex_SL_171971-0006_1x06_P2.54mm_Vertical
- J2: footprint Connector_Molex:Molex_SPOX_5267-07A_1x07_P2.50mm_Vertical -> Connector_Molex:Molex_SL_171971-0007_1x07_P2.54mm_Vertical
- J4: value (none) -> Conn_01x09_Socket
- J5: value (none) -> Conn_01x08_Socket; footprint Connector_PinSocket_2.54mm:PinSocket_1x09_P2.54mm_Vertical -> Connector_PinSocket_2.54mm:PinSocket_1x08_P2.54mm_Vertical
- R1: value 10k -> 4.7k; footprint Resistor_THT:R_Axial_DIN0204_L3.6mm_D1.6mm_P5.08mm_Horizontal -> Resistor_THT:R_Axial_DIN0204_L3.6mm_D1.6mm_P7.62mm_Horizontal
- R2: value 100R -> 4.7k; footprint Resistor_THT:R_Axial_DIN0204_L3.6mm_D1.6mm_P5.08mm_Horizontal -> Resistor_THT:R_Axial_DIN0204_L3.6mm_D1.6mm_P7.62mm_Horizontal
- R3: value 10k -> 1k; footprint Resistor_THT:R_Axial_DIN0204_L3.6mm_D1.6mm_P5.08mm_Horizontal -> Resistor_THT:R_Axial_DIN0204_L3.6mm_D1.6mm_P7.62mm_Horizontal
- R4: value 0R -> 2k; footprint Resistor_SMD:R_0805_2012Metric -> Resistor_THT:R_Axial_DIN0204_L3.6mm_D1.6mm_P7.62mm_Horizontal
- R5, R6: footprint Resistor_SMD:R_0805_2012Metric -> Resistor_THT:R_Axial_DIN0204_L3.6mm_D1.6mm_P7.62mm_Horizontal
- R7: value 1k -> 2k; footprint Resistor_SMD:R_0805_2012Metric -> Resistor_THT:R_Axial_DIN0204_L3.6mm_D1.6mm_P7.62mm_Horizontal
- R8: value 2k -> 0.47k; footprint Resistor_SMD:R_0805_2012Metric -> Resistor_THT:R_Axial_DIN0204_L3.6mm_D1.6mm_P7.62mm_Horizontal
- R9: value 4.7k -> 1k; footprint Resistor_SMD:R_0805_2012Metric -> Resistor_THT:R_Axial_DIN0204_L3.6mm_D1.6mm_P7.62mm_Horizontal
- moved J1 108.7 mm to (51.8, 128.2)
- moved J11 108.2 mm to (50.1, 101.1)
- moved J14 85.7 mm to (134.7, 80.2), turned to 90 degrees
- moved J4 81.8 mm to (21.0, 54.8)
- moved J5 81.4 mm to (48.9, 57.3)
- moved J13 70.3 mm to (115.8, 37.7), turned to 180 degrees
- moved J12 68.3 mm to (101.2, 37.3), turned to 180 degrees
- moved R8 67.7 mm to (64.3, 50.7)
- moved C2 66.7 mm to (65.7, 118.2)
- moved R9 65.4 mm to (64.3, 56.9)
- moved J9 59.5 mm to (35.1, 37.6), turned to 180 degrees
- moved J15 58.9 mm to (135.2, 100.7), turned to 90 degrees
- moved J16 54.3 mm to (134.5, 60.7)
- moved C1 52.7 mm to (65.6, 127.5)
- moved J6 34.8 mm to (73.1, 37.5), turned to 180 degrees
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Connections:
- J2 pad 1: unconnected-(J2-Pin_1-Pad1) -> GSM_RST
- J2 pad 7: 5V -> +5V
- J5 pad 1: ANT -> G14
- J5 pad 2: GND -> G15
- J5 pad 3: RST -> unconnected-(J5-Pin_3-Pad3)
- J5 pad 4: I02 -> unconnected-(J5-Pin_4-Pad4)
- J5 pad 8: G15 -> GND
- R1 pad 1: Net-(R1-Pad1) -> G12
- R1 pad 2: GND -> +3.3V
- R2 pad 1: Net-(R1-Pad1) -> G35
- R2 pad 2: I02 -> +3.3V
- R3 pad 1: +3.3V -> Net-(J10-Pin_2)
- R3 pad 2: RST -> G27
- R4 pad 1: ANT -> G27
- R4 pad 2: Net-(J3-In) -> GND
- R5 pad 1: G12 -> G21
- R6 pad 1: G35 -> G22
- R7 pad 1: Net-(J10-Pin_2) -> +5V
- R7 pad 2: G27 -> G33
- R8 pad 1: G27 -> +3.3V
- R8 pad 2: GND -> Net-(D1-A)
- R9 pad 1: G21 -> G15
- R9 pad 2: +3.3V -> Net-(D2-A)
- U1 pad 15: unconnected-(U1-IO13-Pad15) -> GSM_RST
Routing:
- net GND: track 0.00 -> 517.5 mm
- net +3.3V: track 0.00 -> 301.5 mm, vias 0 -> 1
- net +5V: track 0.00 -> 266.0 mm, vias 0 -> 3
- net G22: track 0.00 -> 208.6 mm, vias 0 -> 2
- net G21: track 0.00 -> 197.3 mm, vias 0 -> 1
- net G12: track 0.00 -> 118.5 mm, vias 0 -> 2
- net G35: track 0.00 -> 113.0 mm, vias 0 -> 3
- net G34: track 0.00 -> 104.0 mm, vias 0 -> 3
- net G33: track 0.00 -> 101.0 mm, vias 0 -> 2
- net G15: track 0.00 -> 72.0 mm
- net GSM_RST: track 0.00 -> 67.1 mm, vias 0 -> 1
- net G5: track 0.00 -> 63.2 mm
- net G27: track 0.00 -> 57.6 mm, vias 0 -> 1
- net Net-(J10-Pin_2): track 0.00 -> 56.2 mm, vias 0 -> 2
- net G23: track 0.00 -> 51.0 mm
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- added copper zone on B.Cu, net GND
- added copper zone on F.Cu, net GND
Other:
- board size 103 x 91.2 mm -> 271.8 x 116.6 mm
- board text added: "+3.3V"
- board text added: "+5V"
- board text added: "ESP32-DEVKIT"
- board text added: "GATE WAY BOARD"
- board text added: "RAINFALL"
- board text removed: "LDO"
- board text removed: "RAINFALL_SENSOR"

Commit message: Updated LED footprints to THT
Parts:
- added D3: LED, LED_THT:LED_D5.0mm, F.Cu at (221.0, 105.3)
- added D4: 1N5822, Diode_THT:D_DO-201AD_P12.70mm_Horizontal, F.Cu at (203.5, 105.0)
- added D5: 1N5822, Diode_THT:D_DO-201AD_P12.70mm_Horizontal, F.Cu at (203.5, 111.7)
- added D6: 1N5822, Diode_THT:D_DO-201AD_P12.70mm_Horizontal, F.Cu at (203.5, 118.5)
- added D7: LED, LED_THT:LED_D5.0mm, F.Cu at (221.0, 112.8)
- added J19: SOLAR_INPUT, TerminalBlock_MetzConnect:TerminalBlock_MetzConnect_Type055_RT01502HDWU_1x02_P5.00mm_Horizontal, F.Cu at (192.6, 63.9)
- added J20: 8.4V, Connector_PinSocket_2.54mm:PinSocket_1x01_P2.54mm_Vertical, F.Cu at (225.0, 61.2)
- added J21: 0V, Connector_PinSocket_2.54mm:PinSocket_1x01_P2.54mm_Vertical, F.Cu at (225.0, 65.8)
- added J22: IN+, Connector_PinSocket_2.54mm:PinSocket_1x01_P2.54mm_Vertical, F.Cu at (225.0, 70.4)
- added J23: DCJACK_INPUT, TerminalBlock_MetzConnect:TerminalBlock_MetzConnect_Type055_RT01502HDWU_1x02_P5.00mm_Horizontal, F.Cu at (192.6, 74.2)
- added J24: IN-, Connector_PinSocket_2.54mm:PinSocket_1x01_P2.54mm_Vertical, F.Cu at (225.0, 75.0)
- added J25: 12.6V, Connector_PinSocket_2.54mm:PinSocket_1x01_P2.54mm_Vertical, F.Cu at (225.0, 79.6)
- added J26: P+, Connector_PinSocket_2.54mm:PinSocket_1x01_P2.54mm_Vertical, F.Cu at (225.0, 84.1)
- added J27: P-, Connector_PinSocket_2.54mm:PinSocket_1x01_P2.54mm_Vertical, F.Cu at (229.6, 61.2)
- added J28: 4.2V, Connector_PinSocket_2.54mm:PinSocket_1x01_P2.54mm_Vertical, F.Cu at (229.6, 65.8)
- added J29: OUT+, Connector_PinSocket_2.54mm:PinSocket_1x01_P2.54mm_Vertical, F.Cu at (229.6, 70.4)
- added J3: BATTERY_INPUT, TerminalBlock_MetzConnect:TerminalBlock_MetzConnect_Type055_RT01504HDWU_1x04_P5.00mm_Horizontal, F.Cu at (204.7, 96.3)
- added J30: OUT-, Connector_PinSocket_2.54mm:PinSocket_1x01_P2.54mm_Vertical, F.Cu at (229.6, 75.0)
- added J31: IN+, Connector_PinSocket_2.54mm:PinSocket_1x01_P2.54mm_Vertical, F.Cu at (229.6, 79.6)
- added J32: IN-, Connector_PinSocket_2.54mm:PinSocket_1x01_P2.54mm_Vertical, F.Cu at (229.6, 84.1)
- added J33: 5V_OUTPUT, TerminalBlock_MetzConnect:TerminalBlock_MetzConnect_Type055_RT01502HDWU_1x02_P5.00mm_Horizontal, F.Cu at (192.6, 84.6)
- added J34: OUT+, Connector_PinSocket_2.54mm:PinSocket_1x01_P2.54mm_Vertical, F.Cu at (234.1, 61.2)
- added J35: OUT-, Connector_PinSocket_2.54mm:PinSocket_1x01_P2.54mm_Vertical, F.Cu at (234.1, 65.8)
- added J36: IN, Connector_PinSocket_2.54mm:PinSocket_1x02_P2.54mm_Vertical, F.Cu at (228.4, 116.7)
- added J37: Conn_01x03_Socket, Connector_PinSocket_2.54mm:PinSocket_1x03_P2.54mm_Vertical, F.Cu at (225.5, 93.6)
- added J38: Conn_01x03_Socket, Connector_PinSocket_2.54mm:PinSocket_1x03_P2.54mm_Vertical, F.Cu at (230.1, 93.6)
- added J39: 3.3V_OUTPUT, TerminalBlock_MetzConnect:TerminalBlock_MetzConnect_Type055_RT01502HDWU_1x02_P5.00mm_Horizontal, F.Cu at (192.6, 94.9)
- added J40: OUT, Connector_PinSocket_2.54mm:PinSocket_1x02_P2.54mm_Vertical, F.Cu at (232.9, 116.7)
- added J41: Conn_01x20_Socket, Connector_PinSocket_2.54mm:PinSocket_1x20_P2.54mm_Vertical, F.Cu at (182.2, 61.2)
- added J42: 12.6V, Connector_PinSocket_2.54mm:PinSocket_1x01_P2.54mm_Vertical, F.Cu at (234.1, 70.4)
- added J43: 12.6V, Connector_PinSocket_2.54mm:PinSocket_1x01_P2.54mm_Vertical, F.Cu at (234.1, 75.0)
- added J44: 12.6V, Connector_PinSocket_2.54mm:PinSocket_1x01_P2.54mm_Vertical, F.Cu at (234.1, 79.6)
- added J45: 12.6V, Connector_PinSocket_2.54mm:PinSocket_1x01_P2.54mm_Vertical, F.Cu at (234.1, 84.1)
- added J46: Conn_01x20_Socket, Connector_PinSocket_2.54mm:PinSocket_1x20_P2.54mm_Vertical, F.Cu at (186.8, 61.2)
- added J47: I2C, TerminalBlock_MetzConnect:TerminalBlock_MetzConnect_Type055_RT01502HDWU_1x02_P5.00mm_Horizontal, F.Cu at (192.6, 105.2)
- added R10: 4.7k, Resistor_THT:R_Axial_DIN0207_L6.3mm_D2.5mm_P7.62mm_Horizontal, F.Cu at (202.7, 60.9)
- added R11: 4.7k, Resistor_THT:R_Axial_DIN0207_L6.3mm_D2.5mm_P7.62mm_Horizontal, F.Cu at (202.7, 65.0)
- added R12: 10K, Resistor_THT:R_Axial_DIN0207_L6.3mm_D2.5mm_P7.62mm_Horizontal, F.Cu at (202.7, 69.0)
- added R13: 20k, Resistor_THT:R_Axial_DIN0207_L6.3mm_D2.5mm_P7.62mm_Horizontal, F.Cu at (202.7, 73.1)
- added R14: 10K, Resistor_THT:R_Axial_DIN0207_L6.3mm_D2.5mm_P7.62mm_Horizontal, F.Cu at (202.7, 77.1)
- added R15: 13k, Resistor_THT:R_Axial_DIN0207_L6.3mm_D2.5mm_P7.62mm_Horizontal, F.Cu at (202.7, 81.2)
- added R16: 10K, Resistor_THT:R_Axial_DIN0207_L6.3mm_D2.5mm_P7.62mm_Horizontal, F.Cu at (202.7, 85.2)
- added R17: 1.5K, Resistor_THT:R_Axial_DIN0207_L6.3mm_D2.5mm_P7.62mm_Horizontal, F.Cu at (202.7, 89.3)
- added R18: 10K, Resistor_THT:R_Axial_DIN0207_L6.3mm_D2.5mm_P7.62mm_Horizontal, F.Cu at (213.5, 60.9)
- added R19: 2k, Resistor_THT:R_Axial_DIN0207_L6.3mm_D2.5mm_P7.62mm_Horizontal, F.Cu at (213.5, 65.0)
- added R20: 10K, Resistor_THT:R_Axial_DIN0207_L6.3mm_D2.5mm_P7.62mm_Horizontal, F.Cu at (213.5, 69.0)
- added R21: 1.2K, Resistor_THT:R_Axial_DIN0207_L6.3mm_D2.5mm_P7.62mm_Horizontal, F.Cu at (213.5, 73.1)
- added R22: 10K, Resistor_THT:R_Axial_DIN0207_L6.3mm_D2.5mm_P7.62mm_Horizontal, F.Cu at (213.5, 77.1)
- added R23: 13k, Resistor_THT:R_Axial_DIN0207_L6.3mm_D2.5mm_P7.62mm_Horizontal, F.Cu at (213.5, 81.2)
- added R24: 10K, Resistor_THT:R_Axial_DIN0207_L6.3mm_D2.5mm_P7.62mm_Horizontal, F.Cu at (213.5, 85.2)
- added R25: 13k, Resistor_THT:R_Axial_DIN0207_L6.3mm_D2.5mm_P7.62mm_Horizontal, F.Cu at (213.5, 89.3)
- added SW2: SW_SPST, Button_Switch_THT:SW_DIP_SPSTx01_Slide_9.78x4.72mm_W7.62mm_P2.54mm, F.Cu at (228.0, 104.8)
- added SW3: SW_SPST, Button_Switch_THT:SW_DIP_SPSTx01_Slide_9.78x4.72mm_W7.62mm_P2.54mm, F.Cu at (228.0, 111.2)
Connections:
- J2 pad 7: +5V -> 5V
