File: KiCAD FILES_PCB/.history/gateway.kicad_sch (KiCad schematic)
At the start: 39 parts, among them J1 Real Time Clock, J10 WIND VANE, J11 SD CARD, J12 SOIL TEMP, J13 DHT 22, J14 SH25, J15 ATM PRESSURE, J16 SOIL MOISTURE, J2 GSM, J3 Conn_Coaxial, J4 Conn_01x09_Socket, J5 Conn_01x09_Socket, J6 I2C, J7 WIND SPEED, J8 LIGHT INTENSITY, J9 RAINFALL SENSOR, SW1 SW_Push, SW2 SW_Push, U1 ESP32-DEVKITC-32U, U10 AMS1117-3.3

Commit message: Updated gateway board PCB
Parts:
- removed C3: 10uF, Capacitor_THT:CP_Radial_D10.0mm_P7.50mm, symbol Device:C
- removed C4: 22uF, Capacitor_THT:CP_Radial_D10.0mm_P7.50mm, symbol Device:C
- removed C5, C6: 100n, Capacitor_THT:CP_Radial_D10.0mm_P7.50mm, symbol Device:C
- removed C7, C8: 10pF, Capacitor_SMD:C_0402_1005Metric_Pad0.74x0.62mm_HandSolder, symbol Device:C
- removed J3: Conn_Coaxial, Connector_Coaxial:U.FL_Molex_MCRF_73412-0110_Vertical, symbol Connector:Conn_Coaxial
- removed J5: Conn_01x09_Socket, Connector_PinSocket_2.54mm:PinSocket_1x09_P2.54mm_Vertical, symbol Connector:Conn_01x09_Socket
- removed R10: 4.7k, Resistor_SMD:R_0805_2012Metric, symbol Device:R
- removed R11: 2k, Resistor_SMD:R_0805_2012Metric, symbol Device:R
- removed SW1, SW2: SW_Push, Button_Switch_THT:SW_PUSH_6mm_H4.3mm, symbol Switch:SW_Push
- removed U10: AMS1117-3.3, Package_TO_SOT_SMD:SOT-223-3_TabPin2, symbol Regulator_Linear:AMS1117-3.3
- added D1: RED, LED_SMD:LED_0402_1005Metric, symbol Device:LED
- added D2: YELLOW, LED_SMD:LED_0402_1005Metric, symbol Device:LED
- added J17: +3.3V, TerminalBlock_Phoenix:TerminalBlock_Phoenix_MKDS-1-2-3.81_1x02_P3.81mm_Horizontal, symbol Connector:Screw_Terminal_01x02
- added J18: +5V, TerminalBlock_Phoenix:TerminalBlock_Phoenix_MKDS-1-2-3.81_1x02_P3.81mm_Horizontal, symbol Connector:Screw_Terminal_01x02
- added J5: Conn_01x08_Socket, Connector_PinSocket_2.54mm:PinSocket_1x08_P2.54mm_Vertical, symbol Connector:Conn_01x08_Socket
- C1, C2: footprint Capacitor_THT:CP_Radial_D10.0mm_P7.50mm -> Capacitor_THT:CP_Radial_D4.0mm_P2.00mm
- J1, J11: footprint Connector_Molex:Molex_SPOX_5267-06A_1x06_P2.50mm_Vertical -> Connector_Molex:Molex_SL_171971-0006_1x06_P2.54mm_Vertical
- J2: footprint Connector_Molex:Molex_SPOX_5267-07A_1x07_P2.50mm_Vertical -> Connector_Molex:Molex_SL_171971-0007_1x07_P2.54mm_Vertical
- R1: value 10k -> 4.7k; footprint Resistor_THT:R_Axial_DIN0204_L3.6mm_D1.6mm_P5.08mm_Horizontal -> Resistor_THT:R_Axial_DIN0204_L3.6mm_D1.6mm_P7.62mm_Horizontal
- R2: value 100R -> 4.7k; footprint Resistor_THT:R_Axial_DIN0204_L3.6mm_D1.6mm_P5.08mm_Horizontal -> Resistor_THT:R_Axial_DIN0204_L3.6mm_D1.6mm_P7.62mm_Horizontal
- R3: value 10k -> 1k; footprint Resistor_THT:R_Axial_DIN0204_L3.6mm_D1.6mm_P5.08mm_Horizontal -> Resistor_THT:R_Axial_DIN0204_L3.6mm_D1.6mm_P7.62mm_Horizontal
- R4: value 0R -> 2k; footprint Resistor_SMD:R_0805_2012Metric -> Resistor_THT:R_Axial_DIN0204_L3.6mm_D1.6mm_P7.62mm_Horizontal
- R5, R6: footprint Resistor_SMD:R_0805_2012Metric -> Resistor_THT:R_Axial_DIN0204_L3.6mm_D1.6mm_P7.62mm_Horizontal
- R7: value 1k -> 2k; footprint Resistor_SMD:R_0805_2012Metric -> Resistor_THT:R_Axial_DIN0204_L3.6mm_D1.6mm_P7.62mm_Horizontal
- R8: value 2k -> 0.47k; footprint Resistor_SMD:R_0805_2012Metric -> Resistor_THT:R_Axial_DIN0204_L3.6mm_D1.6mm_P7.62mm_Horizontal
- R9: value 4.7k -> 1k; footprint Resistor_SMD:R_0805_2012Metric -> Resistor_THT:R_Axial_DIN0204_L3.6mm_D1.6mm_P7.62mm_Horizontal
Connections:
- net ANT is gone; now on net G27: R4.1
- net I02 is gone; now on net +3.3V: R2.2
- net RST is gone; now on net G27: R3.2
- net +3.3V: now also R1.2, R8.1, J17.1 (Pin_1); no longer R3.1, R9.2
- net +5V: now also R7.1, J18.1 (Pin_1)
- net G12: now also R1.1; no longer R5.1
- net G14: now also J5.1 (Pin_1)
- net G15: now also R9.1, J5.2 (Pin_2)
- net G21: now also R5.1; no longer R9.1
- net G22: now also R6.1
- net G27: no longer R7.2, R8.1
- net G33: now also R7.2
- net G35: now also R2.1; no longer R6.1
- net GND: now also R4.2, D1.1 (K), D2.1 (K), J17.2 (Pin_2), J18.2 (Pin_2), J5.8 (Pin_8); no longer R1.2, R8.2
- net GSM_RST: now reaches U1.15 (IO13)
- net GSM_RST: now also J2.1 (Pin_1)
- net at J10.2 (Pin_2): now also R3.1; no longer R7.1
- new net: D2.2 (A), R9.2
- new net: D1.2 (A), R8.2
Other:
- note added: "3.3V SUPPLY"
- note added: "5V SUPPLY"
- note removed: "BOOT,ANT AND RESET BUTTONS"
- note removed: "LDO"
- title: GATEWAY BOARD -> POWER SCHEMATIC

Commit message: Updated LED footprints to THT
Parts:
- D1, D2: footprint LED_SMD:LED_0402_1005Metric -> LED_THT:LED_D3.0mm
Changed lines of the file:
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@@
 			)
 		)
-		(property "Footprint" "LED_SMD:LED_0402_1005Metric"
+		(property "Footprint" "LED_THT:LED_D3.0mm"
 			(at 152.4 330.2 0)
 			(hide yes)
@@
 			)
 		)
-		(property "Footprint" "LED_SMD:LED_0402_1005Metric"
+		(property "Footprint" "LED_THT:LED_D3.0mm"
 			(at 240.03 328.93 0)
 			(hide yes)
