File: KiCAD FILES_PCB/power.kicad_sch (KiCad schematic)
At the start: 0 parts

Commit message: Updated LED footprints to THT
Parts:
- added D3, D7: LED, LED_THT:LED_D5.0mm, symbol Device:LED
- added D4, D5, D6: 1N5822, Diode_THT:D_DO-201AD_P12.70mm_Horizontal, symbol Diode:1N5822
- added J19: SOLAR_INPUT, TerminalBlock_MetzConnect:TerminalBlock_MetzConnect_Type055_RT01502HDWU_1x02_P5.00mm_Horizontal, symbol Connector:Screw_Terminal_01x02
- added J20: 8.4V, Connector_PinSocket_2.54mm:PinSocket_1x01_P2.54mm_Vertical, symbol Connector:Conn_01x01_Socket
- added J21: 0V, Connector_PinSocket_2.54mm:PinSocket_1x01_P2.54mm_Vertical, symbol Connector:Conn_01x01_Socket
- added J22, J31: IN+, Connector_PinSocket_2.54mm:PinSocket_1x01_P2.54mm_Vertical, symbol Connector:Conn_01x01_Socket
- added J23: DCJACK_INPUT, TerminalBlock_MetzConnect:TerminalBlock_MetzConnect_Type055_RT01502HDWU_1x02_P5.00mm_Horizontal, symbol Connector:Screw_Terminal_01x02
- added J24, J32: IN-, Connector_PinSocket_2.54mm:PinSocket_1x01_P2.54mm_Vertical, symbol Connector:Conn_01x01_Socket
- added J25, J42, J43, J44, J45: 12.6V, Connector_PinSocket_2.54mm:PinSocket_1x01_P2.54mm_Vertical, symbol Connector:Conn_01x01_Socket
- added J26: P+, Connector_PinSocket_2.54mm:PinSocket_1x01_P2.54mm_Vertical, symbol Connector:Conn_01x01_Socket
- added J27: P-, Connector_PinSocket_2.54mm:PinSocket_1x01_P2.54mm_Vertical, symbol Connector:Conn_01x01_Socket
- added J28: 4.2V, Connector_PinSocket_2.54mm:PinSocket_1x01_P2.54mm_Vertical, symbol Connector:Conn_01x01_Socket
- added J29, J34: OUT+, Connector_PinSocket_2.54mm:PinSocket_1x01_P2.54mm_Vertical, symbol Connector:Conn_01x01_Socket
- added J3: BATTERY_INPUT, TerminalBlock_MetzConnect:TerminalBlock_MetzConnect_Type055_RT01504HDWU_1x04_P5.00mm_Horizontal, symbol Connector:Screw_Terminal_01x04
- added J30, J35: OUT-, Connector_PinSocket_2.54mm:PinSocket_1x01_P2.54mm_Vertical, symbol Connector:Conn_01x01_Socket
- added J33: 5V_OUTPUT, TerminalBlock_MetzConnect:TerminalBlock_MetzConnect_Type055_RT01502HDWU_1x02_P5.00mm_Horizontal, symbol Connector:Screw_Terminal_01x02
- added J36: IN, Connector_PinSocket_2.54mm:PinSocket_1x02_P2.54mm_Vertical, symbol Connector:Conn_01x02_Socket
- added J37, J38: Conn_01x03_Socket, Connector_PinSocket_2.54mm:PinSocket_1x03_P2.54mm_Vertical, symbol Connector:Conn_01x03_Socket
- added J39: 3.3V_OUTPUT, TerminalBlock_MetzConnect:TerminalBlock_MetzConnect_Type055_RT01502HDWU_1x02_P5.00mm_Horizontal, symbol Connector:Screw_Terminal_01x02
- added J40: OUT, Connector_PinSocket_2.54mm:PinSocket_1x02_P2.54mm_Vertical, symbol Connector:Conn_01x02_Socket
- added J41, J46: Conn_01x20_Socket, Connector_PinSocket_2.54mm:PinSocket_1x20_P2.54mm_Vertical, symbol Connector:Conn_01x20_Socket
- added J47: I2C, TerminalBlock_MetzConnect:TerminalBlock_MetzConnect_Type055_RT01502HDWU_1x02_P5.00mm_Horizontal, symbol Connector:Screw_Terminal_01x02
- added R10, R11: 4.7k, Resistor_THT:R_Axial_DIN0207_L6.3mm_D2.5mm_P7.62mm_Horizontal, symbol Device:R
- added R12, R14, R16, R18, R20, R22, R24: 10K, Resistor_THT:R_Axial_DIN0207_L6.3mm_D2.5mm_P7.62mm_Horizontal, symbol Device:R
- added R13: 20k, Resistor_THT:R_Axial_DIN0207_L6.3mm_D2.5mm_P7.62mm_Horizontal, symbol Device:R
- added R15, R23, R25: 13k, Resistor_THT:R_Axial_DIN0207_L6.3mm_D2.5mm_P7.62mm_Horizontal, symbol Device:R
- added R17: 1.5K, Resistor_THT:R_Axial_DIN0207_L6.3mm_D2.5mm_P7.62mm_Horizontal, symbol Device:R
- added R19: 2k, Resistor_THT:R_Axial_DIN0207_L6.3mm_D2.5mm_P7.62mm_Horizontal, symbol Device:R
- added R21: 1.2K, Resistor_THT:R_Axial_DIN0207_L6.3mm_D2.5mm_P7.62mm_Horizontal, symbol Device:R
- added SW2, SW3: SW_SPST, Button_Switch_THT:SW_DIP_SPSTx01_Slide_9.78x4.72mm_W7.62mm_P2.54mm, symbol Switch:SW_SPST
Connections:
- new net: D3.2 (A), R10.2
- new net: D4.2 (A), J29.1 (Pin_1)
- new net: D7.2 (A), R11.2
- new net: D5.2 (A), SW3.2 (B)
- new net +3.3V: J39.1 (Pin_1), J40.2 (Pin_2), R12.1
- new net +5V: J33.1 (Pin_1), J34.1 (Pin_1), J36.1 (Pin_1), J46.18 (Pin_18), R14.1
- new net 3V3-1: J41.18 (Pin_18)
- new net 3V3-2: J46.20 (Pin_20)
- new net 3V3_INPUT: J41.6 (Pin_6), R12.2, R13.1
- new net 5V1: J37.3 (Pin_3), J38.3 (Pin_3), J41.20 (Pin_20)
- new net 5V_INPUT: J41.7 (Pin_7), R14.2, R15.1
- new net A10: J46.7 (Pin_7)
- new net A11: J46.8 (Pin_8)
- new net A12: J46.9 (Pin_9)
- new net A15: J46.10 (Pin_10)
- new net A7: J41.13 (Pin_13)
- new net A8: J46.5 (Pin_5)
- new net A9: J46.6 (Pin_6)
- new net B+: J25.1 (Pin_1), J3.4 (Pin_4)
- new net B-: J21.1 (Pin_1), J3.1 (Pin_1)
- new net B0: J41.14 (Pin_14)
- new net B1: J28.1 (Pin_1), J3.2 (Pin_2)
- new net B10: J41.17 (Pin_17)
- new net B12: J46.1 (Pin_1)
- new net B13: J46.2 (Pin_2)
- new net B14: J46.3 (Pin_3)
- new net B15: J46.4 (Pin_4)
- new net B2: J20.1 (Pin_1), J3.3 (Pin_3)
- new net B3: J46.11 (Pin_11)
- new net B4: J46.12 (Pin_12)
- new net B5: J46.13 (Pin_13)
- new net B8: J46.16 (Pin_16)
- new net B9: J46.17 (Pin_17)
- new net BATT2_INPUT: J41.11 (Pin_11), R22.2, R23.1
- new net BATT2_TEST: J38.2 (Pin_2), R22.1
- new net BATT_INPUT: J41.9 (Pin_9), R18.2, R19.1
- new net BATT_TEST: J44.1 (Pin_1), R10.1, R18.1
- new net BMS_P+: D4.1 (K), J26.1 (Pin_1), J31.1 (Pin_1), J45.1 (Pin_1), R11.1
- new net C13: J41.2 (Pin_2)
- new net C14: J41.3 (Pin_3)
- new net C15: J41.4 (Pin_4)
- new net DC+: J23.2 (Pin_2), SW2.1 (A)
- new net DC-: J19.1 (Pin_1), J23.1 (Pin_1), J24.1 (Pin_1)
- new net DCJACK_TEST: D6.2 (A), R16.1, SW2.2 (B)
- new net DC_INPUT: J41.8 (Pin_8), R16.2, R17.1
- new net GND: D3.1 (K), D7.1 (K), J27.1 (Pin_1), J30.1 (Pin_1), J32.1 (Pin_1), J33.2 (Pin_2), J35.1 (Pin_1), J36.2 (Pin_2), J39.2 (Pin_2), J40.1 (Pin_1), J46.19 (Pin_19), R13.2, R15.2, R17.2, R19.2, R21.2, R23.2, R25.2
- new net GND1: J37.1 (Pin_1), J38.1 (Pin_1), J41.19 (Pin_19)
- new net IP+1: D5.1 (K), D6.1 (K), J43.1 (Pin_1), R20.1
- new net IP-1: J22.1 (Pin_1), J42.1 (Pin_1)
- new net R: J41.5 (Pin_5)
- new net S+: J19.2 (Pin_2), SW3.1 (A)
- new net SCL: J46.14 (Pin_14), J47.2 (Pin_2)
- new net SDA: J46.15 (Pin_15), J47.1 (Pin_1)
- new net SOLAR2_INPUT: J41.12 (Pin_12), R24.2, R25.1
- new net SOLAR2_TEST: J37.2 (Pin_2), R24.1
- new net SOLAR_INPUT: J41.10 (Pin_10), R20.2, R21.1
- new net VB: J41.1 (Pin_1)
- no-connect marks 0 -> 29
Other:
- note added: "12V - 5V BUCK CONVERTER"
- note added: "5V - 3.3V LDO"
- note added: "A0"
- note added: "A1"
- note added: "A2"
- note added: "A3"
- note added: "A4"
- note added: "A5"
- note added: "A6"
- note added: "ACS712_MODULE"
- note added: "B1"
- note added: "B2"
- note added: "BATTERY INPUT AND BMS_MODULE"
- note added: "BMS_3S30A_MODULE"
- note added: "CN4015-2_MODULE"
- note added: "CURRENT SENSORS"
- note added: "GND"
- note added: "HW122_MODULE"
- note added: "Inputs connected through an OR-ing circuit in case the user accidentally turns both switches on at the same time"
- note added: "MICROCONTROLLER SECTION"
- note added: "OUT"
- note added: "POWER BOARD"
- note added: "SOLAR INPUT AND BUCK_CONVERTER"
- note added: "STM32F401_MODULE"
- note added: "VCC"
- note added: "VOLTAGE DIVIDERS"
