File: KiCAD FILES_PCB/_restore_backup_2026-07-07T10-18-56-602/AWS PROJECT.kicad_pcb (KiCad board)
At the start: 2 copper layers, 271.8 x 116.6 mm, 92 parts, among them J1 Real Time Clock, J10 WIND VANE, J11 SD CARD, J12 SOIL TEMP, J13 DHT 22, J14 SH25, J15 ATM PRESSURE, J16 SOIL MOISTURE, J17 +3.3V, J18 +5V, J19 SOLAR_INPUT, J2 GSM, J20 8.4V, J21 0V, J22 IN+, J23 DCJACK_INPUT, J24 IN-, J25 12.6V, J26 P+, J27 P-, J28 4.2V, J29 OUT+, J3 BATTERY_INPUT, J30 OUT-, J31 IN+, J32 IN-, J33 5V_OUTPUT, J34 OUT+, J35 OUT-, J36 IN, J37 Conn_01x03_Socket, J38 Conn_01x03_Socket, J39 3.3V_OUTPUT, J4 Conn_01x09_Socket, J40 OUT, J41 Conn_01x20_Socket, J42 12.6V, J43 12.6V, J44 12.6V, J45 12.6V, J46 Conn_01x20_Socket, J47 I2C, J5 Conn_01x08_Socket, J6 I2C, J7 WIND SPEED, J8 LIGHT INTENSITY, J9 RAINFALL SENSOR, SW2 SW_SPST, SW3 SW_SPST, U1 ESP32-DEVKITC-32U

Commit message: Updated LED footprints to THT
Parts:
- removed D3, D7: LED, LED_THT:LED_D5.0mm
- removed D4, D5, D6: 1N5822, Diode_THT:D_DO-201AD_P12.70mm_Horizontal
- removed J19: SOLAR_INPUT, TerminalBlock_MetzConnect:TerminalBlock_MetzConnect_Type055_RT01502HDWU_1x02_P5.00mm_Horizontal
- removed J20: 8.4V, Connector_PinSocket_2.54mm:PinSocket_1x01_P2.54mm_Vertical
- removed J21: 0V, Connector_PinSocket_2.54mm:PinSocket_1x01_P2.54mm_Vertical
- removed J22, J31: IN+, Connector_PinSocket_2.54mm:PinSocket_1x01_P2.54mm_Vertical
- removed J23: DCJACK_INPUT, TerminalBlock_MetzConnect:TerminalBlock_MetzConnect_Type055_RT01502HDWU_1x02_P5.00mm_Horizontal
- removed J24, J32: IN-, Connector_PinSocket_2.54mm:PinSocket_1x01_P2.54mm_Vertical
- removed J25, J42, J43, J44, J45: 12.6V, Connector_PinSocket_2.54mm:PinSocket_1x01_P2.54mm_Vertical
- removed J26: P+, Connector_PinSocket_2.54mm:PinSocket_1x01_P2.54mm_Vertical
- removed J27: P-, Connector_PinSocket_2.54mm:PinSocket_1x01_P2.54mm_Vertical
- removed J28: 4.2V, Connector_PinSocket_2.54mm:PinSocket_1x01_P2.54mm_Vertical
- removed J29, J34: OUT+, Connector_PinSocket_2.54mm:PinSocket_1x01_P2.54mm_Vertical
- removed J3: BATTERY_INPUT, TerminalBlock_MetzConnect:TerminalBlock_MetzConnect_Type055_RT01504HDWU_1x04_P5.00mm_Horizontal
- removed J30, J35: OUT-, Connector_PinSocket_2.54mm:PinSocket_1x01_P2.54mm_Vertical
- removed J33: 5V_OUTPUT, TerminalBlock_MetzConnect:TerminalBlock_MetzConnect_Type055_RT01502HDWU_1x02_P5.00mm_Horizontal
- removed J36: IN, Connector_PinSocket_2.54mm:PinSocket_1x02_P2.54mm_Vertical
- removed J37, J38: Conn_01x03_Socket, Connector_PinSocket_2.54mm:PinSocket_1x03_P2.54mm_Vertical
- removed J39: 3.3V_OUTPUT, TerminalBlock_MetzConnect:TerminalBlock_MetzConnect_Type055_RT01502HDWU_1x02_P5.00mm_Horizontal
- removed J40: OUT, Connector_PinSocket_2.54mm:PinSocket_1x02_P2.54mm_Vertical
- removed J41, J46: Conn_01x20_Socket, Connector_PinSocket_2.54mm:PinSocket_1x20_P2.54mm_Vertical
- removed J47: I2C, TerminalBlock_MetzConnect:TerminalBlock_MetzConnect_Type055_RT01502HDWU_1x02_P5.00mm_Horizontal
- removed R10, R11: 4.7k, Resistor_THT:R_Axial_DIN0207_L6.3mm_D2.5mm_P7.62mm_Horizontal
- removed R12, R14, R16, R18, R20, R22, R24: 10K, Resistor_THT:R_Axial_DIN0207_L6.3mm_D2.5mm_P7.62mm_Horizontal
- removed R13: 20k, Resistor_THT:R_Axial_DIN0207_L6.3mm_D2.5mm_P7.62mm_Horizontal
- removed R15, R23, R25: 13k, Resistor_THT:R_Axial_DIN0207_L6.3mm_D2.5mm_P7.62mm_Horizontal
- removed R17: 1.5K, Resistor_THT:R_Axial_DIN0207_L6.3mm_D2.5mm_P7.62mm_Horizontal
- removed R19: 2k, Resistor_THT:R_Axial_DIN0207_L6.3mm_D2.5mm_P7.62mm_Horizontal
- removed R21: 1.2K, Resistor_THT:R_Axial_DIN0207_L6.3mm_D2.5mm_P7.62mm_Horizontal
- removed SW2, SW3: SW_SPST, Button_Switch_THT:SW_DIP_SPSTx01_Slide_9.78x4.72mm_W7.62mm_P2.54mm
Connections:
- J2 pad 7: 5V -> +5V
