File: KiCAD FILES_PCB/_restore_backup_2026-07-07T10-18-56-602/AWS PROJECT.kicad_sch (KiCad schematic)
At the start: 0 parts

Commit message: Updated LED footprints to THT
Other:
- title: POWER SCHEMATIC -> GENERAL  DESIGN SHEET
Changed lines of the file:
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@@
 	(paper "A4")
 	(title_block
-		(title "POWER SCHEMATIC")
-		(date "2026-07-05")
+		(title "GENERAL  DESIGN SHEET")
 		(company "AdeMNEA IoT-ra")
-		(comment 1 "Designed By Edrine Ssennungi")
+		(comment 1 "Designed By TN Muhanguzi")
 		(comment 2 "For MPSE Research at Makerere University")
 	)
