File: KiCAD FILES_PCB/_restore_backup_2026-07-07T10-18-56-602/gateway.kicad_sch (KiCad schematic)
At the start: 31 parts, among them J1 Real Time Clock, J10 WIND VANE, J11 SD CARD, J12 SOIL TEMP, J13 DHT 22, J14 SH25, J15 ATM PRESSURE, J16 SOIL MOISTURE, J17 +3.3V, J18 +5V, J2 GSM, J4 Conn_01x09_Socket, J5 Conn_01x08_Socket, J6 I2C, J7 WIND SPEED, J8 LIGHT INTENSITY, J9 RAINFALL SENSOR, U1 ESP32-DEVKITC-32U

Commit message: Updated LED footprints to THT
Parts:
- D1, D2: footprint LED_THT:LED_D3.0mm -> LED_SMD:LED_0402_1005Metric
Other:
- title: POWER SCHEMATIC -> GATEWAY BOARD
Changed lines of the file:
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@@
 	(paper "A1")
 	(title_block
-		(title "POWER SCHEMATIC")
-		(date "2026-07-05")
+		(title "GATEWAY BOARD")
+		(date "2026-07-04")
 		(rev "V-1.1")
 		(company "AdeMNEA IoT-ra")
@@
 			(font
 				(size 7.62 7.62)
-				(thickness 1.524)
+				(thickness 1.016)
 				(bold yes)
 			)
@@
 			)
 		)
-		(property "Footprint" "LED_THT:LED_D3.0mm"
+		(property "Footprint" "LED_SMD:LED_0402_1005Metric"
 			(at 152.4 330.2 0)
 			(hide yes)
@@
 			)
 		)
-		(property "Footprint" "LED_THT:LED_D3.0mm"
+		(property "Footprint" "LED_SMD:LED_0402_1005Metric"
 			(at 240.03 328.93 0)
 			(hide yes)
