File: KiCAD FILES__PCB__Ver3/AWS GATEWAY/AWS GATEWAY.kicad_sch (KiCad schematic)
At the start: 36 parts, among them J35 Screw_Terminal_01x02, J36 Screw_Terminal_01x02, J37 Screw_Terminal_01x02, J38 Screw_Terminal_01x02, J39 Screw_Terminal_01x02, J40 Screw_Terminal_01x04, J41 Screw_Terminal_01x04, J42 Screw_Terminal_01x02, J43 Screw_Terminal_01x03, J44 Screw_Terminal_01x03, J45 Screw_Terminal_01x03, J46 Screw_Terminal_01x03, J48 Screw_Terminal_01x02, J49 Screw_Terminal_01x02, J56 Screw_Terminal_01x02, J57 Screw_Terminal_01x02, J58 Screw_Terminal_01x02, J59 Screw_Terminal_01x02, J66 Screw_Terminal_01x02, U1 ESP32-DEVKITC-32U

Commit message: edit on page seetings/titles and version control
Other:
- company: (none) -> IoT-ra Lab
- title: (none) -> AWS GATEWAY SCHEMATIC
Changed lines of the file:
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@@
 	(generator_version "10.0")
 	(paper "A2")
+	(title_block
+		(title "AWS GATEWAY SCHEMATIC")
+		(rev "Version 03")
+		(company "IoT-ra Lab")
+		(comment 1 "For AdEMNEA Project, 2025-2026")
+		(comment 2 "By TN Muhanguzi and team at github.com/marydovika/AWS")
+	)
 	(rectangle
 		(start 171.45 243.332)
