File: KiCAD FILES__PCB__Ver3/AWS POWER/AWS POWER/AWS POWER.kicad_sch (KiCad schematic)
At the start: 44 parts, among them J18 Screw_Terminal_01x02, J47 Screw_Terminal_01x03, J60 Screw_Terminal_01x02, J61 Screw_Terminal_01x02, J62 Screw_Terminal_01x02, J63 Screw_Terminal_01x04, J64 Screw_Terminal_01x02, J65 Screw_Terminal_01x02, J69 Screw_Terminal_01x02, K1 SRD-05VDC-SL-C, K2 SRD-05VDC-SL-C, Q1 NPN, Q2 NPN, SW6 SW_SPST, SW7 SW_SPST

Commit message: edit on page seetings/titles and version control
Other:
- company: (none) -> IoT-ra Lab
- title: (none) -> AWS POWER SCHEMATIC
Changed lines of the file:
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@@
 	(generator_version "10.0")
 	(paper "A2")
+	(title_block
+		(title "AWS POWER SCHEMATIC")
+		(rev "Version 03")
+		(company "IoT-ra Lab")
+		(comment 1 "By TN Muhanguzi, and Intern team on github.com/marydovika/AWS")
+		(comment 2 "For AdEMNEA Project, 2025-2026")
+	)
 	(rectangle
 		(start 340.995 79.375)
